File: pcb/cyberdeck-alpha.kicad_sch (KiCad schematic)
At the start: 426 parts, among them J1 CPU_FAN, J10 Conn_01x30, J11 Conn_01x22, J12 HDMI_C_1.3, J13 USB_C_Receptacle_USB2.0_16P, J14 Conn_01x06, J15 Conn_02x20_Odd_Even, J16 1-2199119-5, J17 2199119-3, J18 SIM_Card, J19 TSOP77438TR, J2 GP_LB, J20 Conn_01x22, J3 GP_RB, J4 JOYSTICK, J5 Conn_01x06_Pin, J6 USB_C_Receptacle_USB2.0_16P, J7 Conn_01x05, J8 PJ-342B, J9 SPK, Q1 IRLML6244, Q2 AO4407A, Q3 AO4407A, Q4 BSS138, Q5 IRLML6244, U1 W25Q128JVS, U10 TPS62180YZFR, U11 TPS62180YZFR, U12 SY6280_OCP, U13 FAN5333ASX, U14 USBLC6-2SC6, U15 SY6280_OCP, U2 STM32F072CBT6, U3 XC6206, U4 S-8254AAWFT-TB-G, U5 RP2040, U6 USBLC6-2SC6, U7 CH334R, U8 PAM8406AB, U9 PCM2706CPJT, X1 X322512MSB4SI, X2 X322512MSB4SI, X3 X322512MSB4SI

Commit message: before M2 B key
Parts:
- H1: value MountingHole -> CM5MountingHoles
- J15: LCSC (none) -> C2895000
- Module3: LCSC (none) -> C6782225
Connections:
- net USB3_0_RX_N: now reaches Module3.128 (USB3-0-RX_N)
- net USB3_0_RX_P: now reaches Module3.130 (USB3-0-RX_P)
- net USB3_0_D_P: now reaches Module3.134 (USB3-0-D_P), SJ1.1
- net USB3_0_D_N: now reaches Module3.136 (USB3-0-D_N), SJ2.1
- net USB3_0_TX_N: now reaches Module3.140 (USB3-0-TX_N)
- net USB3_0_TX_P: now reaches Module3.142 (USB3-0-TX_P)
- no-connect marks 80 -> 92
Other:
- note added: "Rpi CM5"
- moved on the sheet: C28, C32, C33, C79, C83, H1, J10, J11, J20, R42, R54, R55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

Commit message: updates
Parts:
- removed BT3, BT4: Battery_Cell, LibraryGlobalFootprints:JST_PH_B2B-PH-SM4-TB_1x02-1MP_P2.00mm_Vertical, symbol Device:Battery_Cell
- removed C17, C72, C73, C74, C76, C77: 100nF, Capacitor_SMD:C_0402_1005Metric, symbol Adafruit TFP401 to 40pin TFT-eagle-import:CAP_CERAMIC0805-NOOUTLINE
- removed C75: 10uF, Capacitor_SMD:C_0603_1608Metric, symbol Device:C_Small
- removed Q2, Q3: AO4407A, Package_SO:SOIC-8_3.9x4.9mm_P1.27mm, symbol Transistor_FET:FDS9435A
- removed R67, R68, R73, R75: 1K, Resistor_SMD:R_0402_1005Metric, symbol Device:R
- removed R69, R70: 5.1K, Resistor_SMD:R_0402_1005Metric, symbol Device:R
- removed R71: 1M, LED_SMD:LED_0805_2012Metric, symbol Device:R
- removed R72: 10R, Capacitor_SMD:C_0603_1608Metric, symbol Device:R
- removed R74: 0R, LibraryGlobalFootprints:HOT(0.25_1.3)-3.2-0R-I, symbol Device:R
- removed TP3, TP4: TestPoint_Small, TestPoint:TestPoint_Pad_2.0x2.0mm, symbol Connector:TestPoint_Small
- removed U4: S-8254AAWFT-TB-G, LibraryGlobalFootprints:SLM8254AAV, symbol LibraryGlobalSymbols:S-8254AAWFT-TB-G
- added C84: 2.2uF, Capacitor_SMD:C_0603_1608Metric, symbol Device:C_Small
- added C85, C86, C87: 220nF, Capacitor_SMD:C_0402_1005Metric, symbol Device:C_Small
- added C88: 100nF, Capacitor_SMD:C_0402_1005Metric, symbol Device:C_Small
- added C89, C90, C91, C92: 100nF, Capacitor_SMD:C_0402_1005Metric, symbol Adafruit TFP401 to 40pin TFT-eagle-import:CAP_CERAMIC0805-NOOUTLINE
- added D30, D32: RB161QS-40T18R, Diode_SMD:D_0402_1005Metric, symbol Device:D_Schottky
- added D31: MMSZ4678T1G, Diode_SMD:D_SOD-123, symbol Device:D_Zener
- added D33: MMSZ5246BS-7-F, Diode_SMD:D_SOD-323, symbol Device:D_Zener
- added NT1, NT2, NT3, NT4, NT5, NT6: NetTie_2, NetTie:NetTie-2_SMD_Pad0.5mm, symbol Device:NetTie_2
- added Q2: CJ2101, Package_TO_SOT_SMD:SOT-323_SC-70, symbol Device:Q_PMOS_Depletion
- added Q6, Q7: SI4174DY-T1-GE3_N-Channel_FET_SOIC-8, Package_SO:SOIC-8_3.9x4.9mm_P1.27mm, symbol LibraryGlobalSymbols:SI4174DY-T1-GE3_N-Channel_FET_SOIC-8
- added R85, R86: 5.1K, Resistor_SMD:R_0402_1005Metric, symbol Device:R
- added R87: 10M, Capacitor_SMD:C_0603_1608Metric, symbol Device:R
- added R88, R92, R93: 100R, Resistor_SMD:R_0402_1005Metric, symbol Device:R
- added R89, R90, R91: 10R, Resistor_SMD:R_0402_1005Metric, symbol Device:R
- added R94: 1m, Resistor_SMD:R_2512_6332Metric, symbol Device:R_Small
- added R95: 10K, Resistor_SMD:R_0402_1005Metric, symbol Device:R
- added TP6: TestPoint_Small, TestPoint:TestPoint_Pad_2.0x2.0mm, symbol Connector:TestPoint_Small
- added U16: BQ76905RGRR, LibraryGlobalFootprints:IC_BQ76905RGRR, symbol LibraryGlobalSymbols:BQ76905RGRR
- added U17: ATtiny202-SS, Package_SO:SOIC-8_3.9x4.9mm_P1.27mm, symbol MCU_Microchip_ATtiny:ATtiny202-SS
- H2: value M.2 Mounting Hole 3mm -> SMTWE2030MTJ; now in the parts list
- H3: value M.2 Mounting Hole 3mm -> SMTWE2040MTJ; LCSC C2928179 -> C2928181
- J15: now in the parts list
- K_81: value SW_RESET -> TS-1088-AR02016
- K_82: value SW_BOOT -> TS-1088-AR02016
- K_83, K_84: value ButtonSmall -> TS-1088-AR02016
- R65: value 1K -> 82K; LCSC C11702 -> C4142
Connections:
- net +VSYS: now also NT6.2
- net BATT+: now also C92.1, NT1.2, NT2.1, NT6.1; no longer R64.1
- net BATT-: now also BT2.2 (-), C84.2, D33.2 (A), NT3.1, NT4.1, R94.2, R95.2, U16.11 (VSS), U16.21 (EXP)
- net CELL1: now also K_79.2, R90.2; no longer R65.1
- net GND: now also J16.SH1, J17.SH1, C90.1, C91.2, D31.2 (A), Q6.3 (S), R87.1, U17.8 (GND); no longer J12.SH1 (SH), K_79.1, U8.17 (GND_THERMAL)
- net PWR_BTN_DETECT: now reaches R65.2
- net PWR_BTN_DETECT: now also U17.3 (PA7)
- net at R64.2: now also D33.1 (K), Q2.2 (S)
- net PWR_BTN_SOFT: now reaches R66.2
- net PWR_BTN_SOFT: now also U17.2 (PA6)
- net CELL2 renamed CM5_PWR_BTN
- net CM5_PWR_BTN: now also Module2.92 (PWR_BUT); no longer BT2.2 (-)
- removed net CM5_PWR _BTN: K_79.2, Module2.92 (PWR_BUT)
- new net: C86.1, C87.1, NT3.2, R91.2
- new net: NT2.2, R89.2
- new net: D32.2 (A), Q2.3 (D)
- new net: C88.1, NT5.2, R93.2
- new net: Q6.1 (D), Q7.1 (D)
- new net: D31.1 (K), Q6.2 (G), R86.1, R87.2
- new net: C89.1, C90.2
- new net: D30.2 (A), NT1.1
- new net: R92.2, U16.6 (SRP)
- new net: R93.1, U16.7 (SRN)
- new net: Q7.2 (G), R85.1
- new net: C88.2, NT4.2, R92.1
- new net: C91.1, C92.2
- new net: D30.1 (K), R88.2
- new net: K_79.1, R64.1, R65.1, R95.1
- new net BQ_3V3: Q2.1 (G), U16.15 (REGOUT), U17.1 (VCC)
- new net BQ_BATT+: C85.2, R89.1, U16.18 (VC5)
- new net BQ_BATT-: C87.2, R91.1, U16.5 (VC0)
- new net BQ_CELL1: C85.1, C86.2, R90.1, U16.1 (VC3A), U16.19 (VC4A), U16.2 (VC3B), U16.20 (VC4B), U16.3 (VC2), U16.4 (VC1)
- new net BQ_CHG: R86.2, U16.10 (CHG)
- new net BQ_DSG: R85.2, U16.9 (DSG)
- new net BQ_REGSRC: C84.1, R88.1, U16.16 (REGSRC), U16.17 (BAT)
- new net BQ_SCL: U16.12 (SCL), U17.5 (PA2)
- new net BQ_SDA: U16.13 (SDA), U17.4 (PA1)
- new net BQ_TS: D32.1 (K), U16.8 (TS)
- new net DSCH_PATH: C89.2, NT5.1, Q7.3 (S), R94.1
- new net SHIP_MODE: TP6.1, U17.7 (PA3)
- new net TINY202_UPDI: U17.6 (~{RESET}/PA0)
- no-connect marks 92 -> 105
Other:
- moved on the sheet: BT1, BT2, TP1, TP2, TP5

Commit message: BMS and USB-C 3.0 port complete
Parts:
- removed D_70: D_Schottky, Diode_SMD:D_SOD-123, symbol Device:D_Small
- added C17, C72, C73, C74, C75: 100nF, Capacitor_SMD:C_0402_1005Metric, symbol Adafruit TFP401 to 40pin TFT-eagle-import:CAP_CERAMIC0805-NOOUTLINE
- added D34: TPD2EUSB30DRTR, LibraryGlobalFootprints:TPD2EUSB30DRTR, symbol LibraryGlobalSymbols:TPD2EUSB30DRTR
- added J21: DX07S024JJ2R1300, LibraryGlobalFootprints:DX07S024JJ2R1300, symbol LibraryGlobalSymbols:DX07S024JJ2R1300
- added J22: USB3_A, LibraryGlobalFootprints:U-A-39DS-Y-1, symbol Connector:USB3_A
- added NT7: NetTie_2, NetTie:NetTie-2_SMD_Pad0.5mm, symbol Device:NetTie_2
- added R67, R70: 200K, Resistor_SMD:R_0402_1005Metric, symbol Device:R
- added R68: 909K, Resistor_SMD:R_0402_1005Metric, symbol Device:R
- added R69: 10K, Resistor_SMD:R_0402_1005Metric, symbol Device:R
- added U18: TPS25751SRSMR, LibraryGlobalFootprints:TPS25751SRSMR, symbol LibraryGlobalSymbols:TPS25751SRSMR
- added U19: HD3SS3220IRNHT, LibraryGlobalFootprints:HD3SS3220, symbol LibraryGlobalSymbols:HD3SS3220IRNHT
- added U20, U21: TPD4EUSB30DQAR, LibraryGlobalFootprints:TPD4EUSB30DQAR, symbol LibraryGlobalSymbols:TPD4EUSB30DQAR
- added U4: BQ25792RQMR, LibraryGlobalFootprints:BQ25792RQMR, symbol LibraryGlobalSymbols:BQ25792RQMR
- BT1, BT2: LCSC C265003 -> C7433663
Connections:
- net +3.3V_MAIN: now also R67.1, U19.8 (VCC33)
- net +5V_MAIN: now also C17.1, J21.A4 (VBUSA1), J21.A9 (VBUSA2), J21.B4 (VBUSB1), J21.B9 (VBUSB2), R68.1, R69.1, R70.1, U19.30 (VDD5); no longer J13.A4 (VBUS), J13.A9 (VBUS), J13.B4 (VBUS), J13.B9 (VBUS), U14.5 (VBUS)
- net CM5_CC1: no longer J13.A5 (CC1)
- net CM5_CC2: no longer J13.B5 (CC2)
- net GND: now also C17.2, D34.3 (GND), J21.A1 (GNDA1), J21.A12 (GNDA2), J21.B1 (GNDB1), J21.B12 (GNDB2), J21.S1 (SHIELD), J21.S2 (SHIELD), J21.S3 (SHIELD), J21.S4 (SHIELD), NT7.1, U18.11 (GND), U18.12 (GND), U18.14 (GND), U18.33 (GND), U19.12 (~{ENN_MUX}), U19.13 (GND), U19.28 (GND), U19.29 (~{ENN_CC}), U19.31 (EXP_PAD), U20.3, U20.8, U21.3, U21.8; no longer C90.1, C91.2, D31.2 (A), Q6.3 (S), R87.1
- net M2B_USB3_RX_N: now also U19.10 (RXN)
- net M2B_USB3_RX_P: now also U19.9 (RXP)
- net M2B_USB3_TX_N: now also U19.7 (TXN)
- net M2B_USB3_TX_P: now also U19.6 (TXP)
- net M2B_USBD_N: now also D34.1 (D+), J21.A7 (DA-), J21.B7 (DB-)
- net M2B_USBD_P: now also D34.2 (D-), J21.A6 (DA+), J21.B6 (DB+)
- net PWR_BTN_SOFT: no longer names the net of R66.2, U17.2 (PA6)
- new net: C90.1, C91.2, D31.2 (A), NT7.2, Q6.3 (S), R87.1
- new net: R70.2, U19.4 (PORT)
- new net: C75.1, U19.21 (TX2P)
- new net: R67.2, U19.11 (DIR)
- new net: C72.1, U19.16 (TX1N)
- new net: C73.1, U19.17 (TX1P)
- new net: C74.1, U19.20 (TX2N)
- new net: R69.2, U19.3 (CURRENT_MODE)
- new net: R68.2, U19.5 (VBUS_DET)
- new net BAT: U4.22 (BAT), U4.23 (BAT)
- new net PD_CC1: J13.A5 (CC1), U18.24 (CC1)
- new net PD_CC2: J13.B5 (CC2), U18.25 (CC2)
- new net USB31_CC1: J21.A5 (CC1), U19.2 (CC1)
- new net USB31_CC2: J21.B5 (CC2), U19.1 (CC2)
- new net USB31_RX1_N: J21.B10 (RX1-), U19.14 (RX1N), U20.5
- new net USB31_RX1_P: J21.B11 (RX1+), U19.15 (RX1P), U20.4
- new net USB31_RX2_N: J21.A10 (RX2-), U19.18 (RX2N), U21.5
- new net USB31_RX2_P: J21.A11 (RX2+), U19.19 (RX2P), U21.4
- new net USB31_TX1_N: C72.2, J21.A3 (TX1-), U20.2
- new net USB31_TX1_P: C73.2, J21.A2 (TX1+), U20.1
- new net USB31_TX2_N: C74.2, J21.B3 (TX2-), U21.2
- new net USB31_TX2_P: C75.2, J21.B2 (TX2+), U21.1
- new net VBUS: J13.A4 (VBUS), J13.A9 (VBUS), J13.B4 (VBUS), J13.B9 (VBUS), U14.5 (VBUS), U4.2 (VBUS), U4.3 (VBUS)
- no-connect marks 105 -> 111
Other:
- note added: "USB-C 3.0 DFP Port + Mux"
- moved on the sheet: NT6, R66, U17

Commit message: add firmware
Parts:
- added C100, C101, C107: 100nF, Capacitor_SMD:C_0402_1005Metric, symbol Device:C_Small
- added C102, C103, C108, C109, C110, C95, C96, C97, C98, C99: 10uF, Capacitor_SMD:C_0805_2012Metric, symbol Device:C_Small
- added C76: 4.7uF, Capacitor_SMD:C_0402_1005Metric, symbol Device:C_Small
- added C77, C93: 47nF, Capacitor_SMD:C_0402_1005Metric, symbol Device:C_Small
- added C94: 1nF, Capacitor_SMD:C_0402_1005Metric, symbol Device:C_Small
- added D35: LED_0402, LED_SMD:LED_0402_1005Metric, symbol Device:LED
- added L6: 1uH, Inductor_SMD:L_1008_2520Metric, symbol Device:L
- added R71: 100R, Resistor_SMD:R_0402_1005Metric, symbol Device:R
- added R72: 6.04K, Resistor_SMD:R_0402_1005Metric, symbol Device:R
- added R73: 127K, Resistor_SMD:R_0402_1005Metric, symbol Device:R
- added R74: 100K, Resistor_SMD:R_0402_1005Metric, symbol Device:R
- added R75, R96: 10K, Resistor_SMD:R_0402_1005Metric, symbol Device:R_Small
- added R97: 3.3K, Resistor_SMD:R_0402_1005Metric, symbol Device:R
- C17, C20, C32, C66, C67, C68, C69, C70, C71, C72, C73, C74, C75, C79, C83, C89, C90, C91, C92: symbol Adafruit TFP401 to 40pin TFT-eagle-import:CAP_CERAMIC0805-NOOUTLINE -> Device:C_Small
Connections:
- net +3.3V_MAIN: no longer C79.1, C83.1
- net +VSYS: now also U4.25 (SYS), C107.1, C108.2, C109.2, C110.2; no longer C54.2, C55.2, NT6.2, U10.A1 (VIN1), U10.B1 (VIN1), U10.C1 (VIN1), U10.D1 (VIN2), U10.E1 (VIN2), U10.E4 (EN), U10.F1 (VIN2)
- net GND: now also U4.10 (ACDRV2), U4.11 (ACDRV1), U4.13 (~{CE}), U4.27 (GND), C100.2, C101.2, C102.2, C103.1, C107.2, C108.1, C109.1, C110.1, C76.1, C94.2, C95.2, C96.1, C97.2, C98.1, C99.1, R72.1, R74.1, R96.2; no longer C20.1
- net at U4.1 (STAT): now also D35.1 (K)
- net at U4.16 (TS): now also R75.2, R96.1
- net at U4.17 (ILIM_HIZ): now also R73.1, R74.2
- net at U4.18 (BATP): now also R71.1
- net at U4.19 (BTST2): now also C93.1
- net at U4.20 (PROG): now also R72.2
- net at U4.24 (SDRV): now also C94.1
- net at U4.26 (SW2): now also C93.2, L6.2
- net at U4.28 (SW1): now also C77.2, L6.1
- net PMID: now reaches U4.29 (PMID)
- net PMID: now also C100.1, C97.1, C98.2, C99.2
- net at U4.4 (BTST1): now also C77.1
- net at U4.5 (REGN): now also C76.2
- net at U4.8 (VAC2): now also U4.9 (VAC1)
- net BAT renamed +VBATT
- net +VBATT: now also C54.2, C55.2, NT6.2, U10.A1 (VIN1), U10.B1 (VIN1), U10.C1 (VIN1), U10.D1 (VIN2), U10.E1 (VIN2), U10.E4 (EN), U10.F1 (VIN2), C95.1, C96.2, R71.2
- net BATT+ renamed CELL+
- net BATT- renamed CELL-
- net VBUS renamed +VBUS
- net +VBUS: now also C101.1, C102.1, C103.2
- new net: D35.2 (A), R97.1
- new net REGN: R73.2, R75.1, R97.2
- no-connect marks 111 -> 113
Other:
- moved on the sheet: C28, C35, U4

Commit message: charging circuit design
Parts:
- removed R65: 82K, Resistor_SMD:R_0402_1005Metric, symbol Device:R
- added C104, C105, C111, C121, C122: 10uF, Capacitor_SMD:C_0805_2012Metric, symbol Device:C_Small
- added C106, C113, C114, C119, C120: 100nF, Capacitor_SMD:C_0402_1005Metric, symbol Device:C_Small
- added C112: 4.7uF, Capacitor_SMD:C_0402_1005Metric, symbol Device:C_Small
- added C115, C116: 22uF, Capacitor_SMD:C_0805_2012Metric, symbol Device:C_Small
- added C117, C118: 330pF, Capacitor_SMD:C_0603_1608Metric, symbol Device:C_Small
- added Q3, Q8: SI4174DY-T1-GE3_N-Channel_FET_SOIC-8, Package_SO:SOIC-8_3.9x4.9mm_P1.27mm, symbol LibraryGlobalSymbols:SI4174DY-T1-GE3_N-Channel_FET_SOIC-8
- J22: now not fitted; now left out of the parts list
Connections:
- net +3.3V_MAIN: now also U18.32 (VIN_3V3)
- net +5V_MAIN: now also U18.28 (PP5V), U18.29 (PP5V), C119.1, C120.1, C121.1, C122.1
- net +VBUS: now also U18.26 (VBUS), U18.27 (VBUS), C106.1, C112.1, C113.1, C114.1, Q8.3 (S); no longer C101.1, C102.1, C103.2, U4.2 (VBUS), U4.3 (VBUS)
- net BQ_REGSRC: now also C84.2; no longer C84.1
- net CELL-: now also C84.1; no longer C84.2
- net CELL1: no longer K_79.2
- net CM5_PWR_BTN: now also K_79.1
- net CM5_USB_D_N: now also U18.23 (GPIO5/USB_N/MD2)
- net CM5_USB_D_P: now also U18.22 (GPIO5/USB_P/MD1)
- net GND: now also K_79.2, C104.2, C105.2, C106.2, C111.2, C112.2, C113.2, C114.2, C115.2, C116.2, C117.1, C118.1, C119.2, C120.2, C121.2, C122.2
- net PD_CC1: now also C117.2
- net PD_CC2: now also C118.2
- net CHG_SCL: now reaches U4.14 (SCL)
- net CHG_SCL: now also U18.16 (I2Cc_SCL)
- net CHG_SDA: now reaches U4.15 (SDA)
- net CHG_SDA: now also U18.15 (I2Cc_SDA)
- net CHG_INT: now reaches U4.21 (~{INT})
- net CHG_INT: now also U18.17 (I2Cc_IRQ)
- net CHG_3V3: now reaches R64.1, R95.1
- net CHG_3V3: now also U18.1 (LDO_3V3), C104.1; no longer K_79.1
- net +VCHG: now reaches U18.19 (VSYS)
- net +VCHG: now also C101.1, C102.1, C103.2, U4.2 (VBUS), U4.3 (VBUS), C111.1, C115.1, C116.1, Q3.3 (S)
- net GATE_VCHG: now reaches U18.20 (GATE_VSYS)
- net GATE_VCHG: now also Q3.2 (G)
- net GATE_VBUS: now reaches U18.21 (GATE_VBUS)
- net GATE_VBUS: now also Q8.2 (G)
- net at U18.4 (LDO_1V5): now also C105.1
- net PWR_BTN_DETECT: no longer names the net of U17.3 (PA7)
- new net: Q3.1 (D), Q8.1 (D)
- no-connect marks 113 -> 114
Other:
- note added: "Battery Charger"
- note added: "CM5 USB System Port"
- note added: "USB A Port"
- note added: "USB PD Power Supply"
- note removed: "CM5 USB Port"
- moved on the sheet: C100, C101, C102, C103, C107, C108, C109, C110, C84, C85, C86, C87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

Commit message: added power and charging to layout
Parts:
- removed NT4, NT5: NetTie_2, NetTie:NetTie-2_SMD_Pad0.5mm, symbol Device:NetTie_2
- added C123: 100nF, Capacitor_SMD:C_0402_1005Metric, symbol Device:C_Small
- added JP1, JP2: SolderJumper_3_Open, Jumper:SolderJumper-3_P1.3mm_Open_RoundedPad1.0x1.5mm, symbol Jumper:SolderJumper_3_Open
- added K_85: TS-1088-AR02016, LibraryGlobalFootprints:BTN_SMD_4x3mm, symbol Switch:SW_Push
- added SJ10: 3V_IN, LibraryGlobalFootprints:SOLDERJUMPER_ARROW_NOPASTE, symbol Adafruit TFP401 to 40pin TFT-eagle-import:SOLDERJUMPER
- added SJ11: 5V_IN, LibraryGlobalFootprints:SOLDERJUMPER_ARROW_NOPASTE, symbol Adafruit TFP401 to 40pin TFT-eagle-import:SOLDERJUMPER
- added SJ12: 5V_OUT, LibraryGlobalFootprints:SOLDERJUMPER_ARROW_NOPASTE, symbol Adafruit TFP401 to 40pin TFT-eagle-import:SOLDERJUMPER
- added SJ13: 3V_OUT, LibraryGlobalFootprints:SOLDERJUMPER_ARROW_NOPASTE, symbol Adafruit TFP401 to 40pin TFT-eagle-import:SOLDERJUMPER
- added SJ14: SHP_OFF, LibraryGlobalFootprints:SOLDERJUMPER_ARROW_NOPASTE, symbol Adafruit TFP401 to 40pin TFT-eagle-import:SOLDERJUMPER
- added SJ15: PD_PSU, LibraryGlobalFootprints:SOLDERJUMPER_ARROW_NOPASTE, symbol Adafruit TFP401 to 40pin TFT-eagle-import:SOLDERJUMPER
- added SJ8: 3V_EN, LibraryGlobalFootprints:SOLDERJUMPER_ARROW_NOPASTE, symbol Adafruit TFP401 to 40pin TFT-eagle-import:SOLDERJUMPER
- added SJ9: 5V_EN, LibraryGlobalFootprints:SOLDERJUMPER_ARROW_NOPASTE, symbol Adafruit TFP401 to 40pin TFT-eagle-import:SOLDERJUMPER
- added TP10, TP11, TP12, TP3, TP4, TP7, TP8: TestPoint_Small, TestPoint:TestPoint_Pad_2.0x2.0mm, symbol Connector:TestPoint_Small
- added U22: AT24CS01-SSHM, Package_SO:SOIC-8_3.9x4.9mm_P1.27mm, symbol Memory_EEPROM:AT24CS01-SSHM
- Q3, Q6, Q7, Q8: LCSC C144929 -> C144929
Connections:
- net +3.3V_MAIN: now also C79.1, C83.1, C123.1, SJ13.1, U22.8 (VCC); no longer C64.2, C65.2, L3.2, L4.2, R51.2, R52.2, U11.A4 (VO)
- net +5V_MAIN: now also SJ12.1; no longer C56.2, C57.2, C58.2, C59.2, C61.2, C62.2, L1.2, L2.2, R48.2, R49.2, U10.A4 (VO), U11.A1 (VIN1), U11.B1 (VIN1), U11.C1 (VIN1), U11.D1 (VIN2), U11.E1 (VIN2), U11.E4 (EN), U11.F1 (VIN2)
- net +VBATT: no longer C54.2, C55.2, U10.A1 (VIN1), U10.B1 (VIN1), U10.C1 (VIN1), U10.D1 (VIN2), U10.E1 (VIN2), U10.E4 (EN), U10.F1 (VIN2)
- net +VBUS: now also Q8.1 (S), Q8.2 (S)
- net +VCHG: now also SJ15.1; no longer C111.1, C115.1, C116.1, Q3.3 (S), U18.19 (VSYS)
- net +VSYS: now also SJ11.2
- net CELL-: now also C88.2, R92.1
- net CHG_INT: now also TP12.1
- net CHG_SCL: now also TP10.1, U22.6 (SCL)
- net CHG_SDA: now also TP11.1, U22.5 (SDA)
- net CM5_USB_D_N: now also JP2.2 (C); no longer U14.6 (I/O1), U18.23 (GPIO5/USB_N/MD2)
- net CM5_USB_D_P: now also JP1.2 (C); no longer U14.4 (I/O2), U18.22 (GPIO5/USB_P/MD1)
- net DSCH_PATH: now also C88.1, Q7.1 (S), Q7.2 (S), R93.2
- net GATE_VBUS: now also Q8.4 (G); no longer Q8.2 (G)
- net GATE_VCHG: now also Q3.4 (G); no longer Q3.2 (G)
- net GND: now also C123.2, K_85.2, TP3.1, U22.1 (A0), U22.2 (A1), U22.3 (A2), U22.4 (GND), U22.7 (WP)
- net HUB_US_D+: now also JP1.1 (A)
- net HUB_US_D-: now also JP2.1 (A)
- net M2B_USB3_RX_N: now also U19.9 (RXP); no longer U19.10 (RXN)
- net M2B_USB3_RX_P: now also U19.10 (RXN); no longer U19.9 (RXP)
- net REGN: now also C76.2, U4.5 (REGN)
- net SHIP_MODE: now also K_85.1; no longer TP6.1
- net TINY202_UPDI: now also TP4.1
- net USB31_RX1_N: now also U19.15 (RX1P), U20.2, U20.9 (NC_9); no longer U19.14 (RX1N), U20.5
- net USB31_RX1_P: now also U19.14 (RX1N), U20.1, U20.10 (NC_10); no longer U19.15 (RX1P), U20.4
- net USB31_RX2_N: now also U21.1, U21.10 (NC_10); no longer U21.5
- net USB31_RX2_P: now also U21.2, U21.9 (NC_9); no longer U21.4
- net USB31_TX1_N: now also U20.5, U20.6 (NC_6); no longer U20.2
- net USB31_TX1_P: now also U20.4, U20.7 (NC_7); no longer U20.1
- net USB31_TX2_N: now also C75.2, U21.4, U21.7 (NC_7); no longer C74.2, U21.2
- net USB31_TX2_P: now also C74.2, U21.5, U21.6 (NC_6); no longer C75.2, U21.1
- net GND_OUT: now reaches C90.1, C91.2, D31.2 (A), NT7.2, Q6.3 (S), R87.1
- net GND_OUT: now also Q6.1 (S), Q6.2 (S)
- net at D31.1 (K), R86.1, R87.2: now also Q6.4 (G); no longer Q6.2 (G)
- net at R85.1: now also Q7.4 (G); no longer Q7.2 (G)
- net +VCHG_OUT: now reaches Q3.1 (S)
- net +VCHG_OUT: now also C111.1, C115.1, C116.1, Q3.2 (S), Q3.3 (S), U18.19 (VSYS), SJ15.2; no longer Q8.1 (D)
- net at C75.1: now also U19.20 (TX2N); no longer U19.21 (TX2P)
- net at U19.16 (TX1N): now also C73.1; no longer C72.1
- net at U19.17 (TX1P): now also C72.1; no longer C73.1
- net at C74.1: now also U19.21 (TX2P); no longer U19.20 (TX2N)
- net at U18.10 (I2Ct_IRQ): now also TP6.1
- net at U18.8 (I2Ct_SDA): now also TP7.1
- net at U18.9 (I2Ct_SCL): now also TP8.1
- net CHG_3V3: no longer names the net of R64.1, R95.1
- net CHG_3V3: now also SJ14.2; no longer C104.1, U18.1 (LDO_3V3)
- new net: SJ9.1, U10.E4 (EN)
- new net: Q6.5 (D), Q6.6 (D), Q6.7 (D), Q6.8 (D), Q7.5 (D), Q7.6 (D), Q7.7 (D), Q7.8 (D)
- new net: Q3.5 (D), Q3.6 (D), Q3.7 (D), Q3.8 (D), Q8.5 (D), Q8.6 (D), Q8.7 (D), Q8.8 (D)
- new net: SJ8.1, U11.E4 (EN)
- new net 3V3_IN: C61.2, C62.2, SJ10.1, SJ8.2, U11.A1 (VIN1), U11.B1 (VIN1), U11.C1 (VIN1), U11.D1 (VIN2), U11.E1 (VIN2), U11.F1 (VIN2)
- new net 3V3_MAIN: C64.2, C65.2, L3.2, L4.2, R51.2, R52.2, SJ13.2, U11.A4 (VO)
- new net 3V3_SHIP_MODE_OFF: C104.1, SJ14.1, U18.1 (LDO_3V3)
- new net 5V_IN: C54.2, C55.2, SJ11.1, SJ9.2, U10.A1 (VIN1), U10.B1 (VIN1), U10.C1 (VIN1), U10.D1 (VIN2), U10.E1 (VIN2), U10.F1 (VIN2)
- new net 5V_MAIN: C56.2, C57.2, C58.2, C59.2, L1.2, L2.2, R48.2, R49.2, SJ10.2, SJ12.2, U10.A4 (VO)
- new net USB2_SYS_N: JP2.3 (B), U14.6 (I/O1), U18.23 (GPIO5/USB_N/MD2)
- new net USB2_SYS_P: JP1.3 (B), U14.4 (I/O2), U18.22 (GPIO5/USB_P/MD1)
Other:
- note added: "USB-C PD Charge / CM5 System Port"
- note removed: "CM5 USB System Port"
- moved on the sheet: C100, C101, C102, C103, C107, C108, C109, C110, C61, C62, C63, C64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
