File: pcb-deck/cyberdeck-alpha.kicad_pcb (KiCad board)
At the start: 4 copper layers, 105.8 x 160.2 mm, 532 parts, among them J1 CPU_FAN, J10 DM3AT-SF-PEJM5, J11 Conn_01x22, J12 HDMI_C_1.3, J13 USB_C_Receptacle_USB2.0_16P, J15 PZ254-2-20-W-8.5, J16 1-2199119-5, J19 TSOP77438TR, J2 GP_LB, J20 Conn_01x22, J21 DX07S024JJ2R1300, J22 USB3_A, J3 GP_RB, J4 JOYSTICK, J5 Conn_01x06_Pin, J6 USB_C_Receptacle_USB2.0_16P, J7 Conn_01x05, J8 PJ-342B, J9 SPK, Q1 IRLML6244, Q2 CJ2101, Q3 SI4174DY-T1-GE3_N-Channel_FET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, Q5 IRLML6244, Q6 SI4174DY-T1-GE3_N-Channel_FET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, Q7 SI4174DY-T1-GE3_N-Channel_FET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, Q8 SI4174DY-T1-GE3_N-Channel_FET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, U1 W25Q128JVS, U10 TPS62180YZFR, U11 TPS62180YZFR, U12 SY6280_OCP, U13 USBLC6-2SC6, U14 USBLC6-2SC6, U15 SY6280_OCP, U16 BQ76905RGRR, U17 ATtiny404-SS, U18 TPS25751SRSMR, U19 HD3SS3220IRNHT, U2 STM32F072CBT6, U20 TPD4EUSB30DQAR, U21 TPD4EUSB30DQAR, U22 AT24CS01-SSHM, U23 CH334R, U24 PC817, U25 SY6280_OCP, U26 SY6280_OCP, U27 PC817, U28 SY6280_OCP, U3 XC6206, U4 BQ25792RQMR, U5 RP2040, U6 USBLC6-2SC6, U7 CH334R, U8 PAM8406AB, U9 PCM2706CPJT, X1 X322512MSB4SI, X2 X322512MSB4SI, X3 X322512MSB4SI, X4 X322512MSB4SI

Commit message: pcb updates
Parts:
- removed K_80: ZX-QC66-4.3TP, LibraryGlobalFootprints:ZX-QC66-7.5TP
- added C131: 100nF, Capacitor_SMD:C_0402_1005Metric, B.Cu at (177.6, 24.1)
- added C132: 100nF, Capacitor_SMD:C_0402_1005Metric, B.Cu at (202.6, 68.6)
- added C133: 1nF-2kV, Capacitor_SMD:C_1206_3216Metric, B.Cu at (78.8, 133.9)
- added C134: 100nF, Capacitor_SMD:C_0402_1005Metric, B.Cu at (74.5, 118.1)
- added C135: 10nF, Capacitor_SMD:C_0402_1005Metric, B.Cu at (74.5, 120.0)
- added C136: 100nF, Capacitor_SMD:C_0402_1005Metric, B.Cu at (74.5, 122.0)
- added C78: 20pF, Capacitor_SMD:C_0402_1005Metric, B.Cu at (169.2, 31.6)
- added C80: 20pF, Capacitor_SMD:C_0402_1005Metric, B.Cu at (166.5, 31.6)
- added C81: 20pF, Capacitor_SMD:C_0402_1005Metric, B.Cu at (167.8, 31.6)
- added C82: 0.1µF, Capacitor_SMD:C_0402_1005Metric, B.Cu at (158.4, 17.1)
- added D24: SMF05C, LibraryGlobalFootprints:SMF05C, B.Cu at (167.7, 38.1)
- added D25: LED_0402, LED_SMD:LED_0402_1005Metric, B.Cu at (149.1, 16.9)
- added D26: LED_0402, LED_SMD:LED_0402_1005Metric, B.Cu at (74.3, 114.1)
- added D37: LED_0402, LED_SMD:LED_0402_1005Metric, B.Cu at (74.3, 116.1)
- added H3: SMTWE2025MTJ, LibraryGlobalFootprints:M.2 M2 nut standoff, B.Cu at (164.8, 64.8)
- added H4: SMTWE2030MTJ, LibraryGlobalFootprints:M.2 M2 nut standoff, F.Cu at (233.5, 72.2)
- added J14: USB_C_Receptacle_USB2.0_16P, LibraryGlobalFootprints:USB_C_Receptacle_HRO_TYPE-C-31-M-12, B.Cu at (90.1, 49.7)
- added J17: 2199230-3, LibraryGlobalFootprints:2199230-3 M.2 B key, B.Cu at (164.9, 23.1)
- added J18: SIM_Card, LibraryGlobalFootprints:MICRO SIM 7P H1.35, B.Cu at (165.2, 43.8)
- added K_79: GP_MODE, LibraryGlobalFootprints:dome-tactile-pad, F.Cu at (202.0, 112.0)
- added R108: 100K, Resistor_SMD:R_0402_1005Metric, B.Cu at (200.1, 59.9)
- added R109: 3.4K, Resistor_SMD:R_0402_1005Metric, B.Cu at (178.7, 18.8)
- added R110: 470R, Resistor_SMD:R_0402_1005Metric, B.Cu at (74.5, 135.2)
- added R111: 3.4K, Resistor_SMD:R_0402_1005Metric, B.Cu at (202.6, 66.6)
- added R112: 75R, Resistor_SMD:R_0603_1608Metric, B.Cu at (78.0, 114.4)
- added R113: 75R, Resistor_SMD:R_0603_1608Metric, B.Cu at (78.0, 116.9)
- added R114: 75R, Resistor_SMD:R_0603_1608Metric, B.Cu at (78.0, 119.4)
- added R115: 75R, Resistor_SMD:R_0603_1608Metric, B.Cu at (78.0, 121.9)
- added R116: 100R, Resistor_SMD:R_0402_1005Metric, B.Cu at (74.5, 137.2)
- added R117: 100R, Resistor_SMD:R_0402_1005Metric, B.Cu at (74.5, 139.2)
- added R76: 22R, Resistor_SMD:R_0402_1005Metric, B.Cu at (169.2, 33.6)
- added R77: 22R, Resistor_SMD:R_0402_1005Metric, B.Cu at (166.5, 33.6)
- added R78: 22R, Resistor_SMD:R_0402_1005Metric, B.Cu at (167.8, 33.6)
- added R79: 10K, Resistor_SMD:R_0402_1005Metric, B.Cu at (170.6, 28.4)
- added R80: 10K, Resistor_SMD:R_0402_1005Metric, B.Cu at (168.6, 28.4)
- added R81: 3.3K, Resistor_SMD:R_0402_1005Metric, B.Cu at (150.8, 17.2)
- added R82: 470R, Resistor_SMD:R_0402_1005Metric, B.Cu at (74.5, 133.2)
- added SJ1: PCIE_PWR, LibraryGlobalFootprints:SOLDERJUMPER_ARROW_NOPASTE, B.Cu at (202.5, 60.0)
- added U29: SY6280_OCP, Package_TO_SOT_SMD:SOT-23-5, B.Cu at (178.2, 21.4)
- added U30: SY6280_OCP, Package_TO_SOT_SMD:SOT-23-5, B.Cu at (206.6, 66.0)
- added U31: ~, LibraryGlobalFootprints:G24P02S, B.Cu at (90.3, 134.2)
- added U32: AT3H7B-CuH-S, Package_SO:SSOP-4_4.4x2.6mm_P1.27mm, B.Cu at (40.5, 74.3)
- J9: value SPK -> RJ45_LED_Shielded; footprint LibraryGlobalFootprints:1x04_P2.54 SMD pads only -> LibraryGlobalFootprints:RC01812
- K_73: value ZX-QC66-4.3TP -> GP_START; footprint LibraryGlobalFootprints:ZX-QC66-7.5TP -> LibraryGlobalFootprints:dome-tactile-pad
- K_74: value ZX-QC66-4.3TP -> GP_SELECT; footprint LibraryGlobalFootprints:ZX-QC66-7.5TP -> LibraryGlobalFootprints:dome-tactile-pad
- R87: footprint Capacitor_SMD:C_0603_1608Metric -> Resistor_SMD:R_0603_1608Metric
- U24: value PC817 -> AT3H7B-CuH-S; footprint LibraryGlobalFootprints:PC817X3CSP9F -> Package_SO:SSOP-4_4.4x2.6mm_P1.27mm
- U27: value PC817 -> USBLC6-2SC6; footprint LibraryGlobalFootprints:PC817X3CSP9F -> Package_TO_SOT_SMD:SOT-23-6
- moved G*** 235.5 mm to (29.2, 74.2)
- moved G*** 235.5 mm to (29.5, 60.6)
- moved S1 190.1 mm to (62.7, 20.8), turned to 90 degrees
- moved C130 174.5 mm to (253.1, 25.2), turned to -90 degrees
- moved R103 171.1 mm to (253.1, 27.1), turned to 90 degrees
- moved C129 167.9 mm to (249.5, 29.3), turned to -90 degrees
- moved R102 164.4 mm to (249.5, 31.3), turned to -90 degrees
- moved R104 163.5 mm to (242.6, 28.8)
- moved U28 160.9 mm to (251.8, 30.4), turned to -90 degrees
- moved J10 150.6 mm to (244.8, 19.2), turned to 0 degrees
- moved C128 146.2 mm to (252.8, 74.0), turned to 90 degrees
- moved R59 142.6 mm to (252.8, 72.0), turned to -90 degrees
- moved R60 138.2 mm to (246.8, 71.9), turned to 0 degrees
- moved U26 135.8 mm to (250.1, 73.3), turned to 0 degrees
- moved D_70 134.9 mm to (243.2, 72.6), turned to 0 degrees
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Connections:
- C70 pad 1: +3.3V_MAIN -> +3.3V_M2PCIE
- C71 pad 1: +3.3V_MAIN -> +3.3V_M2PCIE
- J10 pad 5: unconnected-(J10-CLK-Pad5) -> /SD_CLK
- J10 pad P1: Net-(J10-SHIELD-PadP1) -> GND
- J13 pad A4: +VBUS -> Net-(U14-VBUS)
- J13 pad A5: /PD_CC1 -> /CM5_CC1
- J13 pad A9: +VBUS -> Net-(U14-VBUS)
- J13 pad B4: +VBUS -> Net-(U14-VBUS)
- J13 pad B5: /PD_CC2 -> /CM5_CC2
- J13 pad B9: +VBUS -> Net-(U14-VBUS)
- J16 pad 12: +3.3V_MAIN -> +3.3V_M2PCIE
- J16 pad 14: +3.3V_MAIN -> +3.3V_M2PCIE
- J16 pad 16: +3.3V_MAIN -> +3.3V_M2PCIE
- J16 pad 18: +3.3V_MAIN -> +3.3V_M2PCIE
- J16 pad 2: +3.3V_MAIN -> +3.3V_M2PCIE
- J16 pad 4: +3.3V_MAIN -> +3.3V_M2PCIE
- J16 pad 70: +3.3V_MAIN -> +3.3V_M2PCIE
- J16 pad 72: +3.3V_MAIN -> +3.3V_M2PCIE
- J16 pad 74: +3.3V_MAIN -> +3.3V_M2PCIE
- J7 pad 1: /JOYSTICK_Y -> +3.3V_MAIN
- J7 pad 2: GND -> /JOYSTICK_X
- J7 pad 4: /JOYSTICK_X -> GND
- J7 pad 5: +3.3V_MAIN -> /JOYSTICK_Y
- J9 pad 1: Net-(J9-Pin_1) -> /ETH_TX0_P
- J9 pad 2: Net-(J9-Pin_2) -> /ETH_TX0_N
- J9 pad 3: Net-(J9-Pin_3) -> /ETH_RX1_P
- J9 pad 4: Net-(J9-Pin_4) -> /ETH_BL2_P
- LS1 pad 1: Net-(J9-Pin_2) -> Net-(U8-LOUT-)
- LS1 pad 2: Net-(J9-Pin_1) -> Net-(U8-LOUT+)
- LS2 pad 1: Net-(J9-Pin_3) -> Net-(U8-ROUT-)
- LS2 pad 2: Net-(J9-Pin_4) -> Net-(U8-ROUT+)
- Module2 pad 10: unconnected-(Module2-Ethernet_Pair0_N-Pad10) -> /ETH_D0_N
- Module2 pad 11: unconnected-(Module2-Ethernet_Pair2_P-Pad11) -> /ETH_D2_P
- Module2 pad 12: unconnected-(Module2-Ethernet_Pair0_P-Pad12) -> /ETH_D0_P
- Module2 pad 15: unconnected-(Module2-Ethernet_nLED3(3.3v)-Pad15) -> /ETH_LED_G
- Module2 pad 17: unconnected-(Module2-Ethernet_nLED2(3.3v)-Pad17) -> /ETH_LED_Y
- Module2 pad 18: unconnected-(Module2-Ethernet_SYNC_OUT(3.3v)-Pad18) -> /IEEE1588_SYNC_OUT_3V3
- Module2 pad 21: unconnected-(Module2-LED_nACT-Pad21) -> /CM5_ACT_LED
- Module2 pad 3: unconnected-(Module2-Ethernet_Pair3_P-Pad3) -> /ETH_D3_P
- Module2 pad 4: unconnected-(Module2-Ethernet_Pair1_P-Pad4) -> /ETH_D1_P
- Module2 pad 5: unconnected-(Module2-Ethernet_Pair3_N-Pad5) -> /ETH_D3_N
- Module2 pad 6: unconnected-(Module2-Ethernet_Pair1_N-Pad6) -> /ETH_D1_N
- Module2 pad 9: unconnected-(Module2-Ethernet_Pair2_N-Pad9) -> /ETH_D2_N
- Module2 pad 95: unconnected-(Module2-LED_nPWR-Pad95) -> /CM5_PWR_LED
- Module3 pad 106: /PCIE-PWR_EN -> /M2B_POWER_OFF
- R45 pad 2: unconnected-(R45-Pad2) -> Net-(U9-D+)
- U13 pad 4: /HUB2_DS_1_D+ -> /PORT_USBA2_D+
- U13 pad 6: /HUB2_DS_1_D- -> /PORT_USBA2_D-
- U14 pad 5: +VBUS -> Net-(U14-VBUS)
- U18 pad 22: /USB2_D_P -> /CHG_USBD_P
- U18 pad 23: /USB2_D_N -> /CHG_USBD_N
- U27 pad 1: unconnected-(U27-Pad1) -> Net-(J14-D--PadA7)
- U27 pad 2: unconnected-(U27-Pad2) -> GND
- U27 pad 3: unconnected-(U27-Pad3) -> Net-(J14-D+-PadA6)
- U27 pad 4: unconnected-(U27-Pad4) -> /CHG_USBD_P
- U5 pad 38: /JOYSTICK_X -> /JOYSTICK_Y
- U5 pad 39: /JOYSTICK_Y -> /JOYSTICK_X
- U6 pad 5: +5V_PORT -> +5V_PORT_C
- U8 pad 1: Net-(J9-Pin_1) -> Net-(U8-LOUT+)
- U8 pad 14: Net-(J9-Pin_3) -> Net-(U8-ROUT-)
- U8 pad 16: Net-(J9-Pin_4) -> Net-(U8-ROUT+)
- U8 pad 3: Net-(J9-Pin_2) -> Net-(U8-LOUT-)
Routing:
- net +3.3V_MAIN: track 533.1 -> 289.9 mm, vias 26 -> 15
- net (no net): track 185.7 -> 34.3 mm, vias 10 -> 2
- net +5V_MAIN: track 406.9 -> 274.1 mm, vias 14 -> 9
- net /PD_CC1: track 143.6 -> 19.3 mm, vias 5 -> 3
- net /USB2_D_P: track 120.3 -> 0.00 mm, vias 3 -> 0
- net /PD_CC2: track 138.0 -> 18.5 mm, vias 7 -> 3
- net /USB2_D_N: track 118.6 -> 0.00 mm, vias 3 -> 0
- net /MIPI1_SDA: track 170.2 -> 57.5 mm, vias 5 -> 3
- net /MIPI1_SCL: track 171.1 -> 60.9 mm, vias 6 -> 2
- net +VBUS: track 134.4 -> 27.1 mm, vias 5 -> 1
- net /CM5_PWR_BTN: track 116.0 -> 31.0 mm, vias 3 -> 1
- net /CM5_USB_OTG_ID: track 59.9 -> 0.00 mm, vias 2 -> 0
- net /HUB_US_D-: track 120.2 -> 60.6 mm, vias 4 -> 1
- net /MIPI1_D3_P: track 1.74 -> 59.5 mm, vias 1 -> 2
- net /HUB_US_D+: track 115.5 -> 59.0 mm, vias 3 -> 1
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Other:
- board size 105.8 x 160.2 mm -> 195.4 x 160.2 mm
- board text added: "2230"
- board text added: "2242"
- board text added: "40"
- board text added: "CHG"
- board text added: "Camera"
- board text added: "GPIO16/26"
- board text added: "M.2 PCIe / NVMe"
- board text added: "MICROSD"
- board text added: "MIPI1"
- board text added: "USB-A 5Gbps"
- board text removed: "1-2: 22pin DSI, 2-3: 30pin DSI"
- board text removed: "123"
- board text removed: "22P"
- board text removed: "30P"
- board text removed: "<-- use flux!"
- board text removed: "BACKLITE DRIVER"
- board text removed: "GPIO16"
- board text removed: "GPIO26"
- board text removed: "L+"
- board text removed: "L-"
- board text removed: "M.2 NVMe SSD"
- board text removed: "MIPI 1"
- board text removed: "R+"
- board text removed: "R-"
- board text removed: "SPEAKERS"
