File: pcb-deck/cyberdeck-alpha.kicad_pcb (KiCad board)
At the start: 4 copper layers, 195.4 x 160.2 mm, 573 parts, among them J1 CPU_FAN, J10 DM3AT-SF-PEJM5, J11 Conn_01x22, J12 HDMI_C_1.3, J13 USB_C_Receptacle_USB2.0_16P, J14 USB_C_Receptacle_USB2.0_16P, J15 PZ254-2-20-W-8.5, J16 1-2199119-5, J17 2199230-3, J18 SIM_Card, J19 TSOP77438TR, J2 GP_LB, J20 Conn_01x22, J21 DX07S024JJ2R1300, J22 USB3_A, J3 GP_RB, J4 JOYSTICK, J5 Conn_01x06_Pin, J6 USB_C_Receptacle_USB2.0_16P, J7 Conn_01x05, J8 PJ-342B, J9 RJ45_LED_Shielded, Q1 IRLML6244, Q2 CJ2101, Q3 SI4174DY-T1-GE3_N-Channel_FET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, Q5 IRLML6244, Q6 SI4174DY-T1-GE3_N-Channel_FET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, Q7 SI4174DY-T1-GE3_N-Channel_FET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, Q8 SI4174DY-T1-GE3_N-Channel_FET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, U1 W25Q128JVS, U10 TPS62180YZFR, U11 TPS62180YZFR, U12 SY6280_OCP, U13 USBLC6-2SC6, U14 USBLC6-2SC6, U15 SY6280_OCP, U16 BQ76905RGRR, U17 ATtiny404-SS, U18 TPS25751SRSMR, U19 HD3SS3220IRNHT, U2 STM32F072CBT6, U20 TPD4EUSB30DQAR, U21 TPD4EUSB30DQAR, U22 AT24CS01-SSHM, U23 CH334R, U24 AT3H7B-CuH-S, U25 SY6280_OCP, U26 SY6280_OCP, U27 USBLC6-2SC6, U28 SY6280_OCP, U29 SY6280_OCP, U3 XC6206, U30 SY6280_OCP, U32 AT3H7B-CuH-S, U4 BQ25792RQMR, U5 RP2040, U6 USBLC6-2SC6, U7 CH334R, U8 PAM8406AB, U9 PCM2706CPJT, X1 X322512MSB4SI, X2 X322512MSB4SI, X3 X322512MSB4SI, X4 X322512MSB4SI

Commit message: add firmwares
Parts:
- removed the G*** at (184.4, 73.7)
- moved J9 67.0 mm to (160.7, 112.2)
- moved F1 3.28 mm to (164.5, 120.0)
- moved K_76 0.78 mm to (161.7, 107.0)
- moved K_77 0.78 mm to (155.0, 100.2)
- moved K_78 0.77 mm to (168.5, 100.2)
- moved K_75 0.69 mm to (161.8, 93.5)
Routing:
- net +5V_MAIN: track 274.1 -> 270.8 mm
- net +5V_KB: track 4.02 -> 7.28 mm
- net /GP_BTN_DN: track 67.4 -> 66.9 mm
Other:
- outline, holes or cut-outs redrawn
- board text added: "A"
- board text added: "B"
- board text added: "MODE"
- board text added: "POWER"
- board text added: "SELECT"
- board text added: "START"
- board text removed: "LAY THINE EYES VPON IT, AND SEE THAT IT IS BARREN{dblquote}"
- board text removed: "MODE_BTN"
- board text removed: "POWER_BTN"
- board text removed: "PWR_LED"
- board text removed: "SELECT_BTN"
- board text removed: "START_BTN"
- board text removed: "{dblquote}BEHOLD! THE PCB ON WHICH I PLACE MINE FVCKS"
