File: pcb-deck/cyberdeck-alpha.kicad_pcb (KiCad board)
At the start: 4 copper layers, 208.1 x 160.2 mm, 611 parts, among them J1 CPU_FAN, J10 DM3AT-SF-PEJM5, J11 Conn_01x22, J12 HDMI_C_1.3, J13 USB_C_Receptacle_USB2.0_16P, J14 USB_C_Receptacle_USB2.0_16P, J15 PZ254-2-20-W-8.5, J16 1-2199119-5, J17 2199230-3, J18 SIM_Card, J19 TSOP77438TR, J2 GP_LB, J20 Conn_01x22, J21 DX07S024JJ2R1300, J22 USB3_A, J23 Conn_01x06_Pin, J24 Conn_01x06_Pin, J25 USB_C_Receptacle_USB2.0_16P, J3 GP_RB, J4 JOYSTICK, J5 Conn_01x06_Pin, J6 USB_C_Receptacle_USB2.0_16P, J7 Conn_01x05, J8 PJ-342B, J9 RJ45_LED_Shielded, Q1 IRLML6244, Q2 CJ2101, Q3 SI4174DY-T1-GE3_N-Channel_FET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, Q5 IRLML6244, Q6 SI4174DY-T1-GE3_N-Channel_FET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, Q7 SI4174DY-T1-GE3_N-Channel_FET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, Q8 SI4174DY-T1-GE3_N-Channel_FET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, U1 W25Q128JVS, U10 TPS62180YZFR, U11 TPS62180YZFR, U12 SY6280_OCP, U13 USBLC6-2SC6, U14 USBLC6-2SC6, U15 SY6280_OCP, U16 BQ76905RGRR, U17 ATtiny404-SS, U18 TPS25751SRSMR, U19 HD3SS3220IRNHT, U2 STM32F072CBT6, U20 TPD4EUSB30DQAR, U21 TPD4EUSB30DQAR, U22 AT24CS01-SSHM, U23 CH334R, U24 AT3H7B-CuH-S, U25 SY6280_OCP, U26 SY6280_OCP, U27 USBLC6-2SC6, U28 SY6280_OCP, U29 SY6280_OCP, U3 XC6206, U30 SY6280_OCP, U32 AT3H7B-CuH-S, U33 SY6280_OCP, U34 SY6280_OCP, U35 TLV70012_SOT23-5, U36 TUSB8041, U37 RAK4630, U38 TPS70933DBVR, U39 USBLC6-2SC6, U4 BQ25792RQMR, U5 RP2040, U6 USBLC6-2SC6, U7 CH334R, U8 PAM8406AB, U9 PCM2706CPJT, X1 X322512MSB4SI, X2 X322512MSB4SI, X3 X322512MSB4SI, X4 X322512MSB4SI, X5 X322512MSB4SI

Commit message: work on PCB
Parts:
- J7: footprint LibraryGlobalFootprints:AFC01-S05FCA-00_1x05_P0.5mm_FFC_Bottom_Contact -> LibraryGlobalFootprints:AFC07-S05ECA-00
- moved J7 4.26 mm to (174.9, 118.3)
Routing:
- net CHA_GND: track 43.2 -> 36.7 mm
Changed lines of the file:
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@@
 		(sheetname "/")
 		(sheetfile "cyberdeck-alpha.kicad_sch")
+		(units
+			(unit
+				(name "A")
+				(pins "1" "2")
+			)
+		)
 		(attr smd)
 		(duplicate_pad_numbers_are_jumpers no)
@@
 		(sheetname "/")
 		(sheetfile "cyberdeck-alpha.kicad_sch")
+		(units
+			(unit
+				(name "A")
+				(pins "1" "2")
+			)
+		)
 		(attr smd)
 		(duplicate_pad_numbers_are_jumpers no)
@@
 		)
 	)
-	(footprint "LibraryGlobalFootprints:AFC01-S05FCA-00_1x05_P0.5mm_FFC_Bottom_Contact"
+	(footprint "LibraryGlobalFootprints:AFC07-S05ECA-00"
 		(layer "B.Cu")
-		(at 170.6 118.325)
+		(at 174.86 118.34)
+		(descr "AFC07-S05ECA-00")
 		(property "Reference" "J7"
-			(at 0.11 -3.445 0)
+			(at -4.1 1.5 180)
 			(unlocked yes)
 			(layer "B.SilkS")
@@
 		)
 		(property "Value" "Conn_01x05"
-			(at 0.12 -12.38 180)
+			(at -4 -6.4 180)
 			(unlocked yes)
 			(layer "B.Fab")
@@
 			)
 		)
-		(property "LCSC" "C5213747"
+		(property "LCSC" "C262578"
 			(at 0 0 0)
 			(unlocked yes)
@@
 		(duplicate_pad_numbers_are_jumpers no)
 		(fp_rect
-			(start -3.75 0.7)
-			(end 3.75 -5.45)
+			(start -8 -0.5)
+			(end -0.5 -5.25)
 			(stroke
 				(width 0.1)
@@
 			(layer "B.SilkS")
 		)
-		(fp_circle
-			(center -3.4 0.35)
-			(end -3.35 0.4)
-			(stroke
-				(width 0.1)
-				(type solid)
-			)
-			(fill yes)
-			(layer "B.SilkS")
-		)
 		(fp_text user "${REFERENCE}"
-			(at 0.12 -13.88 180)
+			(at -4 -7.9 180)
 			(unlocked yes)
 			(layer "B.Fab")
@@
 			)
 		)
-		(pad "" smd rect
-			(at -2.7 -2.68)
-			(size 2 1.6)
-			(layers "B.Cu" "B.Mask" "B.Paste")
-		)
-		(pad "" smd rect
-			(at 2.7 -2.68)
-			(size 2 1.6)
-			(layers "B.Cu" "B.Mask" "B.Paste")
-		)
 		(pad "1" smd rect
-			(at -0.99 0)
-			(size 0.3 1.3)
+			(at -3.25 0)
+			(size 0.3 1.2)
 			(layers "B.Cu" "B.Mask" "B.Paste")
 			(net "+3.3V_MAIN")
@@
 		)
 		(pad "2" smd rect
-			(at -0.5 0)
-			(size 0.3 1.3)
+			(at -3.75 0)
+			(size 0.3 1.2)
 			(layers "B.Cu" "B.Mask" "B.Paste")
 			(net "/JOYSTICK_X")
@@
 		)
 		(pad "3" smd rect
-			(at 0 0)
-			(size 0.3 1.3)
+			(at -4.25 0)
+			(size 0.3 1.2)
 			(layers "B.Cu" "B.Mask" "B.Paste")
 			(net "/JOYSTICK_BTN")
@@
 		)
 		(pad "4" smd rect
-			(at 0.5 0)
-			(size 0.3 1.3)
+			(at -4.75 0)
+			(size 0.3 1.2)
 			(layers "B.Cu" "B.Mask" "B.Paste")
 			(net "GND")
@@
 		)
 		(pad "5" smd rect
-			(at 1 0)
-			(size 0.3 1.3)
+			(at -5.25 0)
+			(size 0.3 1.2)
 			(layers "B.Cu" "B.Mask" "B.Paste")
 			(net "/JOYSTICK_Y")
@@
 			(pintype "passive")
 		)
+		(pad "MP" smd rect
+			(at -6.85 -2.17)
+			(size 2.2 3.3)
+			(layers "B.Cu" "B.Mask" "B.Paste")
+		)
+		(pad "MP" smd rect
+			(at -1.65 -2.17)
+			(size 2.2 3.3)
+			(layers "B.Cu" "B.Mask" "B.Paste")
+		)
 		(embedded_fonts no)
-		(model "${TANGLES_MODEL_DIR}/FPC-5.stp"
+		(model "${TANGLES_MODEL_DIR}/AFC07-S05FCA-00.stp"
 			(offset
-				(xyz -1 0.3 0)
+				(xyz 4.5 -2.75 0)
 			)
 			(scale
@@
 			)
 			(rotate
-				(xyz -0 -0 -0)
+				(xyz -90 -0 -0)
 			)
 		)
@@
 	)
 	(segment
-		(start 158.7 120.96)
-		(end 159.436765 120.223235)
-		(width 0.6)
-		(layer "In2.Cu")
-		(net "CHA_GND")
-	)
-	(segment
-		(start 153.5625 120.25)
-		(end 155.73 120.25)
-		(width 0.6)
-		(layer "In2.Cu")
-		(net "CHA_GND")
-	)
-	(segment
-		(start 156.44 120.96)
-		(end 158.7 120.96)
-		(width 0.6)
-		(layer "In2.Cu")
-		(net "CHA_GND")
-	)
-	(segment
-		(start 155.73 120.25)
-		(end 156.44 120.96)
-		(width 0.6)
-		(layer "In2.Cu")
-		(net "CHA_GND")
-	)
-	(segment
 		(start 195.4675 66.2225)
 		(end 195.4675 66.7225)
@@
 		(net "/ETH_D3_P")
 	)
+	(via
+		(at 176.643223 84.823223)
+		(size 0.4)
+		(drill 0.2)
+		(layers "F.Cu" "B.Cu")
+		(net "/ETH_D3_P")
+	)
 	(segment
 		(start 202.235634 21.38677)
@@
 	)
 	(via
-		(at 176.643223 84.823223)
+		(at 191.52 40.55)
 		(size 0.4)
 		(drill 0.2)
 		(layers "F.Cu" "B.Cu")
-		(net "/ETH_D3_P")
+		(net "/ETH_D1_P")
 	)
 	(via
-		(at 191.52 40.55)
+		(at 177.453223 78.513223)
 		(size 0.4)
 		(drill 0.2)
@@
 	)
 	(via
-		(at 177.453223 78.513223)
+		(at 188.03 40.48)
 		(size 0.4)
 		(drill 0.2)
 		(layers "F.Cu" "B.Cu")
-		(net "/ETH_D1_P")
+		(net "/ETH_D3_N")
 	)
 	(via
-		(at 188.03 40.48)
+		(at 176.996777 85.176777)
 		(size 0.4)
 		(drill 0.2)
@@
 	)
 	(via
-		(at 176.996777 85.176777)
+		(at 192.02 40.55)
 		(size 0.4)
 		(drill 0.2)
 		(layers "F.Cu" "B.Cu")
-		(net "/ETH_D3_N")
+		(net "/ETH_D1_N")
 	)
 	(via
-		(at 192.02 40.55)
+		(at 177.806777 78.866777)
 		(size 0.4)
 		(drill 0.2)
@@
 	)
 	(via
-		(at 177.806777 78.866777)
+		(at 177.093223 82.346777)
 		(size 0.4)
 		(drill 0.2)
 		(layers "F.Cu" "B.Cu")
-		(net "/ETH_D1_N")
+		(net "/ETH_D2_N")
 	)
 	(via
@@
 	)
 	(via
-		(at 177.093223 82.346777)
+		(at 179.913223 76.136777)
 		(size 0.4)
 		(drill 0.2)
 		(layers "F.Cu" "B.Cu")
-		(net "/ETH_D2_N")
+		(net "/ETH_D0_N")
 	)
 	(via
@@
 	)
 	(via
-		(at 179.913223 76.136777)
+		(at 190.08 40.5)
 		(size 0.4)
 		(drill 0.2)
 		(layers "F.Cu" "B.Cu")
-		(net "/ETH_D0_N")
+		(net "/ETH_D2_P")
 	)
 	(via
-		(at 190.08 40.5)
+		(at 177.446777 81.993223)
 		(size 0.4)
 		(drill 0.2)
@@
 	)
 	(via
-		(at 177.446777 81.993223)
+		(at 180.45 75.783223)
 		(size 0.4)
 		(drill 0.2)
 		(layers "F.Cu" "B.Cu")
-		(net "/ETH_D2_P")
+		(net "/ETH_D0_P")
 	)
 	(via
@@
 		(net "/ETH_D0_P")
 	)
-	(via
-		(at 180.45 75.783223)
-		(size 0.4)
-		(drill 0.2)
-		(layers "F.Cu" "B.Cu")
-		(net "/ETH_D0_P")
-	)
