File: pcb-deck/cyberdeck-alpha.kicad_sch (KiCad schematic)
At the start: 523 parts, among them J1 CPU_FAN, J10 Conn_01x30, J11 Conn_01x22, J12 HDMI_C_1.3, J13 USB_C_Receptacle_USB2.0_16P, J14 Conn_01x06, J15 Conn_02x20_Odd_Even, J16 1-2199119-5, J17 2199119-3, J18 SIM_Card, J19 TSOP77438TR, J2 GP_LB, J20 Conn_01x22, J21 DX07S024JJ2R1300, J22 USB3_A, J3 GP_RB, J4 JOYSTICK, J5 Conn_01x06_Pin, J6 USB_C_Receptacle_USB2.0_16P, J7 Conn_01x05, J8 PJ-342B, J9 SPK, Q1 IRLML6244, Q2 CJ2101, Q3 SI4174DY-T1-GE3_N-Channel_FET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, Q4 BSS138, Q5 IRLML6244, Q6 SI4174DY-T1-GE3_N-Channel_FET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, Q7 SI4174DY-T1-GE3_N-Channel_FET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, Q8 SI4174DY-T1-GE3_N-Channel_FET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, U1 W25Q128JVS, U10 TPS62180YZFR, U11 TPS62180YZFR, U12 SY6280_OCP, U13 FAN5333ASX, U14 USBLC6-2SC6, U15 SY6280_OCP, U16 BQ76905RGRR, U17 ATtiny202-SS, U18 TPS25751SRSMR, U19 HD3SS3220IRNHT, U2 STM32F072CBT6, U20 TPD4EUSB30DQAR, U21 TPD4EUSB30DQAR, U22 AT24CS01-SSHM, U23 CH334R, U3 XC6206, U4 BQ25792RQMR, U5 RP2040, U6 USBLC6-2SC6, U7 CH334R, U8 PAM8406AB, U9 PCM2706CPJT, X1 X322512MSB4SI, X2 X322512MSB4SI, X3 X322512MSB4SI, X4 X322512MSB4SI

Commit message: add reference files for first revision
Parts:
- added D36: LED_0402, LED_SMD:LED_0402_1005Metric, symbol Device:LED
- added R98: 3.3K, Resistor_SMD:R_0402_1005Metric, symbol Device:R
Connections:
- net BQ_3V3: now also R98.2
- net GND: now also C20.1; no longer K_85.2, U17.8 (GND)
- net at U17.3 (PA7): now also D36.1 (K)
- net CELL- renamed BATT_GND
- net BATT_GND: now also K_85.2, U17.8 (GND)
- new net: D36.2 (A), R98.1
Other:
- moved on the sheet: BT1, BT2

Commit message: updates - need to clean up
Parts:
- removed D25: MBR0540, Diode_SMD:D_SOD-123, symbol Diode:MBR0540
- removed D26: MM3Z24VT1G, Diode_SMD:D_SOD-323, symbol Device:D
- removed F4: 500mA, Fuse:Fuse_0603_1608Metric, symbol Device:Fuse_Small
- removed J10: Conn_01x30, LibraryGlobalFootprints:AFC07-S30ECA-00, symbol Connector_Generic_MountingPin:Conn_01x30_MountingPin
- removed J14: Conn_01x06, LibraryGlobalFootprints:AFC07-S06ECA-00, symbol Connector_Generic_MountingPin:Conn_01x06_MountingPin
- removed JP13: SolderJumper_10_Open, LibraryGlobalFootprints:SolderJumper-10, symbol LibraryGlobalSymbols:SolderJumper_10_Open
- removed K_79: ZX-QC66-4.3TP, LibraryGlobalFootprints:ZX-QC66-7.5TP, symbol Switch:SW_Push
- removed L5: BRL3225T150K, Inductor_SMD:L_1210_3225Metric, symbol Device:L
- removed R24: 30R, Resistor_SMD:R_0402_1005Metric, symbol Device:R_Small
- removed R57: 10K, Resistor_SMD:R_0805_2012Metric, symbol Adafruit TFP401 to 40pin TFT-eagle-import:RESISTOR0805_NOOUTLINE
- removed R58: 3R, Resistor_SMD:R_0805_2012Metric, symbol Adafruit TFP401 to 40pin TFT-eagle-import:RESISTOR0805_NOOUTLINE
- removed R59, R60: 12R, Resistor_SMD:R_0805_2012Metric, symbol Adafruit TFP401 to 40pin TFT-eagle-import:RESISTOR0805_NOOUTLINE
- removed SJ1: HUB_D_P, LibraryGlobalFootprints:SOLDERJUMPER_ARROW_NOPASTE, symbol Adafruit TFP401 to 40pin TFT-eagle-import:SOLDERJUMPER
- removed SJ2: HUB_D_M, LibraryGlobalFootprints:SOLDERJUMPER_ARROW_NOPASTE, symbol Adafruit TFP401 to 40pin TFT-eagle-import:SOLDERJUMPER
- removed SJ3: +50mA, LibraryGlobalFootprints:SOLDERJUMPER_ARROW_NOPASTE, symbol Adafruit TFP401 to 40pin TFT-eagle-import:SOLDERJUMPER
- removed SJ4: +25mA, LibraryGlobalFootprints:SOLDERJUMPER_ARROW_NOPASTE, symbol Adafruit TFP401 to 40pin TFT-eagle-import:SOLDERJUMPER
- removed SJ5: BKLT_PWR, LibraryGlobalFootprints:SOLDERJUMPER_ARROW_NOPASTE, symbol Adafruit TFP401 to 40pin TFT-eagle-import:SOLDERJUMPER
- removed U13: FAN5333ASX, Package_TO_SOT_SMD:SOT-23-5, symbol Adafruit TFP401 to 40pin TFT-eagle-import:VREG_FAN5331
- removed U17: ATtiny202-SS, Package_SO:SOIC-8_3.9x4.9mm_P1.27mm, symbol MCU_Microchip_ATtiny:ATtiny202-SS
- added C127, C128, C129, C130: 100nF, Capacitor_SMD:C_0402_1005Metric, symbol Device:C_Small
- added D_70: MBR0540, Diode_SMD:D_SOD-123, symbol Device:D_Small
- added J10: DM3AT-SF-PEJM5, LibraryGlobalFootprints:HRS_DM3AT-SF-PEJM5 micro SD slot, symbol LibraryGlobalSymbols:DM3AT-SF-PEJM5
- added K_86: TS-1088-AR02016, LibraryGlobalFootprints:BTN_SMD_4x3mm, symbol Switch:SW_Push
- added K_87: PWR_BTN, LibraryGlobalFootprints:dome-tactile-pad, symbol Switch:SW_Push
- added R100, R101, R99: 4.7K, Resistor_SMD:R_0402_1005Metric, symbol Device:R
- added R102, R103, R24, R59: 10K, Resistor_SMD:R_0402_1005Metric, symbol Device:R
- added R104: 22R, Resistor_SMD:R_0402_1005Metric, symbol Device:R
- added R105, R106, R107: 140R, Resistor_SMD:R_0402_1005Metric, symbol Device:R
- added R57: 100R, Resistor_SMD:R_0402_1005Metric, symbol Device:R_Small
- added R58, R60: 6.8K, Resistor_SMD:R_0402_1005Metric, symbol Device:R
- added SJ16: CHG_SCL, LibraryGlobalFootprints:SOLDERJUMPER_ARROW_NOPASTE, symbol Adafruit TFP401 to 40pin TFT-eagle-import:SOLDERJUMPER
- added SJ17: CHG_SDA, LibraryGlobalFootprints:SOLDERJUMPER_ARROW_NOPASTE, symbol Adafruit TFP401 to 40pin TFT-eagle-import:SOLDERJUMPER
- added TP13, TP14, TP15, TP9: TestPoint_Small, TestPoint:TestPoint_Pad_2.0x2.0mm, symbol Connector:TestPoint_Small
- added U13: USBLC6-2SC6, Package_TO_SOT_SMD:SOT-23-6, symbol Power_Protection:USBLC6-2SC6
- added U17: ATtiny404-SS, Package_SO:SOIC-14_3.9x8.7mm_P1.27mm, symbol MCU_Microchip_ATtiny:ATtiny404-SS
- added U24, U27: PC817, LibraryGlobalFootprints:PC817X3CSP9F, symbol Isolator:PC817
- added U25, U26, U28: SY6280_OCP, Package_TO_SOT_SMD:SOT-23-5, symbol LibraryGlobalSymbols:SY6280_Overcurrent_Protection_Diode
- BT1, BT2: value Battery_Cell -> LiCell
- C68: value 10uF -> 100nF; footprint Capacitor_SMD:C_0805_2012Metric -> Capacitor_SMD:C_0402_1005Metric; LCSC C15850 -> C1525
- C69: value 1uF -> 22uF; LCSC C28323 -> C6119899
- C70: value 1uF -> 100nF; footprint Capacitor_SMD:C_0805_2012Metric -> Capacitor_SMD:C_0402_1005Metric; LCSC C28323 -> C1525
- C71: value 100nF -> 22uF; LCSC C28233 -> C6119899
- J11: LCSC C262642 -> C262566
- J15: value Conn_02x20_Odd_Even -> PZ254-2-20-W-8.5
- JP1, JP2: symbol Jumper:SolderJumper_3_Open -> Jumper:SolderJumper_3_Bridged12
- K_69, K_70, K_71, K_72, K_75, K_76, K_77, K_78: symbol Library:Keyboard_Key_Array_Config -> Switch:SW_Push; now in the parts list
- R63: value 6.8K -> 3.4K; LCSC C25917 -> C4940
- R66: value 1K -> 4.7K; LCSC C11702 -> C25900
Connections:
- net BQ_3V3 is gone; now on net BQ_REGOUT_3V3: Q2.1 (G), R98.2, U16.15 (REGOUT)
- net DISP_LEDN is gone; now on net +3.3V_MAIN: C71.1
- net MIPI1_CLK_A_N is gone; now on net MIPI1_CLK_N: J11.15 (Pin_15)
- net MIPI1_CLK_A_P is gone; now on net MIPI1_CLK_P: J11.14 (Pin_14)
- net MIPI1_D0_A_N is gone; now on net MIPI1_D0_N: J11.21 (Pin_21)
- net MIPI1_D0_A_P is gone; now on net MIPI1_D0_P: J11.20 (Pin_20)
- net MIPI1_D1_A_N is gone; now on net MIPI1_D1_N: J11.18 (Pin_18)
- net MIPI1_D1_A_P is gone; now on net MIPI1_D1_P: J11.17 (Pin_17)
- net MIPI1_D2_A_N is gone; now on net MIPI1_D2_N: J11.12 (Pin_12)
- net MIPI1_D2_A_P is gone; now on net MIPI1_D2_P: J11.11 (Pin_11)
- net MIPI1_D3_A_N is gone; now on net MIPI1_D3_N: J11.9 (Pin_9)
- net MIPI1_D3_A_P is gone; now on net MIPI1_D3_P: J11.8 (Pin_8)
- net USB2_SYS_N is gone; now on net USB2_D_N: JP2.3 (B), U14.6 (I/O1), U18.23 (GPIO5/USB_N/MD2)
- net USB2_SYS_P is gone; now on net USB2_D_P: JP1.3 (B), U14.4 (I/O2), U18.22 (GPIO5/USB_P/MD1)
- net +3.3V_MAIN: now also C70.1, C129.2, R102.1, U28.5 (IN)
- net +5V_CM5: now also C68.1, C69.1, J1.1 (Pin_1); no longer J1.4 (Pin_4)
- net +5V_MAIN: now also C127.2, C128.2, R24.2, R59.2, U25.5 (IN), U26.5 (IN)
- net +5V_PORT: no longer D_69.2 (A), R40.2, R41.2
- net +VSYS: now also SJ10.2
- net 3V3_MAIN: no longer R52.2
- net 5V_MAIN: no longer R49.2, SJ10.2
- net BATT_GND: now also D31.2 (A), R101.1, TP9.1, U17.14 (GND); no longer D33.2 (A)
- net BQ_CELL1: now also K_86.2, U24.4
- net BQ_SCL: now also R100.1, TP15.1, U17.9 (PB0)
- net BQ_SDA: now also R66.1, TP14.1, U17.8 (PB1)
- net CHG_SCL: now also SJ16.2; no longer U18.16 (I2Cc_SCL)
- net CHG_SDA: now also SJ17.2; no longer U18.15 (I2Cc_SDA)
- net CM5_PWR_BTN: no longer R66.1
- net FAN_PWM: now also J1.2 (Pin_2); no longer J1.3 (Pin_3)
- net FAN_TACHO: now also J1.4 (Pin_4); no longer J1.1 (Pin_1)
- net GND: now also C68.2, J1.3 (Pin_3), J22.10 (SHIELD), J22.4 (GND), J22.7 (DRAIN), K_69.1, K_70.1, K_71.1, K_72.1, K_75.1, K_76.1, K_77.1, K_78.1, C127.1, C128.1, C129.1, C130.2, J10.6 (VSS), R103.2, R105.1, R106.1, R107.1, R58.1, R60.1, U13.2 (GND), U24.2, U25.2 (GND), U26.2 (GND), U28.2 (GND); no longer C68.1, D27.3 (PAD), D28.3 (PAD), D29.3 (PAD), J1.2 (Pin_2), K_69.2 (ROW), K_70.2 (ROW), K_71.2 (ROW), K_72.2 (ROW), K_75.2 (ROW), K_76.2 (ROW), K_77.2 (ROW), K_78.2 (ROW)
- net GND_OUT: now also D33.2 (A); no longer D31.2 (A)
- net GP_BTN_A: now also K_69.2; no longer K_69.1 (COL)
- net GP_BTN_B: now also K_70.2; no longer K_70.1 (COL)
- net GP_BTN_DN: now also K_76.2; no longer K_76.1 (COL)
- net GP_BTN_L: now also K_77.2; no longer K_77.1 (COL)
- net GP_BTN_R: now also K_78.2; no longer K_78.1 (COL)
- net GP_BTN_UP: now also K_75.2; no longer K_75.1 (COL)
- net GP_BTN_X: now also K_71.2; no longer K_71.1 (COL)
- net GP_BTN_Y: now also K_72.2; no longer K_72.1 (COL)
- net HUB2_DS_1_D+: now also U13.4 (I/O2)
- net HUB2_DS_1_D-: now also U13.6 (I/O1)
- net HUB_US_D+: now also JP1.2 (C); no longer JP1.1 (A)
- net HUB_US_D-: now also JP2.2 (C); no longer JP2.1 (A)
- net MIPI1_SCL: now also J15.28 (Pin_28), Module2.35 (ID_SC); no longer Module2.80 (SCL0)
- net MIPI1_SDA: now also J15.27 (Pin_27), Module2.36 (ID_SD); no longer Module2.82 (SDA0)
- net SHIP_MODE: now also U17.13 (PA3)
- net TINY202_UPDI: now also R99.2
- net USB3_0_D_N: now also JP2.1 (A)
- net USB3_0_D_P: now also JP1.1 (A)
- net at R43.2, U9.23 (D+): no longer R45.2
- net at D36.1 (K): now also U17.3 (PA5)
- net at Q6.4 (G), R86.1, R87.2: now also D33.1 (K); no longer D31.1 (K)
- net at D23.2 (A): now also R57.2
- net BQ_REGOUT_3V3: now reaches R66.2
- net BQ_REGOUT_3V3: now also R100.2, TP13.1, U17.1 (VCC)
- net RP2040_GPIO_0: now reaches U5.2 (GPIO0)
- net RP2040_GPIO_17: now reaches U5.28 (GPIO17)
- net RP2040_GPIO_1: now reaches U5.3 (GPIO1)
- net RP2040_GPIO_23: now reaches U5.35 (GPIO23)
- net RP2040_GPIO_24: now reaches U5.36 (GPIO24)
- net RP2040_LED_BUILTIN: now reaches U5.37 (GPIO25)
- net RP2040_LED_BUILTIN: now also R57.1
- net RP2040_GPIO_2: now reaches U5.4 (GPIO2)
- net RP2040_GPIO_28_ADC2: now reaches U5.40 (GPIO28_ADC2)
- net RP2040_GPIO_29_ADC3: now reaches U5.41 (GPIO29_ADC3)
- net RP2040_GPIO_3: now reaches U5.5 (GPIO3)
- net at J13.A6 (D+), J13.B6 (D+): now also U14.3 (I/O2); no longer U14.1 (I/O1)
- net at J13.A7 (D-), J13.B7 (D-): now also U14.1 (I/O1); no longer U14.3 (I/O2)
- net at J22.1 (VBUS): now also D_70.1 (K)
- net at J22.2 (D-): now also U13.1 (I/O1)
- net at J22.3 (D+): now also U13.3 (I/O2)
- net IRQt: now reaches TP6.1, U18.10 (I2Ct_IRQ)
- net SHIP_MODE_WAKE: now reaches R64.1, R95.1
- net SHIP_MODE_WAKE: now also K_86.1, U24.3; no longer SJ14.2
- net at Module2.57 (SD_CLK): now also R104.2
- net SD_DAT3: now reaches Module2.61 (SD_DAT3)
- net SD_DAT3: now also J10.2 (CD/DAT3)
- net SD_CMD: now reaches Module2.62 (SD_CMD)
- net SD_CMD: now also J10.3 (CMD)
- net SD_DAT0: now reaches Module2.63 (SD_DAT0)
- net SD_DAT0: now also J10.7 (DAT0)
- net SD_DAT1: now reaches Module2.67 (SD_DAT1)
- net SD_DAT1: now also J10.8 (DAT1)
- net SD_DAT2: now reaches Module2.69 (SD_DAT2)
- net SD_DAT2: now also J10.1 (DAT2)
- net SD_PWR_EN: now reaches Module2.75 (SD_PWR_ON)
- net SD_PWR_EN: now also R102.2, U28.4 (~{EN})
- net at Q2.2 (S), R64.2: now also D31.1 (K); no longer D33.1 (K)
- net SDAt: now reaches TP7.1, U18.8 (I2Ct_SDA)
- net SCLt: now reaches TP8.1, U18.9 (I2Ct_SCL)
- net 3V3_SHIP_MODE_OFF renamed TPS_LDO_3V3
- net TPS_LDO_3V3: now also SJ14.2; no longer SJ14.1
- net CM5_USB_D_N renamed USB2_D_N
- net USB2_D_N: no longer JP2.2 (C)
- net CM5_USB_D_P renamed USB2_D_P
- net USB2_D_P: no longer JP1.2 (C)
- net DISP_INT: no longer names the net of U5.30 (GPIO19)
- removed net DISP_LEDP: C69.1, C70.1
- net DISP_RST renamed RP2040_GPIO_18
- net DISP_SCL renamed RP2040_GPIO_5_SDL
- net DISP_SDA renamed RP2040_GPIO_4_SDA
- net ID_SCL_GPIO_1 renamed MIPI0_SCL
- net MIPI0_SCL: now also Module2.80 (SCL0); no longer J15.28 (Pin_28), Module2.35 (ID_SC)
- net ID_SDA_GPIO_0 renamed MIPI0_SDA
- net MIPI0_SDA: now also Module2.82 (SDA0); no longer J15.27 (Pin_27), Module2.36 (ID_SD)
- new net: R103.1, U28.3 (~{RSET})
- new net: R58.2, U25.3 (~{RSET})
- new net: R24.1, U25.4 (~{EN})
- new net: D29.3 (PAD), R106.2
- new net: R60.2, U26.3 (~{RSET})
- new net: R59.1, U26.4 (~{EN})
- new net: D28.3 (PAD), R105.2
- new net: K_87.2, R101.2
- new net: D27.3 (PAD), R107.2
- new net: R99.1, U17.10 (~{RESET}/PA0)
- new net: J10.P1 (SHIELD), J10.P2 (SHIELD), J10.P3 (SHIELD), J10.P4 (SHIELD)
- new net +3V3_MICRO_SD: C130.1, J10.4 (VDD), U28.1 (OUT)
- new net +5V_PORT_A: D_70.2 (A), U13.5 (VBUS), U26.1 (OUT)
- new net +5V_PORT_C: D_69.2 (A), R40.2, R41.2, U25.1 (OUT)
- new net PWR_BTN: K_87.1, U17.7 (PB2)
- new net SCLc: SJ16.1, U18.16 (I2Cc_SCL)
- new net SDAc: SJ17.1, U18.15 (I2Cc_SDA)
- new net SD_CLK: R104.1
- new net SYS_SHIP_WAKE: SJ14.1, U24.1
- no-connect marks 115 -> 110
Other:
- note added: "BATT_GND Domain"
- note added: "MICRO SD"
- note added: "PD PSU EEPROM"
- note added: "Power BTN / LED"
- note added: "USB-A 2.0 Port"
- note added: "USB-C 2.0 Port"
- note removed: "BACKLIGHT PWR"
- note removed: "Device Power Btn"
- note removed: "ESD Protection"
- note removed: "External Connections"
- note removed: "USB A Port"
- note removed: "USB Port"
- note removed: "VBUS Fuses"
- moved on the sheet: BT1, BT2, C10, C100, C101, C102, C103, C104, C105, C106, C107, C108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

Commit message: pcb updates
Parts:
- removed J9: SPK, LibraryGlobalFootprints:1x04_P2.54 SMD pads only, symbol Connector:Conn_01x04_Pin
- removed K_80: ZX-QC66-4.3TP, LibraryGlobalFootprints:ZX-QC66-7.5TP, symbol Switch:SW_Push
- removed Q4: BSS138, Package_TO_SOT_SMD:SOT-23, symbol Adafruit TFP401 to 40pin TFT-eagle-import:MOSFET-NREFLOW
- removed U27: PC817, LibraryGlobalFootprints:PC817X3CSP9F, symbol Isolator:PC817
- added C131, C132, C134, C136: 100nF, Capacitor_SMD:C_0402_1005Metric, symbol Device:C_Small
- added C133: 1nF-2kV, Capacitor_SMD:C_1206_3216Metric, symbol Device:C_Small
- added C135: 10nF, Capacitor_SMD:C_0402_1005Metric, symbol Device:C_Small
- added D25, D26, D37: LED_0402, LED_SMD:LED_0402_1005Metric, symbol Device:LED
- added H4: SMTWE2030MTJ, LibraryGlobalFootprints:M.2 M2 nut standoff, symbol Mechanical:MountingHole_Pad
- added J14: USB_C_Receptacle_USB2.0_16P, LibraryGlobalFootprints:USB_C_Receptacle_HRO_TYPE-C-31-M-12, symbol Connector:USB_C_Receptacle_USB2.0_16P
- added J9: RJ45_LED_Shielded, LibraryGlobalFootprints:RC01812, symbol Connector:RJ45_LED_Shielded
- added K_79: GP_MODE, LibraryGlobalFootprints:dome-tactile-pad, symbol Switch:SW_Push
- added R108: 100K, Resistor_SMD:R_0402_1005Metric, symbol Device:R
- added R109, R111: 3.4K, Resistor_SMD:R_0402_1005Metric, symbol Device:R
- added R110: 470R, Resistor_SMD:R_0402_1005Metric, symbol Device:R
- added R112, R113, R114, R115: 75R, Resistor_SMD:R_0603_1608Metric, symbol Device:R
- added R116, R117: 100R, Resistor_SMD:R_0402_1005Metric, symbol Device:R_Small
- added SJ1: PCIE_PWR, LibraryGlobalFootprints:SOLDERJUMPER_ARROW_NOPASTE, symbol Adafruit TFP401 to 40pin TFT-eagle-import:SOLDERJUMPER
- added U27: USBLC6-2SC6, Package_TO_SOT_SMD:SOT-23-6, symbol Power_Protection:USBLC6-2SC6
- added U29, U30: SY6280_OCP, Package_TO_SOT_SMD:SOT-23-5, symbol LibraryGlobalSymbols:SY6280_Overcurrent_Protection_Diode
- added U31: ~, LibraryGlobalFootprints:G24P02S, symbol LibraryGlobalSymbols:G24P02S
- added U32: AT3H7B-CuH-S, Package_SO:SSOP-4_4.4x2.6mm_P1.27mm, symbol Isolator:PC817
- C78, C80, C81, C82, D24, J18, R76, R77, R78, R79, R80: now fitted; now in the parts list
- H3: value SMTWE2040MTJ -> SMTWE2025MTJ; LCSC C2928181 -> C2928178; now fitted; now in the parts list
- J17: value 2199119-3 -> 2199230-3; footprint LibraryGlobalFootprints:2199119-3 M.2 B key -> LibraryGlobalFootprints:2199230-3 M.2 B key; now fitted; now in the parts list
- K_73: value ZX-QC66-4.3TP -> GP_START; footprint LibraryGlobalFootprints:ZX-QC66-7.5TP -> LibraryGlobalFootprints:dome-tactile-pad; Description_1 GP_STA -> (none); LCSC C7470157 -> (none)
- K_74: value ZX-QC66-4.3TP -> GP_SELECT; footprint LibraryGlobalFootprints:ZX-QC66-7.5TP -> LibraryGlobalFootprints:dome-tactile-pad; Description_1 GP_SEL -> (none); LCSC C7470157 -> (none)
- R81: value 5.1K -> 3.3K; LCSC C25905 -> C25890; now fitted; now in the parts list
- R82: value 10K -> 470R; LCSC C25744 -> C25117; now fitted; now in the parts list
- R87: footprint Capacitor_SMD:C_0603_1608Metric -> Resistor_SMD:R_0603_1608Metric
- U24: value PC817 -> AT3H7B-CuH-S; footprint LibraryGlobalFootprints:PC817X3CSP9F -> Package_SO:SSOP-4_4.4x2.6mm_P1.27mm; LCSC C3025164 -> C20612660
Connections:
- net +5V_PORT is gone; now on net +5V_PORT_C: U6.5 (VBUS)
- net +3.3V_MAIN: now also J7.1 (Pin_1), C131.2, C132.2, SJ1.1, U29.5 (IN), U30.5 (IN); no longer C70.1, C71.1, J16.12 (3.3V), J16.14 (3.3V), J16.16 (3.3V), J16.18 (3.3V), J16.2 (3.3V), J16.4 (3.3V), J16.70 (3.3V), J16.72 (3.3V), J16.74 (3.3V), J17.2 (3.3V), J17.4 (3.3V), J17.70 (3.3V), J17.72 (3.3V), J17.74 (3.3V), J7.5 (Pin_5), R82.2
- net +VBUS: now also J14.A4 (VBUS), J14.A9 (VBUS), J14.B4 (VBUS), J14.B9 (VBUS), U27.5 (VBUS); no longer J13.A4 (VBUS), J13.A9 (VBUS), J13.B4 (VBUS), J13.B9 (VBUS), U14.5 (VBUS)
- net BATT_GND: now also U32.2
- net CM5_3V3: now also J9.10, J9.12
- net CM5_CC1: now also J13.A5 (CC1)
- net CM5_CC2: now also J13.B5 (CC2)
- net CM5_PWR_BTN: now also U32.4
- net GND: now also J10.P1 (SHIELD), J7.4 (Pin_4), C131.1, C132.1, C134.1, C135.1, C136.1, H4.1, J14.A1 (GND), J14.A12 (GND), J14.B1 (GND), J14.B12 (GND), J14.S1 (SHIELD), K_79.1, R108.1, R109.1, R111.1, R116.1, R117.1, U27.2 (GND), U29.2 (GND), U30.2 (GND), U32.3; no longer J7.2 (Pin_2), R81.1
- net GPIO_6: no longer R81.2
- net GP_BTN_MODE: now also K_79.2
- net HUB2_DS_1_D+: no longer U13.4 (I/O2)
- net HUB2_DS_1_D-: no longer U13.6 (I/O1)
- net JOYSTICK_X: now also J7.2 (Pin_2), U5.39 (GPIO27_ADC1); no longer J7.4 (Pin_4), U5.38 (GPIO26_ADC0)
- net JOYSTICK_Y: now also J7.5 (Pin_5), U5.38 (GPIO26_ADC0); no longer J7.1 (Pin_1), U5.39 (GPIO27_ADC1)
- net M2B_LED: now also D25.1 (K)
- net PD_CC1: now also J14.A5 (CC1); no longer J13.A5 (CC1)
- net PD_CC2: now also J14.B5 (CC2); no longer J13.B5 (CC2)
- net SD_CLK: now also J10.5 (CLK)
- net USB2_D_N: no longer U18.23 (GPIO5/USB_N/MD2)
- net USB2_D_P: no longer U18.22 (GPIO5/USB_P/MD1)
- net at R43.2, U9.23 (D+): now also R45.2
- net ETH_D0_N: now reaches Module2.10 (Ethernet_Pair0_N)
- net ETH_D0_N: now also U31.3 (D1-)
- net ETH_D2_P: now reaches Module2.11 (Ethernet_Pair2_P)
- net ETH_D2_P: now also U31.8 (D3+)
- net ETH_D0_P: now reaches Module2.12 (Ethernet_Pair0_P)
- net ETH_D0_P: now also U31.2 (D1+)
- net ETH_LED_G: now reaches Module2.15 (Ethernet_nLED3(3.3v))
- net ETH_LED_G: now also R110.2
- net ETH_LED_Y: now reaches Module2.17 (Ethernet_nLED2(3.3v))
- net ETH_LED_Y: now also R82.2
- net IEEE1588_SYNC_OUT_3V3: now reaches Module2.18 (Ethernet_SYNC_OUT(3.3v))
- net CM5_ACT_LED: now reaches Module2.21 (LED_nACT)
- net CM5_ACT_LED: now also D26.1 (K)
- net ETH_D3_P: now reaches Module2.3 (Ethernet_Pair3_P)
- net ETH_D3_P: now also U31.11 (D4+)
- net ETH_D1_P: now reaches Module2.4 (Ethernet_Pair1_P)
- net ETH_D1_P: now also U31.5 (D2+)
- net ETH_D3_N: now reaches Module2.5 (Ethernet_Pair3_N)
- net ETH_D3_N: now also U31.12 (D4-)
- net ETH_D1_N: now reaches Module2.6 (Ethernet_Pair1_N)
- net ETH_D1_N: now also U31.6 (D2-)
- net ETH_D2_N: now reaches Module2.9 (Ethernet_Pair2_N)
- net ETH_D2_N: now also U31.9 (D3-)
- net CM5_PWR_LED: now reaches Module2.95 (LED_nPWR)
- net CM5_PWR_LED: now also D37.1 (K)
- net M2B_POWER: no longer names the net of R82.1
- net M2B_POWER: now also J9.11; no longer J17.6 (~{FULL_CARD_POWER_OFF})
- net PCIE-PWR_EN renamed M2B_POWER_OFF
- net M2B_POWER_OFF: now also J17.6 (~{FULL_CARD_POWER_OFF}), R108.2, SJ1.2, U29.4 (~{EN}), U30.4 (~{EN})
- new net: R111.2, U30.3 (~{RSET})
- new net: C133.1, R112.1, R113.1, R114.1, R115.1
- new net: R112.2, U31.24 (CX1)
- new net: D25.2 (A), R81.1
- new net: R114.2, U31.18 (CX3)
- new net: R113.2, U31.21 (CX2)
- new net: R109.2, U29.3 (~{RSET})
- new net: D37.2 (A), R117.2
- new net: D26.2 (A), R116.2
- new net: C135.2, U31.1 (CD1), U31.10 (CD4), U31.4 (CD2), U31.7 (CD3)
- new net: R115.2, U31.15 (CX4)
- new net: J9.9, R110.1
- new net: J13.A4 (VBUS), J13.A9 (VBUS), J13.B4 (VBUS), J13.B9 (VBUS), U14.5 (VBUS)
- new net: J14.A6 (D+), J14.B6 (D+), U27.3 (I/O2)
- new net: J14.A7 (D-), J14.B7 (D-), U27.1 (I/O1)
- new net +3.3V_M2B: J17.2 (3.3V), J17.4 (3.3V), J17.70 (3.3V), J17.72 (3.3V), J17.74 (3.3V), R81.2, U29.1 (OUT)
- new net +3.3V_M2PCIE: C70.1, C71.1, J16.12 (3.3V), J16.14 (3.3V), J16.16 (3.3V), J16.18 (3.3V), J16.2 (3.3V), J16.4 (3.3V), J16.70 (3.3V), J16.72 (3.3V), J16.74 (3.3V), U30.1 (OUT)
- new net CHA_GND: C133.2, C134.2, C136.2, J9.SH
- new net CHG_USBD_N: U18.23 (GPIO5/USB_N/MD2), U27.6 (I/O1)
- new net CHG_USBD_P: U18.22 (GPIO5/USB_P/MD1), U27.4 (I/O2)
- new net ETH_BL2_N: J9.5, U31.16 (X3-)
- new net ETH_BL2_P: J9.4, U31.17 (X3+)
- new net ETH_BL3_N: J9.8, U31.13 (X4-)
- new net ETH_BL3_P: J9.7, U31.14 (X4+)
- new net ETH_RX1_N: J9.6, U31.19 (X2-)
- new net ETH_RX1_P: J9.3, U31.20 (X2+)
- new net ETH_TX0_N: J9.2, U31.22 (X1-)
- new net ETH_TX0_P: J9.1, U31.23 (X1+)
- new net PORT_USBA2_D+: U13.4 (I/O2)
- new net PORT_USBA2_D-: U13.6 (I/O1)
- no-connect marks 110 -> 114
Other:
- note added: "CM5 LEDs"
- note added: "ETHERNET"
- note added: "Power LED"
- note added: "USB-C CM5 System Port"
- note added: "USB-C PD Charge Port"
- note removed: "Power BTN / LED"
- note removed: "USB-C PD Charge / CM5 System Port"
- moved on the sheet: C127, C129, C130, C40, C41, C42, C43, C44, C45, C66, C67, D23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

Commit message: add firmwares
Parts:
- added C137, C138: 100nF, Capacitor_SMD:C_0402_1005Metric, symbol Device:C_Small
- added J23, J24: Conn_01x06_Pin, LibraryGlobalFootprints:1x04_P2.54 SMD pads only, symbol Connector_Generic:Conn_01x04
- added R118, R120: 10K, Resistor_SMD:R_0402_1005Metric, symbol Device:R
- added R119, R121: 6.8K, Resistor_SMD:R_0402_1005Metric, symbol Device:R
- added TP16: TestPoint_Small, TestPoint:TestPoint_Pad_2.0x2.0mm, symbol Connector:TestPoint_Small
- added U33, U34: SY6280_OCP, Package_TO_SOT_SMD:SOT-23-5, symbol LibraryGlobalSymbols:SY6280_Overcurrent_Protection_Diode
- U24, U32: footprint Package_SO:SSOP-4_4.4x2.6mm_P1.27mm -> LibraryGlobalFootprints:SSOP-4_AT3H7B-CuH-S
Connections:
- net +5V_MAIN: now also C137.2, C138.2, R118.2, R120.2, U33.5 (IN), U34.5 (IN)
- net +5V_PORT_C: now also U33.1 (OUT)
- net BATT_GND: now also K_87.2; no longer R101.1
- net BQ_REGSRC: now also TP16.1
- net GND: now also C137.1, C138.1, J23.1 (Pin_1), J24.1 (Pin_1), R119.1, R121.1, U33.2 (GND), U34.2 (GND)
- net HUB2_DS_2_D+: now also J23.3 (Pin_3)
- net HUB2_DS_2_D-: now also J23.2 (Pin_2)
- net HUB2_DS_3_D+: now also J24.2 (Pin_2)
- net HUB2_DS_3_D-: now also J24.3 (Pin_3)
- net at R101.2: no longer K_87.2
- net SOFT_PWR_OUT: now reaches U17.6 (PB3)
- net SOFT_PWR_OUT: now also U32.1
- new net: R120.1, U34.4 (~{EN})
- new net: R121.2, U34.3 (~{RSET})
- new net: R119.2, U33.3 (~{RSET})
- new net: R118.1, U33.4 (~{EN})
- new net +5V_INT_USB: J23.4 (Pin_4), J24.4 (Pin_4), U34.1 (OUT)
Other:
- moved on the sheet: F3, R101

Commit message: add  \sketch for esp32 diagnostic / flashing jig, add tiny1604 BQ controller sketch
Parts:
- removed K_85: TS-1088-AR02016, LibraryGlobalFootprints:BTN_SMD_4x3mm, symbol Switch:SW_Push
- removed NT1, NT2, NT3, NT6, NT7: NetTie_2, NetTie:NetTie-2_SMD_Pad0.5mm, symbol Device:NetTie_2
- removed SJ10: 3V_IN, LibraryGlobalFootprints:SOLDERJUMPER_ARROW_NOPASTE, symbol Adafruit TFP401 to 40pin TFT-eagle-import:SOLDERJUMPER
- added F2: 500mA, Fuse:Fuse_0603_1608Metric, symbol Device:Fuse_Small
- added R122: 430R, Resistor_SMD:R_0402_1005Metric, symbol Device:R
- added R123: 470K, Resistor_SMD:R_0402_1005Metric, symbol Device:R
- added R124: 4.7K, Resistor_SMD:R_0402_1005Metric, symbol Device:R
- R101: value 4.7K -> 430R; LCSC C25900 -> C36356
- R66: value 4.7K -> 10K; LCSC C25900 -> C25744
- SJ11: value 5V_IN -> VSYS_IN
Connections:
- net CELL+ is gone; now on net +VBATT: BT1.1 (+), C92.1, TP1.1
- net CHG_SDA is gone; now on net CHG_SCL: SJ17.2, TP11.1, U22.5 (SDA), U4.15 (SDA)
- net GND_OUT is gone; now on net GND: C90.1, C91.2, D33.2 (A), Q6.1 (S), Q6.2 (S), Q6.3 (S), R87.1
- net +3.3V_MAIN: now also F2.2; no longer C123.1, U18.32 (VIN_3V3), U22.8 (VCC)
- net +VBATT: now also D30.2 (A), R89.2
- net +VSYS: now also SJ11.1; no longer SJ11.2
- net BATT_GND: now also C86.1, C87.1, R91.2, R123.1; no longer R95.2, U32.2
- net BQ_REGOUT_3V3: now also R66.1, R95.1, U32.1; no longer R100.2, R66.2
- net BQ_SCL: now also R66.2; no longer R100.1
- net BQ_SDA: now also R95.2; no longer R66.1
- net CHG_SCL: now also R100.1, R124.1
- net GND: now also R122.1; no longer U24.2
- net SOFT_PWR_OUT: now also R101.2; no longer U32.1
- net BQ_ALERT: now reaches U16.14 (ALERT)
- net BQ_ALERT: now also U17.5 (PA7)
- net at R101.1: now also U32.2
- net 3V3_IN renamed VSYS_IN
- net VSYS_IN: now also C54.2, C55.2, SJ11.2, SJ9.2, U10.A1 (VIN1), U10.B1 (VIN1), U10.C1 (VIN1), U10.D1 (VIN2), U10.E1 (VIN2), U10.F1 (VIN2)
- removed net 5V_IN: C54.2, C55.2, SJ11.1, SJ9.2, U10.A1 (VIN1), U10.B1 (VIN1), U10.C1 (VIN1), U10.D1 (VIN2), U10.E1 (VIN2), U10.F1 (VIN2)
- net SHIP_MODE renamed SHIP_MODE_WAKE_BTN
- net SHIP_MODE_WAKE_BTN: now also K_86.1, R64.1, U24.3, R123.2
- removed net SHIP_MODE_WAKE: K_86.1, R64.1, R95.1, U24.3
- net SYS_SHIP_WAKE renamed SHIP_WAKE_3V3
- new net: R122.2, U24.2
- new net PD_3V3: C123.1, F2.1, R100.2, R124.2, U18.32 (VIN_3V3), U22.8 (VCC)
- no-connect marks 114 -> 113
Other:
- moved on the sheet: C100, C101, C102, C103, C106, C107, C108, C109, C110, C111, C112, C113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
