File: pcb-deck/cyberdeck-alpha.kicad_sch (KiCad schematic)
At the start: 573 parts, among them J1 CPU_FAN, J10 DM3AT-SF-PEJM5, J11 Conn_01x22, J12 HDMI_C_1.3, J13 USB_C_Receptacle_USB2.0_16P, J14 USB_C_Receptacle_USB2.0_16P, J15 PZ254-2-20-W-8.5, J16 1-2199119-5, J17 2199230-3, J18 SIM_Card, J19 TSOP77438TR, J2 GP_LB, J20 Conn_01x22, J21 DX07S024JJ2R1300, J22 USB3_A, J23 Conn_01x06_Pin, J24 Conn_01x06_Pin, J3 GP_RB, J4 JOYSTICK, J5 Conn_01x06_Pin, J6 USB_C_Receptacle_USB2.0_16P, J7 Conn_01x05, J8 PJ-342B, J9 RJ45_LED_Shielded, Q1 IRLML6244, Q2 CJ2101, Q3 SI4174DY-T1-GE3_N-Channel_FET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, Q5 IRLML6244, Q6 SI4174DY-T1-GE3_N-Channel_FET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, Q7 SI4174DY-T1-GE3_N-Channel_FET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, Q8 SI4174DY-T1-GE3_N-Channel_FET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, U1 W25Q128JVS, U10 TPS62180YZFR, U11 TPS62180YZFR, U12 SY6280_OCP, U13 USBLC6-2SC6, U14 USBLC6-2SC6, U15 SY6280_OCP, U16 BQ76905RGRR, U17 ATtiny404-SS, U18 TPS25751SRSMR, U19 HD3SS3220IRNHT, U2 STM32F072CBT6, U20 TPD4EUSB30DQAR, U21 TPD4EUSB30DQAR, U22 AT24CS01-SSHM, U23 CH334R, U24 AT3H7B-CuH-S, U25 SY6280_OCP, U26 SY6280_OCP, U27 USBLC6-2SC6, U28 SY6280_OCP, U29 SY6280_OCP, U3 XC6206, U30 SY6280_OCP, U32 AT3H7B-CuH-S, U33 SY6280_OCP, U34 SY6280_OCP, U4 BQ25792RQMR, U5 RP2040, U6 USBLC6-2SC6, U7 CH334R, U8 PAM8406AB, U9 PCM2706CPJT, X1 X322512MSB4SI, X2 X322512MSB4SI, X3 X322512MSB4SI, X4 X322512MSB4SI

Commit message: controller updates
Parts:
- removed TP9: TestPoint_Small, TestPoint:TestPoint_Pad_2.0x2.0mm, symbol Connector:TestPoint_Small
- added C139, C140, C141, C142, C143, C145, C146, C147, C148, C149, C150, C151, C152: 100nF, Capacitor_SMD:C_0402_1005Metric, symbol Device:C_Small
- added C144, C153: 10uF, Capacitor_SMD:C_0603_1608Metric, symbol Device:C_Small
- added C154, C155: 20pF, Capacitor_SMD:C_0402_1005Metric, symbol Device:C
- added F4, F5: 500mA, Fuse:Fuse_0603_1608Metric, symbol Device:Fuse_Small
- added K_80: TS-1088-AR02016, LibraryGlobalFootprints:BTN_SMD_4x3mm, symbol Switch:SW_Push
- added R125: 4.7K, Resistor_SMD:R_0402_1005Metric, symbol Device:R
- added R126: 1M, Resistor_SMD:R_0805_2012Metric, symbol Device:R
- added R127: 9.53K, Resistor_SMD:R_0402_1005Metric, symbol Device:R_Small
- added TP18: TestPoint_Small, TestPoint:TestPoint_Pad_2.0x2.0mm, symbol Connector:TestPoint_Small
- added U35: TLV70012_SOT23-5, Package_TO_SOT_SMD:SOT-23-5, symbol Regulator_Linear:TLV70012_SOT23-5
- added U36: TUSB8041, Package_DFN_QFN:QFN-64-1EP_9x9mm_P0.5mm_EP6x6mm_ThermalVias, symbol Interface_USB:TUSB8041
- added X5: X322512MSB4SI, Crystal:Crystal_SMD_3225-4Pin_3.2x2.5mm, symbol Device:Crystal_GND24
- D31: value MMSZ4678T1G -> 1.8V; footprint Diode_SMD:D_SOD-123 -> Diode_SMD:D_SOD-323; LCSC C36599 -> C779376
- R98: value 3.3K -> 430R; LCSC C25890 -> C36356
Connections:
- net +3.3V_MAIN: now also C140.2, C141.2, C142.2, C143.2, C144.2, U35.1 (IN), U35.3 (EN), U36.16 (VDD33), U36.34 (VDD33), U36.52 (VDD33), U36.63 (VDD33)
- net +5V_MAIN: now also F4.1
- net +VBATT: now also F5.1
- net BATT_GND: now also C139.2, K_80.2; no longer C88.2
- net BQ_CELL1: no longer K_86.2, U24.4
- net BQ_REGOUT_3V3: now also C139.1
- net BQ_REGSRC: no longer TP16.1
- net CELL1: now also K_86.2, U24.4
- net CHG_SCL: no longer R124.1, SJ17.2, TP11.1, U22.5 (SDA), U4.15 (SDA)
- net CM5_PWR_BTN: now also TP16.1
- net DSCH_PATH: no longer C88.1
- net GND: now also C140.1, C141.1, C142.1, C143.1, C144.1, C145.1, C146.1, C147.1, C148.1, C149.1, C150.1, C151.1, C152.1, C153.1, C154.1, C155.1, R125.1, R126.1, R127.1, U35.2 (GND), U36.65 (VSS), X5.2, X5.4
- net HUB_US_D+: now also JP1.3 (B); no longer JP1.2 (C)
- net HUB_US_D-: now also JP2.3 (B); no longer JP2.2 (C)
- net M2B_USB3_RX_N: no longer Module3.157 (USB3-1-RX_N)
- net M2B_USB3_RX_P: no longer Module3.159 (USB3-1-RX_P)
- net M2B_USB3_TX_N: no longer Module3.169 (USB3-1-TX_N)
- net M2B_USB3_TX_P: no longer Module3.171 (USB3-1-TX_P)
- net M2B_USBD_N: no longer Module3.165 (USB3-1-D_N)
- net M2B_USBD_P: no longer Module3.163 (USB3-1-D_P)
- net PCIE-RX_N: now also J16.41 (PERn0/SATA-B+); no longer J16.47 (PETn0/SATA-A-)
- net PCIE-RX_P: now also J16.43 (PERp0/SATA-B-); no longer J16.49 (PETp0/SATA-A+)
- net PCIE-TX_N: now also J16.49 (PETp0/SATA-A+); no longer J16.43 (PERp0/SATA-B-)
- net PCIE-TX_P: now also J16.47 (PETn0/SATA-A-); no longer J16.41 (PERn0/SATA-B+)
- net PWR_BTN: now also K_80.1
- net SHIP_WAKE_3V3: now also TP18.1
- net USB3_0_D_N: now also U36.54 (USB_DM_UP)
- net USB3_0_D_P: now also U36.53 (USB_DP_UP)
- net USB3_0_RX_N: now also U36.59 (USB_SSRXM_UP)
- net USB3_0_RX_P: now also U36.58 (USB_SSRXP_UP)
- net USB3_0_TX_N: now also U36.56 (USB_SSTXM_UP)
- net USB3_0_TX_P: now also U36.55 (USB_SSTXP_UP)
- net at R92.2, U16.6 (SRP): now also C88.2
- net at R93.1, U16.7 (SRN): now also C88.1
- net USB2_D_N renamed CM5_USB2-D_N
- net CM5_USB2-D_N: now also JP2.2 (C); no longer JP2.3 (B)
- net USB2_D_P renamed CM5_USB2-D_P
- net CM5_USB2-D_P: now also JP1.2 (C); no longer JP1.3 (B)
- new net: R127.2, U36.64 (USB_R1)
- new net: R125.2, U36.49 (TEST)
- new net +1.1V_HUB: C145.2, C146.2, C147.2, C148.2, C149.2, C150.2, C151.2, C152.2, C153.2, U35.5 (OUT), U36.13 (VDD), U36.21 (VDD), U36.28 (VDD), U36.31 (VDD), U36.5 (VDD), U36.51 (VDD), U36.57 (VDD), U36.8 (VDD)
- new net CHG_SDA: R124.1, SJ17.2, TP11.1, U22.5 (SDA), U4.15 (SDA)
- new net USB3_1_D_N: Module3.165 (USB3-1-D_N)
- new net USB3_1_D_P: Module3.163 (USB3-1-D_P)
- new net USB3_1_RX_N: Module3.157 (USB3-1-RX_N)
- new net USB3_1_RX_P: Module3.159 (USB3-1-RX_P)
- new net USB3_1_TX_N: Module3.169 (USB3-1-TX_N)
- new net USB3_1_TX_P: Module3.171 (USB3-1-TX_P)
- new net USB3_HUB_XI: C155.2, U36.62 (XI)
- new net USB3_HUB_XO: C154.2, R126.2, U36.61 (XO), X5.1, X5.3
- no-connect marks 113 -> 119
Other:
- note added: "Mesh Node SDR"
- moved on the sheet: C88, R100, R124, R92, R93, R94

Commit message: updates
Parts:
- removed D1, D2, D3: LED_0402, LED_SMD:LED_0402_1005Metric, symbol Device:LED
- removed F4: 500mA, Fuse:Fuse_0603_1608Metric, symbol Device:Fuse_Small
- removed R20, R21, R22: 30R, Resistor_SMD:R_0402_1005Metric, symbol Device:R_Small
- added C156: 1uF, Capacitor_SMD:C_0402_1005Metric, symbol Device:C_Small
- added C157: 2.2uF, Capacitor_SMD:C_0603_1608Metric, symbol Device:C_Small
- added J25: USB_C_Receptacle_USB2.0_16P, LibraryGlobalFootprints:USB_C_Receptacle_HRO_TYPE-C-31-M-12, symbol Connector:USB_C_Receptacle_USB2.0_16P
- added R128, R129: 5.1K, Resistor_SMD:R_0402_1005Metric, symbol Device:R
- added SJ18: SHP_OFF, LibraryGlobalFootprints:SOLDERJUMPER_ARROW_NOPASTE, symbol Adafruit TFP401 to 40pin TFT-eagle-import:SOLDERJUMPER
- added SJ19: LoRa VBUS, LibraryGlobalFootprints:SOLDERJUMPER_ARROW_NOPASTE, symbol Adafruit TFP401 to 40pin TFT-eagle-import:SOLDERJUMPER
- added TP9: TestPoint_Small, TestPoint:TestPoint_Pad_2.0x2.0mm, symbol Connector:TestPoint_Small
- added U37: RAK4630, LibraryGlobalFootprints:RAK4630, symbol LibraryGlobalSymbols:RAK4630
- added U38: TPS70933DBVR, Package_TO_SOT_SMD:SOT-23-5, symbol Regulator_Linear:LP2985-3.3
- added U39: USBLC6-2SC6, Package_TO_SOT_SMD:SOT-23-6, symbol Power_Protection:USBLC6-2SC6
- D23: Description_1 PWR_LED -> RP2040_LED
- D36: Description_1 BATT_LED -> PWR_LED
- U19: DESCRIPTION Super Speed Type-C DRP Port Controller USB 3.1 3.3V/5V T/R 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 -> (none)
- U31: value ~ -> (none)
Connections:
- net +5V_MAIN: no longer C137.2, C17.1, J21.A4 (VBUSA1), J21.A9 (VBUSA2), J21.B4 (VBUSB1), J21.B9 (VBUSB2), R118.2, R68.1, R69.1, R70.1, U19.30 (VDD5), U33.5 (IN)
- net +5V_PORT_C: no longer U33.1 (OUT)
- net +VBATT: now also SJ18.1, SJ18.2
- net 3V3_MAIN: now also R52.2
- net 5V_MAIN: now also R49.2
- net CM5_USB_OTG_ID: no longer S1.1
- net GND: now also C155.2, C156.2, C157.1, J25.A1 (GND), J25.A12 (GND), J25.B1 (GND), J25.B12 (GND), J25.S1 (SHIELD), R128.1, R129.1, U37.14 (GND1), U37.16 (GND2), U37.22 (GND3), U37.35 (GND4), U37.36 (GND5), U37.38 (GND6), U37.42 (GND7), U38.2 (GND), U39.2 (GND); no longer C155.1, R126.1, S1.2
- net HUB2_DS_1_D+: now also U37.2 (USB-), U39.6 (I/O1)
- net HUB2_DS_1_D-: now also U37.3 (USB+), U39.4 (I/O2)
- net M2B_USB3_RX_N: now also U36.30 (USB_SSRXM_DN4); no longer U19.9 (RXP)
- net M2B_USB3_RX_P: now also U36.29 (USB_SSRXP_DN4); no longer U19.10 (RXN)
- net M2B_USB3_TX_N: now also U36.27 (USB_SSTXM_DN4); no longer U19.7 (TXN)
- net M2B_USB3_TX_P: now also U36.26 (USB_SSTXP_DN4); no longer U19.6 (TXP)
- net M2B_USBD_N: now also U36.25 (USB_DM_DN4); no longer D34.1 (D+), J21.A7 (DA-), J21.B7 (DB-)
- net M2B_USBD_P: now also U36.24 (USB_DP_DN4); no longer D34.2 (D-), J21.A6 (DA+), J21.B6 (DB+)
- net PD_3V3: now also TP9.1
- net USB3_HUB_XI: now also C154.2, R126.2, X5.1; no longer C155.2
- net USB3_HUB_XO: now also C155.1, R126.1; no longer C154.2, R126.2, X5.1
- net at F5.2: now also S1.2
- net C3_USBD_P: now reaches U36.17 (USB_DP_DN3)
- net C3_USBD_P: now also D34.1 (D+), J21.A6 (DA+), J21.B6 (DB+)
- net C3_USBD_N: now reaches U36.18 (USB_DM_DN3)
- net C3_USBD_N: now also D34.2 (D-), J21.A7 (DA-), J21.B7 (DB-)
- net C3_USB3_TX_P: now reaches U36.19 (USB_SSTXP_DN3)
- net C3_USB3_TX_P: now also U19.6 (TXP)
- net C3_USB3_TX_N: now reaches U36.20 (USB_SSTXM_DN3)
- net C3_USB3_TX_N: now also U19.7 (TXN)
- net C3_USB3_RX_P: now reaches U36.22 (USB_SSRXP_DN3)
- net C3_USB3_RX_P: now also U19.9 (RXP)
- net C3_USB3_RX_N: now reaches U36.23 (USB_SSRXM_DN3)
- net C3_USB3_RX_N: now also U19.10 (RXN)
- net LED_0 renamed CAPS_LOCK_LED
- net LED_1: no longer names the net of U2.20 (PB2)
- net LED_2: no longer names the net of U2.21 (PB10)
- net LED_3: no longer names the net of U2.22 (PB11)
- new net: J25.A7 (D-), J25.B7 (D-), U39.1 (I/O1)
- new net: J25.A6 (D+), J25.B6 (D+), U39.3 (I/O2)
- new net: C137.2, R118.2, U33.5 (IN)
- new net: J25.A5 (CC1), R129.2
- new net: SJ19.1, U37.1 (VBUS)
- new net: J25.B5 (CC2), R128.2
- new net +3.3V_LORA: C157.2, U37.20 (VBAT_SX), U37.21 (VBAT_IO_SX), U37.43 (VDD_NRF), U37.44 (VBAT_NRF), U38.5 (VOUT)
- new net +5V_PORT_C3.0: C17.1, J21.A4 (VBUSA1), J21.A9 (VBUSA2), J21.B4 (VBUSB1), J21.B9 (VBUSB2), R68.1, R69.1, R70.1, U19.30 (VDD5), U33.1 (OUT)
- new net LORA_VBUS: J25.A4 (VBUS), J25.A9 (VBUS), J25.B4 (VBUS), J25.B9 (VBUS), SJ19.2, U39.5 (VBUS)
- new net VBATT_LORA: C156.1, S1.1, U38.1 (VIN)
- no-connect marks 119 -> 127
Other:
- note added: "USB HUB 2"
- note removed: "Indicator LEDs"
- note removed: "Power LED"
- moved on the sheet: C137, C154, C155, C17, C72, C73, C74, C75, D23, D34, D4, J13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

Commit message: work on PCB
Parts:
- J7: footprint LibraryGlobalFootprints:AFC01-S05FCA-00_1x05_P0.5mm_FFC_Bottom_Contact -> LibraryGlobalFootprints:AFC07-S05ECA-00; LCSC C5213747 -> C262578
Changed lines of the file:
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@@
 			)
 		)
-		(property "Footprint" "LibraryGlobalFootprints:AFC01-S05FCA-00_1x05_P0.5mm_FFC_Bottom_Contact"
+		(property "Footprint" "LibraryGlobalFootprints:AFC07-S05ECA-00"
 			(at 52.07 242.57 0)
 			(hide yes)
@@
 			)
 		)
-		(property "LCSC" "C5213747"
+		(property "LCSC" "C262578"
 			(at 52.07 242.57 0)
 			(hide yes)
