File: pcb-deck-r1-fixed/cyberdeck-alpha.kicad_pcb (KiCad board)
At the start: 4 copper layers, 105.8 x 152.9 mm, 508 parts, among them J1 CPU_FAN, J10 Conn_01x30, J11 Conn_01x22, J12 HDMI_C_1.3, J13 USB_C_Receptacle_USB2.0_16P, J14 Conn_01x06, J15 Conn_02x20_Odd_Even, J16 1-2199119-5, J19 TSOP77438TR, J2 GP_LB, J20 Conn_01x22, J21 DX07S024JJ2R1300, J3 GP_RB, J4 JOYSTICK, J5 Conn_01x06_Pin, J6 USB_C_Receptacle_USB2.0_16P, J7 Conn_01x05, J8 PJ-342B, J9 SPK, Q1 IRLML6244, Q2 CJ2101, Q3 SI4174DY-T1-GE3_N-Channel_FET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, Q5 IRLML6244, Q6 SI4174DY-T1-GE3_N-Channel_FET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, Q7 SI4174DY-T1-GE3_N-Channel_FET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, Q8 SI4174DY-T1-GE3_N-Channel_FET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, U1 W25Q128JVS, U10 TPS62180YZFR, U11 TPS62180YZFR, U12 SY6280_OCP, U13 FAN5333ASX, U14 USBLC6-2SC6, U15 SY6280_OCP, U16 BQ76905RGRR, U17 ATtiny202-SS, U18 TPS25751SRSMR, U19 HD3SS3220IRNHT, U2 STM32F072CBT6, U20 TPD4EUSB30DQAR, U21 TPD4EUSB30DQAR, U22 AT24CS01-SSHM, U3 XC6206, U4 BQ25792RQMR, U5 RP2040, U6 USBLC6-2SC6, U7 CH334R, U8 PAM8406AB, U9 PCM2706CPJT, X1 X322512MSB4SI, X2 X322512MSB4SI, X3 X322512MSB4SI

Commit message: work on PCB
Parts:
- removed C68: 10uF, Capacitor_SMD:C_0805_2012Metric
- removed C69, C70: 1uF, Capacitor_SMD:C_0805_2012Metric
- removed C71: 100nF, Capacitor_SMD:C_0805_2012Metric
- removed D25: MBR0540, Diode_SMD:D_SOD-123
- removed D26: MM3Z24VT1G, Diode_SMD:D_SOD-323
- removed J10: Conn_01x30, LibraryGlobalFootprints:AFC07-S30ECA-00
- removed J14: Conn_01x06, LibraryGlobalFootprints:AFC07-S06ECA-00
- removed J4: JOYSTICK, LibraryGlobalFootprints:1x04_P2.54 SMD pads only
- removed JP13: SolderJumper_10_Open, LibraryGlobalFootprints:SolderJumper-10
- removed K_79: ZX-QC66-4.3TP, LibraryGlobalFootprints:ZX-QC66-7.5TP
- removed L5: BRL3225T150K, Inductor_SMD:L_1210_3225Metric
- removed NT6, NT7: NetTie_2, NetTie:NetTie-2_SMD_Pad0.5mm
- removed R57: 10K, Resistor_SMD:R_0805_2012Metric
- removed R58: 3R, Resistor_SMD:R_0805_2012Metric
- removed R59, R60: 12R, Resistor_SMD:R_0805_2012Metric
- removed R95: 10K, Resistor_SMD:R_0402_1005Metric
- removed S1: SSSS811101, LibraryGlobalFootprints:SW_SSSS811101
- removed SJ1: HUB_D_P, LibraryGlobalFootprints:SOLDERJUMPER_ARROW_NOPASTE
- removed SJ2: HUB_D_M, LibraryGlobalFootprints:SOLDERJUMPER_ARROW_NOPASTE
- removed SJ3: +50mA, LibraryGlobalFootprints:SOLDERJUMPER_ARROW_NOPASTE
- removed SJ4: +25mA, LibraryGlobalFootprints:SOLDERJUMPER_ARROW_NOPASTE
- removed SJ5: BKLT_PWR, LibraryGlobalFootprints:SOLDERJUMPER_ARROW_NOPASTE
- removed U13: FAN5333ASX, Package_TO_SOT_SMD:SOT-23-5
- added D_71: MBR0540, Diode_SMD:D_SOD-123, B.Cu at (240.0, 28.7)
- added J22: USB_C_Receptacle_USB2.0_16P, LibraryGlobalFootprints:USB_C_Receptacle_HRO_TYPE-C-31-M-12, B.Cu at (151.0, 52.6)
- added K_87: PWR_BTN, LibraryGlobalFootprints:dome-tactile-pad, F.Cu at (202.0, 91.0)
- added R100: 4.7K, Resistor_SMD:R_0402_1005Metric, B.Cu at (162.6, 67.9)
- added R101: 430R, Resistor_SMD:R_0402_1005Metric, B.Cu at (159.0, 67.9)
- added R105: 140R, Resistor_SMD:R_0402_1005Metric, B.Cu at (166.8, 20.4)
- added R106: 140R, Resistor_SMD:R_0402_1005Metric, B.Cu at (171.4, 20.4)
- added R107: 140R, Resistor_SMD:R_0402_1005Metric, B.Cu at (163.6, 21.2)
- added R122: 430R, Resistor_SMD:R_0402_1005Metric, B.Cu at (173.1, 88.5)
- added R123: 470K, Resistor_SMD:R_0402_1005Metric, B.Cu at (169.5, 89.3)
- added R124: 4.7K, Resistor_SMD:R_0402_1005Metric, B.Cu at (163.7, 67.9)
- added R98: 10K, Resistor_SMD:R_0402_1005Metric, B.Cu at (154.8, 84.5)
- added R99: 4.7K, Resistor_SMD:R_0402_1005Metric, B.Cu at (154.8, 86.7)
- added TP14: TestPoint_Small, TestPoint:TestPoint_Pad_2.0x2.0mm, F.Cu at (150.4, 92.4)
- added TP15: TestPoint_Small, TestPoint:TestPoint_Pad_2.0x2.0mm, F.Cu at (150.4, 89.1)
- added TP9: TestPoint_Small, TestPoint:TestPoint_Pad_2.0x2.0mm, F.Cu at (150.4, 96.0)
- added U24: AT3H7B-CuH-S, LibraryGlobalFootprints:SSOP-4_AT3H7B-CuH-S, B.Cu at (171.8, 94.0)
- added U25: USBLC6-2SC6, Package_TO_SOT_SMD:SOT-23-6, B.Cu at (158.6, 58.0)
- added U32: AT3H7B-CuH-S, LibraryGlobalFootprints:SSOP-4_AT3H7B-CuH-S, B.Cu at (156.8, 64.8)
- J7: footprint LibraryGlobalFootprints:AFC01-S05FCA-00_1x05_P0.5mm_FFC_Bottom_Contact -> LibraryGlobalFootprints:AFC07-S05ECA-00
- K_73: value ZX-QC66-4.3TP -> GP_START; footprint LibraryGlobalFootprints:ZX-QC66-7.5TP -> LibraryGlobalFootprints:dome-tactile-pad
- K_74: value ZX-QC66-4.3TP -> GP_SELECT; footprint LibraryGlobalFootprints:ZX-QC66-7.5TP -> LibraryGlobalFootprints:dome-tactile-pad
- K_80: value ZX-QC66-4.3TP -> GP_MODE; footprint LibraryGlobalFootprints:ZX-QC66-7.5TP -> LibraryGlobalFootprints:dome-tactile-pad
- R63: value 6.8K -> 3.4K
- R66: value 1K -> 10K
- U17: value ATtiny202-SS -> ATtiny404-SS; footprint Package_SO:SOIC-8_3.9x4.9mm_P1.27mm -> Package_SO:SOIC-14_3.9x8.7mm_P1.27mm
- moved G*** 67.0 mm to (178.3, 60.2)
- moved R24 64.0 mm to (150.0, 82.0), turned to 180 degrees
- moved D23 62.7 mm to (150.0, 83.1), turned to 180 degrees
- moved JP2 29.1 mm to (216.5, 80.6), turned to 90 degrees
- moved D33 25.9 mm to (149.8, 85.4)
- moved JP1 24.8 mm to (213.9, 80.6), turned to 90 degrees
- moved TP1 23.3 mm to (172.0, 102.9)
- moved J11 23.1 mm to (182.6, 44.0), turned to 90 degrees
- moved C79 22.1 mm to (182.1, 35.3), turned to 180 degrees
- moved R64 20.1 mm to (169.4, 87.7), turned to 180 degrees
- moved TP2 12.7 mm to (172.0, 107.0)
- moved C110 12.5 mm to (172.2, 70.1)
- moved C123 10.5 mm to (163.8, 63.5)
- moved U22 10.5 mm to (168.5, 65.5)
- moved D31 10.5 mm to (166.4, 89.7)
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Connections:
- net /BQ_BATT+ renamed /SENS_BATT+
- net /BQ_BATT- renamed /SENS_BATT-
- net /BQ_CELL1 renamed /SENS_CELL1
- BT1 pad 1: /CELL+ -> +VBATT
- BT2 pad 2: /CELL- -> BAT_GND
- C104 pad 1: /3V3_SHIP_MODE_OFF -> /SHIP_WAKE_3V3
- C20 pad 1: unconnected-(C20-Pad1) -> GND
- C67 pad 2: +5V_MAIN -> +5V_CM5_SUPPLY
- C72 pad 2: /USB31_TX1_N -> /USB31_TX1_P
- C73 pad 2: /USB31_TX1_P -> /USB31_TX1_N
- C84 pad 1: /CELL- -> BAT_GND
- C88 pad 2: /CELL- -> BAT_GND
- C90 pad 1: /GND_OUT -> GND
- C91 pad 2: /GND_OUT -> GND
- C92 pad 1: /CELL+ -> +VBATT
- D23 pad 1: GND -> /PWR_LED
- D27 pad 3: GND -> Net-(D27-PAD)
- D28 pad 3: GND -> Net-(D28-PAD)
- D29 pad 3: GND -> Net-(D29-PAD)
- D31 pad 2: /GND_OUT -> BAT_GND
- D33 pad 2: /CELL- -> GND
- J11 pad 11: /MIPI1_D2_A_P -> /MIPI1_D2_P
- J11 pad 12: /MIPI1_D2_A_N -> /MIPI1_D2_N
- J11 pad 14: /MIPI1_CLK_A_P -> /MIPI1_CLK_P
- J11 pad 15: /MIPI1_CLK_A_N -> /MIPI1_CLK_N
- J11 pad 17: /MIPI1_D1_A_P -> /MIPI1_D1_P
- J11 pad 18: /MIPI1_D1_A_N -> /MIPI1_D1_N
- J11 pad 20: /MIPI1_D0_A_P -> /MIPI1_D0_P
- J11 pad 21: /MIPI1_D0_A_N -> /MIPI1_D0_N
- J11 pad 8: /MIPI1_D3_A_P -> /MIPI1_D3_P
- J11 pad 9: /MIPI1_D3_A_N -> /MIPI1_D3_N
- J13 pad A4: +VBUS -> +5V_CM5_SUPPLY
- J13 pad A5: /PD_CC1 -> /CM5_CC1
- J13 pad A9: +VBUS -> +5V_CM5_SUPPLY
- J13 pad B4: +VBUS -> +5V_CM5_SUPPLY
- J13 pad B5: /PD_CC2 -> /CM5_CC2
- J13 pad B9: +VBUS -> +5V_CM5_SUPPLY
- J15 pad 27: /ID_SDA_GPIO_0 -> /MIPI1_SDA
- J15 pad 28: /ID_SCL_GPIO_1 -> /MIPI1_SCL
- J16 pad 41: /PCIE-TX_P -> /PCIE-RX_N
- J16 pad 43: /PCIE-TX_N -> /PCIE-RX_P
- J16 pad 47: /PCIE-RX_N -> /PCIE-TX_N
- J16 pad 49: /PCIE-RX_P -> /PCIE-TX_P
- J20 pad 2: /ID_SDA_GPIO_0 -> /MIPI0_SDA
- J20 pad 3: /ID_SCL_GPIO_1 -> /MIPI0_SCL
- J7 pad 1: /JOYSTICK_Y -> +3.3V_MAIN
- J7 pad 2: GND -> /JOYSTICK_X
- J7 pad 4: /JOYSTICK_X -> GND
- J7 pad 5: +3.3V_MAIN -> /JOYSTICK_Y
- JP1 pad 1: /HUB_US_D+ -> /USB2_CM5_P
- JP1 pad 2: /CM5_USB_D_P -> /HUB_US_D+
- JP1 pad 3: /USB2_SYS_P -> /USB3_0_D_P
- JP2 pad 1: /HUB_US_D- -> /USB2_CM5_N
- JP2 pad 2: /CM5_USB_D_N -> /HUB_US_D-
- JP2 pad 3: /USB2_SYS_N -> /USB3_0_D_N
- K_85 pad 1: /SHIP_MODE -> /SHIP_BTN
- K_85 pad 2: GND -> BAT_GND
- Module2 pad 35: /ID_SCL_GPIO_1 -> /MIPI1_SCL
- Module2 pad 36: /ID_SDA_GPIO_0 -> /MIPI1_SDA
- Module2 pad 80: /MIPI1_SCL -> /MIPI0_SCL
- Module2 pad 82: /MIPI1_SDA -> /MIPI0_SDA
- Module3 pad 103: /CM5_USB_D_N -> /USB2_CM5_N
- Module3 pad 105: /CM5_USB_D_P -> /USB2_CM5_P
- NT1 pad 2: /CELL+ -> +VBATT
- NT2 pad 1: /CELL+ -> +VBATT
- NT3 pad 1: /CELL- -> BAT_GND
- Q2 pad 2: Net-(D33-K) -> Net-(D31-K)
- Q6 pad 1: /GND_OUT -> GND
- Q6 pad 2: /GND_OUT -> GND
- Q6 pad 3: /GND_OUT -> GND
- Q6 pad 4: Net-(D31-K) -> Net-(D33-K)
- R61 pad 2: +5V_MAIN -> +5V_CM5_SUPPLY
- R64 pad 1: Net-(R64-Pad1) -> /SHIP_BTN
- R64 pad 2: Net-(D33-K) -> Net-(D31-K)
- R66 pad 1: /CM5_PWR_BTN -> /BQ_3V3
- R66 pad 2: Net-(U17-PA6) -> /BQ_SCL
- R83 pad 2: /ID_SCL_GPIO_1 -> /MIPI0_SCL
- R84 pad 2: /ID_SDA_GPIO_0 -> /MIPI0_SDA
- R86 pad 1: Net-(D31-K) -> Net-(D33-K)
- R87 pad 1: /GND_OUT -> GND
- R87 pad 2: Net-(D31-K) -> Net-(D33-K)
- R92 pad 1: /CELL- -> BAT_GND
- R94 pad 2: /CELL- -> BAT_GND
- SJ14 pad 1: /3V3_SHIP_MODE_OFF -> /SHIP_OFF_TRG
- SJ14 pad 2: Net-(R64-Pad1) -> /SHIP_BTN
- TP1 pad 1: /CELL+ -> +VBATT
- TP5 pad 1: /CELL- -> BAT_GND
- U14 pad 4: /USB2_SYS_P -> /USB2_CM5_N
- U14 pad 5: +VBUS -> +5V_CM5_SUPPLY
- U14 pad 6: /USB2_SYS_N -> /USB2_CM5_P
- U15 pad 5: +5V_MAIN -> +5V_CM5_SUPPLY
- U16 pad 11: /CELL- -> BAT_GND
- U16 pad 14: unconnected-(U16-ALERT-Pad14) -> /BQ_ALERT
- U16 pad 21: /CELL- -> BAT_GND
- U17 pad 2: Net-(U17-PA6) -> /PWR_LED
- U17 pad 3: unconnected-(U17-PA7-Pad3) -> /PWR_BTN
- U17 pad 4: /BQ_SDA -> /SHIP_BTN
- U17 pad 5: /BQ_SCL -> /SOFT_PWR_OUT
- U17 pad 6: /TINY202_UPDI -> unconnected-(U17-PB3-Pad6)
- U17 pad 7: /SHIP_MODE -> unconnected-(U17-PB2-Pad7)
- U17 pad 8: GND -> unconnected-(U17-PB1-Pad8)
- U18 pad 1: /3V3_SHIP_MODE_OFF -> /SHIP_WAKE_3V3
- U18 pad 22: /USB2_SYS_P -> /USB2_CHG_P
- U18 pad 23: /USB2_SYS_N -> /USB2_CHG_N
- U19 pad 10: /M2B_USB3_RX_P -> /M2B_USB3_RX_N
- U19 pad 14: /USB31_RX1_P -> /USB31_RX1_N
- U19 pad 15: /USB31_RX1_N -> /USB31_RX1_P
- U19 pad 9: /M2B_USB3_RX_N -> /M2B_USB3_RX_P
Routing:
- net /USB2_SYS_P: track 120.3 -> 0.00 mm, vias 3 -> 0
- net /USB2_SYS_N: track 118.6 -> 0.00 mm, vias 3 -> 0
- net /PD_CC1: track 143.8 -> 27.9 mm, vias 5 -> 3
- net BAT_GND: track 0.00 -> 111.2 mm, vias 0 -> 5
- net /PD_CC2: track 138.1 -> 30.1 mm, vias 7 -> 3
- net /ID_SCL_GPIO_1: track 101.9 -> 0.00 mm, vias 6 -> 0
- net +VBUS: track 134.4 -> 37.4 mm, vias 5 -> 0
- net /ID_SDA_GPIO_0: track 95.3 -> 0.00 mm, vias 4 -> 0
- net /DISP_RST: track 94.6 -> 0.93 mm, vias 3 -> 1
- net /DISP_SCL: track 92.7 -> 1.50 mm, vias 2 -> 1
- net /DISP_INT: track 91.2 -> 1.11 mm, vias 3 -> 1
- net /DISP_SDA: track 91.1 -> 1.05 mm, vias 2 -> 1
- net /USB2_CM5_N: track 0.00 -> 87.5 mm, vias 0 -> 3
- net +VBATT: track 7.84 -> 95.2 mm, vias 0 -> 5
- net /USB2_CM5_P: track 0.00 -> 86.3 mm, vias 0 -> 3
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Other:
- outline, holes or cut-outs redrawn
- board text added: "1-2 CM4 2-3 CM5"
- board text added: "BATT_GND"
- board text added: "BMS_SCL"
- board text added: "BMS_SDA"
- board text added: "CM5 USB"
- board text added: "GPIO"
- board text added: "MIPI1"
- board text added: "RPi 40P"
- board text added: "USB HOST"
- board text removed: "1-2 HUB 2-3 OTG"
- board text removed: "1-2: 22pin DSI, 2-3: 30pin DSI"
- board text removed: "123"
- board text removed: "22P"
- board text removed: "30P"
- board text removed: "<-- use flux!"
- board text removed: "BACKLITE DRIVER"
- board text removed: "MIPI 1"
- board text removed: "ONB. USB SELECT"
- board text removed: "RPi 40P GPIO"
- board text removed: "TOUCH"
- board text removed: "USB CHG, OTG"
- board text removed: "USB HUB"
