File: pcb-deck-r1-fixed/cyberdeck-alpha.kicad_sch (KiCad schematic)
At the start: 523 parts, among them J1 CPU_FAN, J10 Conn_01x30, J11 Conn_01x22, J12 HDMI_C_1.3, J13 USB_C_Receptacle_USB2.0_16P, J14 Conn_01x06, J15 Conn_02x20_Odd_Even, J16 1-2199119-5, J17 2199119-3, J18 SIM_Card, J19 TSOP77438TR, J2 GP_LB, J20 Conn_01x22, J21 DX07S024JJ2R1300, J22 USB3_A, J3 GP_RB, J4 JOYSTICK, J5 Conn_01x06_Pin, J6 USB_C_Receptacle_USB2.0_16P, J7 Conn_01x05, J8 PJ-342B, J9 SPK, Q1 IRLML6244, Q2 CJ2101, Q3 SI4174DY-T1-GE3_N-Channel_FET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, Q4 BSS138, Q5 IRLML6244, Q6 SI4174DY-T1-GE3_N-Channel_FET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, Q7 SI4174DY-T1-GE3_N-Channel_FET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, Q8 SI4174DY-T1-GE3_N-Channel_FET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, U1 W25Q128JVS, U10 TPS62180YZFR, U11 TPS62180YZFR, U12 SY6280_OCP, U13 FAN5333ASX, U14 USBLC6-2SC6, U15 SY6280_OCP, U16 BQ76905RGRR, U17 ATtiny202-SS, U18 TPS25751SRSMR, U19 HD3SS3220IRNHT, U2 STM32F072CBT6, U20 TPD4EUSB30DQAR, U21 TPD4EUSB30DQAR, U22 AT24CS01-SSHM, U23 CH334R, U3 XC6206, U4 BQ25792RQMR, U5 RP2040, U6 USBLC6-2SC6, U7 CH334R, U8 PAM8406AB, U9 PCM2706CPJT, X1 X322512MSB4SI, X2 X322512MSB4SI, X3 X322512MSB4SI, X4 X322512MSB4SI

Commit message: work on PCB
Parts:
- removed C124: 10uF, Capacitor_SMD:C_0603_1608Metric, symbol Device:C_Small
- removed C125: 100nF, Capacitor_SMD:C_0402_1005Metric, symbol Device:C_Small
- removed C126: 22uF, Capacitor_SMD:C_0805_2012Metric, symbol Device:C
- removed C68: 10uF, Capacitor_SMD:C_0805_2012Metric, symbol Device:C_Small
- removed C69, C70: 1uF, Capacitor_SMD:C_0805_2012Metric, symbol Device:C_Small
- removed C71: 100nF, Capacitor_SMD:C_0805_2012Metric, symbol Device:C_Small
- removed D25: MBR0540, Diode_SMD:D_SOD-123, symbol Diode:MBR0540
- removed D26: MM3Z24VT1G, Diode_SMD:D_SOD-323, symbol Device:D
- removed J10: Conn_01x30, LibraryGlobalFootprints:AFC07-S30ECA-00, symbol Connector_Generic_MountingPin:Conn_01x30_MountingPin
- removed J14: Conn_01x06, LibraryGlobalFootprints:AFC07-S06ECA-00, symbol Connector_Generic_MountingPin:Conn_01x06_MountingPin
- removed J22: USB3_A, LibraryGlobalFootprints:U-A-39DS-Y-1, symbol Connector:USB3_A
- removed J4: JOYSTICK, LibraryGlobalFootprints:1x04_P2.54 SMD pads only, symbol Connector:Conn_01x04_Pin
- removed JP13: SolderJumper_10_Open, LibraryGlobalFootprints:SolderJumper-10, symbol LibraryGlobalSymbols:SolderJumper_10_Open
- removed K_79: ZX-QC66-4.3TP, LibraryGlobalFootprints:ZX-QC66-7.5TP, symbol Switch:SW_Push
- removed L5: BRL3225T150K, Inductor_SMD:L_1210_3225Metric, symbol Device:L
- removed NT6, NT7: NetTie_2, NetTie:NetTie-2_SMD_Pad0.5mm, symbol Device:NetTie_2
- removed R57: 10K, Resistor_SMD:R_0805_2012Metric, symbol Adafruit TFP401 to 40pin TFT-eagle-import:RESISTOR0805_NOOUTLINE
- removed R58: 3R, Resistor_SMD:R_0805_2012Metric, symbol Adafruit TFP401 to 40pin TFT-eagle-import:RESISTOR0805_NOOUTLINE
- removed R59, R60: 12R, Resistor_SMD:R_0805_2012Metric, symbol Adafruit TFP401 to 40pin TFT-eagle-import:RESISTOR0805_NOOUTLINE
- removed R65: 0R, Resistor_SMD:R_0402_1005Metric, symbol Device:R
- removed R95: 10K, Resistor_SMD:R_0402_1005Metric, symbol Device:R
- removed S1: SSSS811101, LibraryGlobalFootprints:SW_SSSS811101, symbol LibraryGlobalSymbols:SSSS811101
- removed SJ1: HUB_D_P, LibraryGlobalFootprints:SOLDERJUMPER_ARROW_NOPASTE, symbol Adafruit TFP401 to 40pin TFT-eagle-import:SOLDERJUMPER
- removed SJ2: HUB_D_M, LibraryGlobalFootprints:SOLDERJUMPER_ARROW_NOPASTE, symbol Adafruit TFP401 to 40pin TFT-eagle-import:SOLDERJUMPER
- removed SJ3: +50mA, LibraryGlobalFootprints:SOLDERJUMPER_ARROW_NOPASTE, symbol Adafruit TFP401 to 40pin TFT-eagle-import:SOLDERJUMPER
- removed SJ4: +25mA, LibraryGlobalFootprints:SOLDERJUMPER_ARROW_NOPASTE, symbol Adafruit TFP401 to 40pin TFT-eagle-import:SOLDERJUMPER
- removed SJ5: BKLT_PWR, LibraryGlobalFootprints:SOLDERJUMPER_ARROW_NOPASTE, symbol Adafruit TFP401 to 40pin TFT-eagle-import:SOLDERJUMPER
- removed U13: FAN5333ASX, Package_TO_SOT_SMD:SOT-23-5, symbol Adafruit TFP401 to 40pin TFT-eagle-import:VREG_FAN5331
- removed U17: ATtiny202-SS, Package_SO:SOIC-8_3.9x4.9mm_P1.27mm, symbol MCU_Microchip_ATtiny:ATtiny202-SS
- removed U23: CH334R, Package_SO:QSOP-16_3.9x4.9mm_P0.635mm, symbol Interface_USB:CH334R
- removed X4: X322512MSB4SI, Crystal:Crystal_SMD_3225-4Pin_3.2x2.5mm, symbol Device:Crystal_GND24
- added D_71: MBR0540, Diode_SMD:D_SOD-123, symbol Device:D_Small
- added J22: USB_C_Receptacle_USB2.0_16P, LibraryGlobalFootprints:USB_C_Receptacle_HRO_TYPE-C-31-M-12, symbol Connector:USB_C_Receptacle_USB2.0_16P
- added K_87: PWR_BTN, LibraryGlobalFootprints:dome-tactile-pad, symbol Switch:SW_Push
- added R100, R124, R99: 4.7K, Resistor_SMD:R_0402_1005Metric, symbol Device:R
- added R101, R122: 430R, Resistor_SMD:R_0402_1005Metric, symbol Device:R
- added R105, R106, R107: 140R, Resistor_SMD:R_0402_1005Metric, symbol Device:R
- added R123: 470K, Resistor_SMD:R_0402_1005Metric, symbol Device:R
- added R98: 10K, Resistor_SMD:R_0402_1005Metric, symbol Device:R
- added TP14, TP15, TP9: TestPoint_Small, TestPoint:TestPoint_Pad_2.0x2.0mm, symbol Connector:TestPoint_Small
- added U17: ATtiny404-SS, Package_SO:SOIC-14_3.9x8.7mm_P1.27mm, symbol MCU_Microchip_ATtiny:ATtiny404-SS
- added U24, U32: AT3H7B-CuH-S, LibraryGlobalFootprints:SSOP-4_AT3H7B-CuH-S, symbol Isolator:PC817
- added U25: USBLC6-2SC6, Package_TO_SOT_SMD:SOT-23-6, symbol Power_Protection:USBLC6-2SC6
- J7: footprint LibraryGlobalFootprints:AFC01-S05FCA-00_1x05_P0.5mm_FFC_Bottom_Contact -> LibraryGlobalFootprints:AFC07-S05ECA-00; LCSC C5213747 -> C262578
- K_73: value ZX-QC66-4.3TP -> GP_START; footprint LibraryGlobalFootprints:ZX-QC66-7.5TP -> LibraryGlobalFootprints:dome-tactile-pad; Description_1 GP_STA -> (none); LCSC C7470157 -> (none)
- K_74: value ZX-QC66-4.3TP -> GP_SELECT; footprint LibraryGlobalFootprints:ZX-QC66-7.5TP -> LibraryGlobalFootprints:dome-tactile-pad; Description_1 GP_SEL -> (none); LCSC C7470157 -> (none)
- K_80: value ZX-QC66-4.3TP -> GP_MODE; footprint LibraryGlobalFootprints:ZX-QC66-7.5TP -> LibraryGlobalFootprints:dome-tactile-pad; Description_1 GP_MODE -> (none); LCSC C7470157 -> (none)
- R63: value 6.8K -> 3.4K; LCSC C25917 -> C4940
- R66: value 1K -> 10K; LCSC C11702 -> C25744
- U19: DESCRIPTION Super Speed Type-C DRP Port Controller USB 3.1 3.3V/5V T/R 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 -> (none)
Connections:
- net CELL+ is gone; now on net +VBATT: BT1.1 (+), C92.1, NT1.2, NT2.1, TP1.1
- net HUB2_US_D+ is gone; now on net HUB_DS_3_D+: U7.2 (DP4+)
- net HUB2_US_D- is gone; now on net HUB_DS_3_D-: U7.1 (DM4-)
- net MIPI1_CLK_A_N is gone; now on net MIPI1_CLK_N: J11.15 (Pin_15)
- net MIPI1_CLK_A_P is gone; now on net MIPI1_CLK_P: J11.14 (Pin_14)
- net MIPI1_D0_A_N is gone; now on net MIPI1_D0_N: J11.21 (Pin_21)
- net MIPI1_D0_A_P is gone; now on net MIPI1_D0_P: J11.20 (Pin_20)
- net MIPI1_D1_A_N is gone; now on net MIPI1_D1_N: J11.18 (Pin_18)
- net MIPI1_D1_A_P is gone; now on net MIPI1_D1_P: J11.17 (Pin_17)
- net MIPI1_D2_A_N is gone; now on net MIPI1_D2_N: J11.12 (Pin_12)
- net MIPI1_D2_A_P is gone; now on net MIPI1_D2_P: J11.11 (Pin_11)
- net MIPI1_D3_A_N is gone; now on net MIPI1_D3_N: J11.9 (Pin_9)
- net MIPI1_D3_A_P is gone; now on net MIPI1_D3_P: J11.8 (Pin_8)
- net SHIP_MODE is gone; now on net SHIP_BTN: K_85.1
- net +3.3V_MAIN: now also J7.1 (Pin_1), R100.2, R124.2; no longer J7.5 (Pin_5)
- net +5V_MAIN: now also D_71.2 (A); no longer C67.2, R61.2, U15.5 (IN)
- net +VBUS: now also J22.A4 (VBUS), J22.A9 (VBUS), J22.B4 (VBUS), J22.B9 (VBUS), U25.5 (VBUS); no longer J13.A4 (VBUS), J13.A9 (VBUS), J13.B4 (VBUS), J13.B9 (VBUS), U14.5 (VBUS)
- net BQ_3V3: now also R66.1, R98.1, U17.1 (VCC), U32.1
- net BQ_SCL: now also R66.2, TP14.1, U17.12 (PA2)
- net BQ_SDA: now also R98.2, TP15.1, U17.11 (PA1)
- net CELL1: now also U24.4
- net CHG_SCL: now also R100.1
- net CHG_SDA: now also R124.1
- net CM5_CC1: now also J13.A5 (CC1)
- net CM5_CC2: now also J13.B5 (CC2)
- net CM5_PWR_BTN: now also U32.4; no longer R66.1
- net GND: now also C20.1, C90.1, C91.2, D33.2 (A), J7.4 (Pin_4), Q6.1 (S), Q6.2 (S), Q6.3 (S), R87.1, J22.A1 (GND), J22.A12 (GND), J22.B1 (GND), J22.B12 (GND), J22.S1 (SHIELD), R105.1, R106.1, R107.1, R122.1, U25.2 (GND), U32.3; no longer D23.1 (K), D27.3 (PAD), D28.3 (PAD), D29.3 (PAD), J7.2 (Pin_2), K_85.2
- net HUB_US_D+: now also JP1.2 (C); no longer JP1.1 (A)
- net HUB_US_D-: now also JP2.2 (C); no longer JP2.1 (A)
- net JOYSTICK_X: now also J7.2 (Pin_2); no longer J7.4 (Pin_4)
- net JOYSTICK_Y: now also J7.5 (Pin_5); no longer J7.1 (Pin_1)
- net M2B_USB3_RX_N: now also U19.10 (RXN); no longer U19.9 (RXP)
- net M2B_USB3_RX_P: now also U19.9 (RXP); no longer U19.10 (RXN)
- net MIPI1_SCL: now also J15.28 (Pin_28), Module2.35 (ID_SC); no longer Module2.80 (SCL0)
- net MIPI1_SDA: now also J15.27 (Pin_27), Module2.36 (ID_SD); no longer Module2.82 (SDA0)
- net PCIE-RX_N: now also J16.41 (PERn0/SATA-B+); no longer J16.47 (PETn0/SATA-A-)
- net PCIE-RX_P: now also J16.43 (PERp0/SATA-B-); no longer J16.49 (PETp0/SATA-A+)
- net PCIE-TX_N: now also J16.47 (PETn0/SATA-A-); no longer J16.43 (PERp0/SATA-B-)
- net PCIE-TX_P: now also J16.49 (PETp0/SATA-A+); no longer J16.41 (PERn0/SATA-B+)
- net PD_CC1: now also J22.A5 (CC1); no longer J13.A5 (CC1)
- net PD_CC2: now also J22.B5 (CC2); no longer J13.B5 (CC2)
- net TINY202_UPDI: now also R99.2
- net USB31_RX1_N: now also U19.14 (RX1N); no longer U19.15 (RX1P)
- net USB31_RX1_P: now also U19.15 (RX1P); no longer U19.14 (RX1N)
- net USB31_TX1_N: now also C73.2; no longer C72.2
- net USB31_TX1_P: now also C72.2; no longer C73.2
- net USB3_0_D_N: now also JP2.3 (B)
- net USB3_0_D_P: now also JP1.3 (B)
- net at Q6.4 (G), R86.1, R87.2: now also D33.1 (K); no longer D31.1 (K)
- net BQ_ALERT: now reaches U16.14 (ALERT)
- net BQ_ALERT: now also U17.13 (PA3)
- net SHIP_BTN: now reaches R64.1, SJ14.2
- net SHIP_BTN: now also R123.2, U17.4 (PA6)
- net at Q2.2 (S), R64.2: now also D31.1 (K); no longer D33.1 (K)
- net 3V3_SHIP_MODE_OFF renamed SHIP_WAKE_3V3
- net SHIP_WAKE_3V3: now also U24.1; no longer SJ14.1
- net BQ_BATT+ renamed SENS_BATT+
- net BQ_BATT- renamed SENS_BATT-
- net BQ_CELL1 renamed SENS_CELL1
- net CELL- renamed BAT_GND
- net BAT_GND: now also D31.2 (A), K_85.2, K_87.2, R123.1, TP9.1, U17.14 (GND); no longer D33.2 (A)
- net CM5_USB_D_N renamed USB2_CM5_N
- net USB2_CM5_N: now also JP2.1 (A), U14.4 (I/O2); no longer JP2.2 (C)
- net CM5_USB_D_P renamed USB2_CM5_P
- net USB2_CM5_P: now also JP1.1 (A), U14.6 (I/O1); no longer JP1.2 (C)
- removed net GND_OUT: C90.1, C91.2, D31.2 (A), Q6.1 (S), Q6.2 (S), Q6.3 (S), R87.1
- net HUB2_DS_0_D+ renamed HUB_DS_3_D+
- net HUB2_DS_0_D- renamed HUB_DS_3_D-
- net ID_SCL_GPIO_1 renamed MIPI0_SCL
- net MIPI0_SCL: now also Module2.80 (SCL0); no longer J15.28 (Pin_28), Module2.35 (ID_SC)
- net ID_SDA_GPIO_0 renamed MIPI0_SDA
- net MIPI0_SDA: now also Module2.82 (SDA0); no longer J15.27 (Pin_27), Module2.36 (ID_SD)
- removed net USB2_SYS_N: JP2.3 (B), U14.6 (I/O1), U18.23 (GPIO5/USB_N/MD2)
- removed net USB2_SYS_P: JP1.3 (B), U14.4 (I/O2), U18.22 (GPIO5/USB_P/MD1)
- new net: D28.3 (PAD), R105.2
- new net: D29.3 (PAD), R106.2
- new net: D27.3 (PAD), R107.2
- new net: R101.1, U32.2
- new net: J22.A6 (D+), J22.B6 (D+), U25.1 (I/O1)
- new net: J22.A7 (D-), J22.B7 (D-), U25.3 (I/O2)
- new net: R99.1, U17.10 (~{RESET}/PA0)
- new net: R122.2, U24.2
- new net +5V_CM5_SUPPLY: C67.2, D_71.1 (K), J13.A4 (VBUS), J13.A9 (VBUS), J13.B4 (VBUS), J13.B9 (VBUS), R61.2, U14.5 (VBUS), U15.5 (IN)
- new net PWR_BTN: K_87.1, U17.3 (PA5)
- new net PWR_LED: D23.1 (K), U17.2 (PA4)
- new net SHIP_OFF_TRG: SJ14.1, U24.3
- new net SOFT_PWR_OUT: R101.2, U17.5 (PA7)
- new net USB2_CHG_N: U18.23 (GPIO5/USB_N/MD2), U25.4 (I/O2)
- new net USB2_CHG_P: U18.22 (GPIO5/USB_P/MD1), U25.6 (I/O1)
- no-connect marks 115 -> 105
Other:
- note added: "USB-C CM5 System Port"
- note added: "USB-C PD Charge Port"
- note removed: "BACKLIGHT PWR"
- note removed: "USB A Port"
- note removed: "USB-C PD Charge / CM5 System Port"
- moved on the sheet: BT1, BT2, C123, C17, C28, C32, C33, C67, C72, C73, C74, C75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
