File: PCB/cyberdeck/cyberdeck.kicad_pcb (KiCad board)
At the start: 4 copper layers, 208.1 x 160.2 mm, 634 parts, among them J1 CPU_FAN, J10 DM3AT-SF-PEJM5, J11 Conn_01x22, J12 HDMI_C_1.3, J13 USB_C_Receptacle_USB2.0_16P, J14 USB_C_Receptacle_USB2.0_16P, J15 PZ254-2-20-W-8.5, J16 1-2199119-5, J17 2199230-3, J18 SIM_Card, J19 TSOP77438TR, J2 GP_LB, J20 Conn_01x22, J21 DX07S024JJ2R1300, J22 USB3_A, J23 Conn_01x06_Pin, J24 Conn_01x06_Pin, J25 USB_C_Receptacle_USB2.0_16P, J3 GP_RB, J4 JOYSTICK, J5 Conn_01x06_Pin, J6 USB_C_Receptacle_USB2.0_16P, J7 Conn_01x05, J8 PJ-342B, J9 RJ45_LED_Shielded, Q1 IRLML6244, Q2 CJ2101, Q3 SI4174DY-T1-GE3_N-Channel_FET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, Q5 IRLML6244, Q6 SI4174DY-T1-GE3_N-Channel_FET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, Q7 SI4174DY-T1-GE3_N-Channel_FET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, Q8 SI4174DY-T1-GE3_N-Channel_FET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, U1 W25Q128JVS, U12 SY6280_OCP, U13 USBLC6-2SC6, U14 USBLC6-2SC6, U15 SY6280_OCP, U16 BQ76905RGRR, U17 ATtiny404-SS, U18 TPS25751SRSMR, U19 HD3SS3220IRNHT, U2 STM32F072CBT6, U20 TPD4EUSB30DQAR, U21 TPD4EUSB30DQAR, U22 AT24CS01-SSHM, U23 CH334R, U24 AT3H7B-CuH-S, U25 SY6280_OCP, U26 SY6280_OCP, U27 USBLC6-2SC6, U28 SY6280_OCP, U29 SY6280_OCP, U3 XC6206, U30 SY6280_OCP, U32 AT3H7B-CuH-S, U33 SY6280_OCP, U34 SY6280_OCP, U35 TLV70012_SOT23-5, U36 TUSB8041, U37 RAK4630, U38 TPS70933DBVR, U39 USBLC6-2SC6, U4 BQ25792RQMR, U40 MLX90632, U41 TPS566231RQFR, U42 TPS566231RQFR, U5 RP2040, U6 USBLC6-2SC6, U7 CH334R, U8 PAM8406AB, U9 PCM2706CPJT, X1 X322512MSB4SI, X2 X322512MSB4SI, X3 X322512MSB4SI, X4 X322512MSB4SI, X5 X322512MSB4SI

Commit message: test usb 3 hub, test pwr regs v3
Parts:
- removed J4: JOYSTICK, LibraryGlobalFootprints:1x04_P2.54 SMD pads only
- added R140: 430R, Resistor_SMD:R_0402_1005Metric, F.Cu at (47.5, 57.0)
- added R141: 430R, Resistor_SMD:R_0402_1005Metric, F.Cu at (47.5, 58.9)
- added TP27: TestPoint_Small, TestPoint:TestPoint_Pad_D1.0mm, B.Cu at (167.1, 119.0)
- added TP28: TestPoint_Small, TestPoint:TestPoint_Pad_D1.0mm, B.Cu at (168.4, 120.5)
- added TP29: TestPoint_Small, TestPoint:TestPoint_Pad_D1.0mm, B.Cu at (170.6, 121.4)
- added TP30: TestPoint_Small, TestPoint:TestPoint_Pad_D1.0mm, B.Cu at (173.9, 118.9)
- added TP31: TestPoint_Small, TestPoint:TestPoint_Pad_D1.0mm, B.Cu at (172.6, 120.5)
- added U43: AT3H7B-CuH-S, LibraryGlobalFootprints:SSOP-4_AT3H7B-CuH-S, F.Cu at (50.8, 49.7)
- added U44: AT3H7B-CuH-S, LibraryGlobalFootprints:SSOP-4_AT3H7B-CuH-S, F.Cu at (50.8, 53.9)
- moved G*** 148.1 mm to (273.7, 151.1)
- moved R60 19.5 mm to (232.1, 84.7)
- moved U26 19.5 mm to (235.4, 86.1)
- moved C128 19.5 mm to (238.2, 86.8)
- moved R59 19.5 mm to (238.2, 84.8)
- moved R132 16.1 mm to (111.7, 30.1), turned to 0 degrees
- moved R135 16.0 mm to (111.6, 20.2), turned to 0 degrees
- moved C98 15.8 mm to (65.8, 41.4)
- moved C99 15.8 mm to (65.8, 39.3)
- moved C102 15.8 mm to (59.1, 41.0)
- moved C107 15.8 mm to (62.4, 48.2)
- moved C76 15.8 mm to (59.6, 43.1)
- moved C94 15.8 mm to (62.0, 50.3)
- moved R74 15.8 mm to (63.1, 51.0)
- moved U4 15.8 mm to (59.4, 46.5)
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Connections:
- net Net-(U41-EN) renamed /PWR_TRIGGER_5V
- net Net-(U42-EN) renamed /PWR_TRIGGER_3V3
- J7 pad 1: +3.3V_MAIN -> /JOYSTICK_Y
- J7 pad 2: /JOYSTICK_X -> GND
- J7 pad 4: GND -> /JOYSTICK_X
- J7 pad 5: /JOYSTICK_Y -> +3.3V_MAIN
Routing:
- net /5V_MAIN: track 21.1 -> 2.88 mm, vias 2 -> 0
- net /3V3_MAIN: track 19.5 -> 2.88 mm, vias 2 -> 0
- net VIN: track 21.2 -> 5.32 mm, vias 0 -> 10
- net Net-(U42-FB): track 2.42 -> 9.53 mm
- net Net-(U41-FB): track 2.48 -> 9.53 mm
- net Net-(D_70-K): track 9.84 -> 2.92 mm
- net +5V_PORT_A: track 20.1 -> 13.3 mm
- net /ETH_BL2_N: track 4.21 -> 10.5 mm
- net /ETH_BL3_P: track 4.19 -> 10.3 mm
- net /ETH_BL2_P: track 4.22 -> 10.3 mm
- net /ETH_BL3_N: track 4.19 -> 9.95 mm
- net /ETH_RX1_P: track 3.94 -> 8.93 mm
- net Net-(C133-Pad1): track 26.8 -> 23.7 mm
- net /JOYSTICK_X: track 56.0 -> 59.0 mm
- net /ETH_TX0_N: track 4.34 -> 7.28 mm
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- added copper zone on F.Cu, net /3V3_MAIN
- added copper zone on F.Cu, net /5V_MAIN
- added copper zone on F.Cu, net Net-(U41-SW)
- added copper zone on F.Cu, net Net-(U42-SW)
- added copper zone on F.Cu, net VIN
Other:
- board size 208.1 x 160.2 mm -> 208.1 x 167.2 mm
- board text added: "18x9mm"
- board text added: "3-18V 6 AMP"
- board text added: "BTN"
- board text added: "L7"
