File: PCB/cyberdeck/cyberdeck.kicad_pcb (KiCad board)
At the start: 4 copper layers, 208.1 x 167.2 mm, 642 parts, among them J1 CPU_FAN, J10 DM3AT-SF-PEJM5, J11 Conn_01x22, J12 HDMI_C_1.3, J13 USB_C_Receptacle_USB2.0_16P, J14 USB_C_Receptacle_USB2.0_16P, J15 PZ254-2-20-W-8.5, J16 1-2199119-5, J17 2199230-3, J18 SIM_Card, J19 TSOP77438TR, J2 GP_LB, J20 Conn_01x22, J21 DX07S024JJ2R1300, J22 USB3_A, J23 Conn_01x06_Pin, J24 Conn_01x06_Pin, J25 USB_C_Receptacle_USB2.0_16P, J3 GP_RB, J5 Conn_01x06_Pin, J6 USB_C_Receptacle_USB2.0_16P, J7 Conn_01x05, J8 PJ-342B, J9 RJ45_LED_Shielded, Q1 IRLML6244, Q2 CJ2101, Q3 SI4174DY-T1-GE3_N-Channel_FET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, Q5 IRLML6244, Q6 SI4174DY-T1-GE3_N-Channel_FET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, Q7 SI4174DY-T1-GE3_N-Channel_FET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, Q8 SI4174DY-T1-GE3_N-Channel_FET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, U1 W25Q128JVS, U12 SY6280_OCP, U13 USBLC6-2SC6, U14 USBLC6-2SC6, U15 SY6280_OCP, U16 BQ76905RGRR, U17 ATtiny404-SS, U18 TPS25751SRSMR, U19 HD3SS3220IRNHT, U2 STM32F072CBT6, U20 TPD4EUSB30DQAR, U21 TPD4EUSB30DQAR, U22 AT24CS01-SSHM, U23 CH334R, U24 AT3H7B-CuH-S, U25 SY6280_OCP, U26 SY6280_OCP, U27 USBLC6-2SC6, U28 SY6280_OCP, U29 SY6280_OCP, U3 XC6206, U30 SY6280_OCP, U32 AT3H7B-CuH-S, U33 SY6280_OCP, U34 SY6280_OCP, U35 TLV70012_SOT23-5, U36 TUSB8041, U37 RAK4630, U38 TPS70933DBVR, U39 USBLC6-2SC6, U4 BQ25792RQMR, U40 MLX90632, U41 TPS566231RQFR, U42 TPS566231RQFR, U43 AT3H7B-CuH-S, U44 AT3H7B-CuH-S, U5 RP2040, U6 USBLC6-2SC6, U7 CH334R, U8 PAM8406AB, U9 PCM2706CPJT, X1 X322512MSB4SI, X2 X322512MSB4SI, X3 X322512MSB4SI, X4 X322512MSB4SI, X5 X322512MSB4SI

Commit message: stuff and things
Parts:
- removed D_70: MBR0540, Diode_SMD:D_SOD-123
- removed R79, R80: 10K, Resistor_SMD:R_0402_1005Metric
- added C169: 1uF, Capacitor_SMD:C_0402_1005Metric, F.Cu at (219.5, 29.9)
- added C179: 10uF, Capacitor_SMD:C_0805_2012Metric, F.Cu at (162.0, 45.5)
- added C180: 0.1uF, Capacitor_SMD:C_0805_2012Metric, F.Cu at (162.0, 48.5)
- added C181: 10uF, Capacitor_SMD:C_0805_2012Metric, F.Cu at (162.0, 51.5)
- added C182: 10uF, Capacitor_SMD:C_0805_2012Metric, F.Cu at (162.0, 54.5)
- added C183: 10uF, Capacitor_SMD:C_0805_2012Metric, F.Cu at (166.5, 36.5)
- added C184: 1uF, Capacitor_SMD:C_0805_2012Metric, F.Cu at (166.5, 39.5)
- added C185: 1uF, Capacitor_SMD:C_0805_2012Metric, F.Cu at (166.5, 42.5)
- added C186: 0.1uF, Capacitor_SMD:C_0805_2012Metric, F.Cu at (166.5, 45.5)
- added C55: 0.1uF, Capacitor_SMD:C_0805_2012Metric, F.Cu at (157.6, 36.5)
- added C56: 0.1uF, Capacitor_SMD:C_0805_2012Metric, F.Cu at (157.6, 39.5)
- added C57: 0.1uF, Capacitor_SMD:C_0805_2012Metric, F.Cu at (157.6, 42.5)
- added C58: 0.1uF, Capacitor_SMD:C_0805_2012Metric, F.Cu at (157.6, 45.5)
- added C60: 0.1uF, Capacitor_SMD:C_0805_2012Metric, F.Cu at (157.6, 48.5)
- added C61: 0.1uF, Capacitor_SMD:C_0805_2012Metric, F.Cu at (157.6, 51.5)
- added C62: 0.1uF, Capacitor_SMD:C_0805_2012Metric, F.Cu at (157.6, 54.5)
- added C63: 0.1uF, Capacitor_SMD:C_0805_2012Metric, F.Cu at (162.0, 36.5)
- added C64: 0.1uF, Capacitor_SMD:C_0805_2012Metric, F.Cu at (162.0, 39.5)
- added C65: 10uF, Capacitor_SMD:C_0805_2012Metric, F.Cu at (162.0, 42.5)
- added D1: MBR0540, Diode_SMD:D_SOD-123, F.Cu at (178.0, 41.3)
- added D2: MM3Z24VT1G, Diode_SMD:D_SOD-323, F.Cu at (173.0, 41.1)
- added D3: 1N4148, Diode_SMD:D_SOD-323, F.Cu at (183.0, 39.8)
- added D42: LED_0402, LED_SMD:LED_0402_1005Metric, B.Cu at (150.8, 64.2)
- added D43: LED_0402, LED_SMD:LED_0402_1005Metric, B.Cu at (150.8, 83.5)
- added D_71: MBR0540, Diode_SMD:D_SOD-123, B.Cu at (243.2, 49.1)
- added FB1: Ferrite, Inductor_SMD:L_0805_2012Metric, F.Cu at (192.8, 35.6)
- added FB2: Ferrite, Inductor_SMD:L_0805_2012Metric, F.Cu at (192.8, 38.4)
- added FB3: Ferrite, Inductor_SMD:L_0805_2012Metric, F.Cu at (183.9, 60.2)
- added FB4: Ferrite, Inductor_SMD:L_0805_2012Metric, F.Cu at (183.9, 63.0)
- added H5: SMTWE2030MTJ, LibraryGlobalFootprints:M.2 M2 nut standoff, B.Cu at (196.9, 91.5)
- added LED2: Green, LED_SMD:LED_0805_2012Metric, F.Cu at (150.8, 20.4)
- added LED3: Blue, LED_SMD:LED_0805_2012Metric, F.Cu at (150.9, 23.9)
- added Q4: BSS138, Package_TO_SOT_SMD:SOT-23, F.Cu at (201.1, 68.8)
- added R142: 10K, Resistor_SMD:R_0402_1005Metric, F.Cu at (213.7, 33.3)
- added R143: 90.9K, Resistor_SMD:R_0402_1005Metric, F.Cu at (213.7, 35.3)
- added R144: 33, Resistor_SMD:R_Array_Convex_4x0603, F.Cu at (174.9, 49.8)
- added R145: 33, Resistor_SMD:R_Array_Convex_4x0603, F.Cu at (179.1, 49.8)
- added R146: 10K, Resistor_SMD:R_0805_2012Metric, F.Cu at (175.3, 59.5)
- added R147: 3 ohm, Resistor_SMD:R_0805_2012Metric, F.Cu at (175.3, 62.5)
- added R148: 12 ohm, Resistor_SMD:R_0805_2012Metric, F.Cu at (179.7, 53.6)
- added R149: 12 ohm, Resistor_SMD:R_0805_2012Metric, F.Cu at (179.7, 56.6)
- added R150: 1K, Resistor_SMD:R_0805_2012Metric, F.Cu at (179.7, 59.5)
- added R151: 1K, Resistor_SMD:R_0805_2012Metric, F.Cu at (179.7, 62.5)
- added R152: 100K, Resistor_SMD:R_0402_1005Metric, B.Cu at (171.4, 41.9)
- added R153: 100K, Resistor_SMD:R_0402_1005Metric, B.Cu at (171.4, 46.1)
- added R20: 10K, Resistor_SMD:R_0805_2012Metric, F.Cu at (170.9, 53.6)
- added R21: 10K, Resistor_SMD:R_0805_2012Metric, F.Cu at (170.9, 56.6)
- added R22: 10K, Resistor_SMD:R_0805_2012Metric, F.Cu at (170.9, 59.5)
- added R48: 10K, Resistor_SMD:R_0805_2012Metric, F.Cu at (170.9, 62.5)
- added R49: 10K, Resistor_SMD:R_0805_2012Metric, F.Cu at (175.3, 53.6)
- added R50: 1K, Resistor_SMD:R_0805_2012Metric, F.Cu at (175.3, 56.6)
- added R51: 33, Resistor_SMD:R_Array_Convex_4x0603, F.Cu at (170.8, 45.0)
- added R52: 33, Resistor_SMD:R_Array_Convex_4x0603, F.Cu at (174.9, 45.0)
- added R53: 33, Resistor_SMD:R_Array_Convex_4x0603, F.Cu at (179.1, 45.0)
- added U10: 24LC02BT-I/OT, Package_TO_SOT_SMD:SOT-23-5, F.Cu at (197.6, 36.6)
- added U11: LT1117(3V3), Package_TO_SOT_SMD:SOT-223-3_TabPin2, F.Cu at (157.0, 60.2)
- added U45: FAN5333ASX, Package_TO_SOT_SMD:SOT-23-5, F.Cu at (196.8, 69.5)
- added X7: AFC07-S40ECA-00, LibraryGlobalFootprints:FFC_Receptable_1x40_P0.5mm_AFC07-S40ECA-00, F.Cu at (165.1, 28.7)
- BATT1: renamed from BT1; moved to B.Cu
- BATT2: renamed from BT2; moved to B.Cu
- C100, C101, C102, C103, C104, C105, C106, C107, C108, C109, C110, C111, C112, C113, C114, C115, C116, C117, C118, C119, C120, C121, C122, C123, C139, C177, C178, C76, C77, C84, C85, C86, C87, C88, C89, C90, C91, C92, C93, C94, C95, C96, C97, C98, C99, D30, D31, D32, D33, D35, D36, D38, D39, D40, D41, F2, H4, J14, K_80, K_86, L5, L6, L7, Q2, Q3, Q6, Q7, Q8, R100, R101, R122, R123, R124, R136, R137, R138, R139, R140, R141, R64, R66, R71, R72, R73, R74, R75, R85, R86, R87, R88, R89, R90, R91, R92, R93, R94, R95, R96, R97, R98, R99, SJ14, SJ15, SJ16, SJ17, SJ18, TP1, TP10, TP11, TP12, TP13, TP14, TP15, TP16, TP17, TP18, TP19, TP2, TP3, TP4, TP5, TP6, TP7, TP8, TP9, U16, U17, U18, U22, U24, U27, U32, U4, U43, U44: moved to B.Cu
- C140, C141, C142, C143, C144, C145, C146, C147, C148, C149, C150, C151, C152, C153, C154, C155, C18, C20, C28, C32, C33, C36, C37, C39, C53, G*** (x3), J5, R125, R126, R127, R32, R33, R42, SJ1, U35, U36, U7, U8, X1, X5: moved to F.Cu
- J25: value USB_C_Receptacle_USB2.0_16P -> PJ-342B; footprint LibraryGlobalFootprints:USB_C_Receptacle_HRO_TYPE-C-31-M-12 -> LibraryGlobalFootprints:PJ-342B
- J9: value RJ45_LED_Shielded -> RJ45_Shielded; footprint LibraryGlobalFootprints:RC01812 -> LibraryGlobalFootprints:CONN-SMD_RJ-064
- R128, R129: value 5.1K -> 33; footprint Resistor_SMD:R_0402_1005Metric -> Resistor_SMD:R_Array_Convex_4x0603; moved to F.Cu
- U39: value USBLC6-2SC6 -> TFP401; footprint Package_TO_SOT_SMD:SOT-23-6 -> LibraryGlobalFootprints:TFP401 - S-PQFP-G100; moved to F.Cu
- moved J14 244.5 mm to (251.6, 165.1)
- moved U27 231.0 mm to (243.2, 162.9), turned to 180 degrees
- moved G*** 190.3 mm to (153.3, 169.5), turned to 0 degrees
- moved R130 134.2 mm to (252.4, 12.5)
- moved R131 134.2 mm to (252.4, 14.5)
- moved C158 134.2 mm to (252.4, 16.4)
- moved U40 128.8 mm to (249.2, 12.7)
- moved G*** 128.7 mm to (123.8, 102.6), turned to 55 degrees
- moved TP20 127.4 mm to (221.8, 55.5)
- moved TP24 127.4 mm to (221.8, 59.0)
- moved TP23 127.4 mm to (221.8, 52.3)
- moved TP25 127.4 mm to (221.8, 49.2)
- moved U43 124.6 mm to (175.0, 40.1), turned to 180 degrees
- moved U44 124.6 mm to (175.0, 44.3), turned to 180 degrees
- moved J25 119.6 mm to (247.3, 152.7), turned to 180 degrees
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Connections:
- C137 pad 2: Net-(U33-IN) -> +5V_MAIN
- C17 pad 1: +5V_PORT_C3.0 -> +VBUS_C3.0
- C72 pad 2: /USB31_TX1_N -> /USB31_TX1_P
- C73 pad 2: /USB31_TX1_P -> /USB31_TX1_N
- J11 pad 11: /MIPI1_D2_P -> /MIPI0_D2_P
- J11 pad 12: /MIPI1_D2_N -> /MIPI0_D2_N
- J11 pad 14: /MIPI1_CLK_P -> /MIPI0_CLK_P
- J11 pad 15: /MIPI1_CLK_N -> /MIPI0_CLK_N
- J11 pad 17: /MIPI1_D1_P -> /MIPI0_D1_P
- J11 pad 18: /MIPI1_D1_N -> /MIPI0_D1_N
- J11 pad 2: /MIPI1_SDA -> /MIPI0_SDA
- J11 pad 20: /MIPI1_D0_P -> /MIPI0_D0_P
- J11 pad 21: /MIPI1_D0_N -> /MIPI0_D0_N
- J11 pad 3: /MIPI1_SCL -> /MIPI0_SCL
- J11 pad 5: unconnected-(J11-Pin_5-Pad5) -> /CAM_GPIO1
- J11 pad 6: unconnected-(J11-Pin_6-Pad6) -> /CAM_GPIO0
- J11 pad 8: /MIPI1_D3_P -> /MIPI0_D3_P
- J11 pad 9: /MIPI1_D3_N -> /MIPI0_D3_N
- J16 pad 47: /PCIE-TX_P -> /PCIE-TX_N
- J16 pad 49: /PCIE-TX_N -> /PCIE-TX_P
- J20 pad 11: /MIPI0_D2_P -> /MIPI1_D2_P
- J20 pad 12: /MIPI0_D2_N -> /MIPI1_D2_N
- J20 pad 14: /MIPI0_CLK_P -> /MIPI1_CLK_P
- J20 pad 15: /MIPI0_CLK_N -> /MIPI1_CLK_N
- J20 pad 17: /MIPI0_D1_P -> /MIPI1_D1_P
- J20 pad 18: /MIPI0_D1_N -> /MIPI1_D1_N
- J20 pad 2: /MIPI0_SDA -> /MIPI1_SDA
- J20 pad 20: /MIPI0_D0_P -> /MIPI1_D0_P
- J20 pad 21: /MIPI0_D0_N -> /MIPI1_D0_N
- J20 pad 3: /MIPI0_SCL -> /MIPI1_SCL
- J20 pad 5: /CAM_GPIO1 -> unconnected-(J20-Pin_5-Pad5)
- J20 pad 6: /CAM_GPIO0 -> unconnected-(J20-Pin_6-Pad6)
- J20 pad 8: /MIPI0_D3_P -> /MIPI1_D3_P
- J20 pad 9: /MIPI0_D3_N -> /MIPI1_D3_N
- J21 pad A4: +5V_PORT_C3.0 -> +VBUS_C3.0
- J21 pad A9: +5V_PORT_C3.0 -> +VBUS_C3.0
- J21 pad B4: +5V_PORT_C3.0 -> +VBUS_C3.0
- J21 pad B9: +5V_PORT_C3.0 -> +VBUS_C3.0
- J22 pad 1: Net-(D_70-K) -> +5V_PORT_A
- J22 pad 5: unconnected-(J22-SSRX--Pad5) -> /PORT_USBA_RX_N
- J22 pad 6: unconnected-(J22-SSRX+-Pad6) -> /PORT_USBA_RX_P
- J22 pad 8: unconnected-(J22-SSTX--Pad8) -> /PORT_USBA_TX_N
- J22 pad 9: unconnected-(J22-SSTX+-Pad9) -> /PORT_USBA_TX_P
- J9 pad 10: /CM5_3V3 -> CHA_GND
- J9 pad 11: Net-(J9-Pad11) -> CHA_GND
- J9 pad 12: /CM5_3V3 -> CHA_GND
- J9 pad 9: Net-(J9-Pad9) -> CHA_GND
- R110 pad 1: Net-(J9-Pad9) -> Net-(D43-K)
- R118 pad 2: Net-(U33-IN) -> +5V_MAIN
- R128 pad 1: GND -> /G3
- R128 pad 2: Net-(J25-CC2) -> /G2
- R129 pad 1: GND -> /G7
- R129 pad 2: Net-(J25-CC1) -> /G6
- R54 pad 2: /MIPI1_SDA -> /MIPI0_SDA
- R55 pad 2: /MIPI1_SCL -> /MIPI0_SCL
- R82 pad 1: Net-(J9-Pad11) -> Net-(D42-K)
- R83 pad 2: /MIPI0_SCL -> /MIPI1_SCL
- R84 pad 2: /MIPI0_SDA -> /MIPI1_SDA
- U13 pad 4: /PORT_USBA2_D+ -> /PORT_USBA_D+
- U13 pad 6: /PORT_USBA2_D- -> /PORT_USBA_D-
- U19 pad 14: /USB31_RX1_P -> /USB31_RX1_N
- U19 pad 15: /USB31_RX1_N -> /USB31_RX1_P
- U33 pad 5: Net-(U33-IN) -> +5V_MAIN
- U36 pad 10: unconnected-(U36-USB_DM_DN2-Pad10) -> /PORT_USBA_D-
- U36 pad 11: unconnected-(U36-USB_SSTXP_DN2-Pad11) -> /PORT_USBA_TX_P
- U36 pad 12: unconnected-(U36-USB_SSTXM_DN2-Pad12) -> /PORT_USBA_TX_N
- U36 pad 14: unconnected-(U36-USB_SSRXP_DN2-Pad14) -> /PORT_USBA_RX_P
- U36 pad 15: unconnected-(U36-USB_SSRXM_DN2-Pad15) -> /PORT_USBA_RX_N
- U36 pad 48: unconnected-(U36-USB_VBUS-Pad48) -> /VBUS_DET
- U36 pad 50: unconnected-(U36-GRSTz-Pad50) -> /HUB_RST
- U36 pad 9: unconnected-(U36-USB_DP_DN2-Pad9) -> /PORT_USBA_D+
- U39 pad 1: Net-(J25-D--PadA7) -> GND
- U39 pad 2: GND -> /PWRDN
- U39 pad 3: Net-(J25-D+-PadA6) -> Net-(U39A-ST)
- U39 pad 4: /HUB2_DS_1_D- -> GND
- U39 pad 5: /LORA_VBUS -> GND
- U39 pad 6: /HUB2_DS_1_D+ -> VDDIO
- U43 pad 4: /5V_IN -> /VBATT
- U44 pad 4: /3V3_IN -> /VBATT
Routing:
- net +3.3V_MAIN: track 279.3 -> 161.1 mm, vias 16 -> 7
- net +5V_MAIN: track 280.6 -> 205.7 mm, vias 14 -> 10
- net /HUB2_DS_0_D+: track 67.5 -> 4.44 mm, vias 2 -> 1
- net /HUB2_DS_0_D-: track 66.8 -> 4.23 mm, vias 2 -> 1
- net +5V_INT_USB: track 62.3 -> 0.00 mm, vias 3 -> 0
- net /HUB_US_D-: track 60.6 -> 0.00 mm, vias 1 -> 0
- net /HUB_US_D+: track 59.0 -> 0.00 mm, vias 1 -> 0
- net /JOYSTICK_X: track 59.0 -> 2.95 mm, vias 2 -> 0
- net /DAC_USB_D+: track 60.5 -> 5.06 mm, vias 2 -> 1
- net /DAC_USB_D-: track 58.5 -> 4.89 mm, vias 2 -> 1
- net /MIPI1_D3_P: track 51.9 -> 0.00 mm, vias 2 -> 0
- net /MIPI1_D3_N: track 51.8 -> 0.00 mm, vias 2 -> 0
- net /JOYSTICK_Y: track 52.2 -> 2.97 mm, vias 2 -> 0
- net /HUB2_DS_3_D+: track 48.0 -> 0.00 mm, vias 4 -> 0
- net /HUB2_DS_3_D-: track 47.2 -> 0.00 mm, vias 4 -> 0
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- added copper zone on F.Cu, net +5V_MAIN
- removed copper zone on B.Cu, net +5V_MAIN
Other:
- board size 208.1 x 167.2 mm -> 209.6 x 164.2 mm
- board text added: "Joystick"
- board text added: "Line-In"
- board text added: "LoRa PWR"
- board text added: "SIM"
- board text added: "SPEAKERS"
- board text added: "USB 2.0"
- board text added: "USB 3.0"
- board text added: "jetdeck.io"
- board text removed: "16MB"
- board text removed: "18x9mm"
- board text removed: "3-18V 6 AMP"
- board text removed: "3.3V"
- board text removed: "5V"
- board text removed: "Accessory"
- board text removed: "Amp"
- board text removed: "CH334R"
- board text removed: "CM5 BOOT"
- board text removed: "EN"
- board text removed: "Flash"
- board text removed: "MCU"
- board text removed: "PAM8406"
- board text removed: "QMK Keyboard"
- board text removed: "RP2040"
- board text removed: "STM32F"
- board text removed: "Thumbstick"
- board text removed: "USB Hub"
- board text removed: "USB-A 5Gbps"
- board text removed: "VIN"
