File: PCB/cyberdeck/cyberdeck.kicad_sch (KiCad schematic)
At the start: 636 parts, among them J1 CPU_FAN, J10 DM3AT-SF-PEJM5, J11 Conn_01x22, J12 HDMI_C_1.3, J13 USB_C_Receptacle_USB2.0_16P, J14 USB_C_Receptacle_USB2.0_16P, J15 PZ254-2-20-W-8.5, J16 1-2199119-5, J17 2199230-3, J18 SIM_Card, J19 TSOP77438TR, J2 GP_LB, J20 Conn_01x22, J21 DX07S024JJ2R1300, J22 USB3_A, J23 Conn_01x06_Pin, J24 Conn_01x06_Pin, J25 USB_C_Receptacle_USB2.0_16P, J3 GP_RB, J5 Conn_01x06_Pin, J6 USB_C_Receptacle_USB2.0_16P, J7 Conn_01x05, J8 PJ-342B, J9 RJ45_LED_Shielded, Q1 IRLML6244, Q2 CJ2101, Q3 SI4174DY-T1-GE3_N-Channel_FET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, Q5 IRLML6244, Q6 SI4174DY-T1-GE3_N-Channel_FET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, Q7 SI4174DY-T1-GE3_N-Channel_FET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, Q8 SI4174DY-T1-GE3_N-Channel_FET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, U1 W25Q128JVS, U12 SY6280_OCP, U13 USBLC6-2SC6, U14 USBLC6-2SC6, U15 SY6280_OCP, U16 BQ76905RGRR, U17 ATtiny404-SS, U18 TPS25751SRSMR, U19 HD3SS3220IRNHT, U2 STM32F072CBT6, U20 TPD4EUSB30DQAR, U21 TPD4EUSB30DQAR, U22 AT24CS01-SSHM, U23 CH334R, U24 AT3H7B-CuH-S, U25 SY6280_OCP, U26 SY6280_OCP, U27 USBLC6-2SC6, U28 SY6280_OCP, U29 SY6280_OCP, U3 XC6206, U30 SY6280_OCP, U32 AT3H7B-CuH-S, U33 SY6280_OCP, U34 SY6280_OCP, U35 TLV70012_SOT23-5, U36 TUSB8041, U37 RAK4630, U38 TPS70933DBVR, U39 USBLC6-2SC6, U4 BQ25792RQMR, U40 MLX90632, U41 TPS566231RQFR, U42 TPS566231RQFR, U43 AT3H7B-CuH-S, U44 AT3H7B-CuH-S, U5 RP2040, U6 USBLC6-2SC6, U7 CH334R, U8 PAM8406AB, U9 PCM2706CPJT, X1 X322512MSB4SI, X2 X322512MSB4SI, X3 X322512MSB4SI, X4 X322512MSB4SI, X5 X322512MSB4SI

Commit message: stuff and things
Parts:
- removed J25: USB_C_Receptacle_USB2.0_16P, LibraryGlobalFootprints:USB_C_Receptacle_HRO_TYPE-C-31-M-12, symbol Connector:USB_C_Receptacle_USB2.0_16P
- removed R128, R129: 5.1K, Resistor_SMD:R_0402_1005Metric, symbol Device:R
- removed U39: USBLC6-2SC6, Package_TO_SOT_SMD:SOT-23-6, symbol Power_Protection:USBLC6-2SC6
- added C179, C181, C182, C183, C65: 10uF, Capacitor_SMD:C_0805_2012Metric, symbol Adafruit TFP401 to 40pin TFT-eagle-import:CAP_CERAMIC0805-NOOUTLINE
- added C180, C186, C55, C56, C57, C60, C61, C62, C63, C64: 0.1uF, Capacitor_SMD:C_0805_2012Metric, symbol Adafruit TFP401 to 40pin TFT-eagle-import:CAP_CERAMIC0805-NOOUTLINE
- added C184, C185: 1uF, Capacitor_SMD:C_0805_2012Metric, symbol Adafruit TFP401 to 40pin TFT-eagle-import:CAP_CERAMIC0805-NOOUTLINE
- added C58: 0.1uF, Capacitor_SMD:C_0805_2012Metric, symbol Adafruit TFP401 to 40pin TFT-eagle-import:CAP_CERAMIC_0805MP
- added C59: 100uF - REMOVED, Library-display-driver:PANASONIC_C, symbol Adafruit TFP401 to 40pin TFT-eagle-import:CAP_ELECTROLYTICPANASONIC_C
- added D1: MBR0540, Diode_SMD:D_SOD-123, symbol Diode:MBR0540
- added D2: MM3Z24VT1G, Diode_SMD:D_SOD-323, symbol Device:D
- added D3: 1N4148, Diode_SMD:D_SOD-323, symbol Diode:1N4148
- added D42, D43: LED_0402, LED_SMD:LED_0402_1005Metric, symbol Device:LED
- added FB1, FB2, FB3, FB4: Ferrite, Inductor_SMD:L_0805_2012Metric, symbol Adafruit TFP401 to 40pin TFT-eagle-import:FERRITE_0805MP
- added H5: SMTWE2030MTJ, LibraryGlobalFootprints:M.2 M2 nut standoff, symbol Mechanical:MountingHole_Pad
- added J25: PJ-342B, LibraryGlobalFootprints:PJ-342B, symbol LibraryGlobalSymbols:PJ-342B
- added J26: Conn_01x04_Pin, Connector_PinHeader_1.00mm:PinHeader_1x04_P1.00mm_Vertical, symbol Connector:Conn_01x04_Pin
- added JP3: HEADER-1X2ROUND, Library-display-driver:1X02_ROUND, symbol Adafruit TFP401 to 40pin TFT-eagle-import:HEADER-1X2ROUND
- added JP7: HEADER-1X476MIL, Library-display-driver:1X04_ROUND_76, symbol Adafruit TFP401 to 40pin TFT-eagle-import:HEADER-1X476MIL
- added L1: BRL3225T150K, Library-display-driver:INDUCTOR_5X5MM_NR5040_NOTHERMALS, symbol Adafruit TFP401 to 40pin TFT-eagle-import:INDUCTORNR5040
- added LED2: Green, LED_SMD:LED_0805_2012Metric, symbol Device:LED
- added LED3: Blue, LED_SMD:LED_0805_2012Metric, symbol Device:LED
- added Q4: BSS138, Package_TO_SOT_SMD:SOT-23, symbol Adafruit TFP401 to 40pin TFT-eagle-import:MOSFET-NREFLOW
- added R128, R129, R144, R145, R51, R52, R53: 33, Resistor_SMD:R_Array_Convex_4x0603, symbol Adafruit TFP401 to 40pin TFT-eagle-import:RESISTOR_4PACK_US
- added R146, R20, R21, R22, R48: 10K, Resistor_SMD:R_0805_2012Metric, symbol Adafruit TFP401 to 40pin TFT-eagle-import:RESISTOR0805_NOOUTLINE
- added R147: 3 ohm, Resistor_SMD:R_0805_2012Metric, symbol Adafruit TFP401 to 40pin TFT-eagle-import:RESISTOR0805_NOOUTLINE
- added R148, R149: 12 ohm, Resistor_SMD:R_0805_2012Metric, symbol Adafruit TFP401 to 40pin TFT-eagle-import:RESISTOR0805_NOOUTLINE
- added R150, R151, R50: 1K, Resistor_SMD:R_0805_2012Metric, symbol Adafruit TFP401 to 40pin TFT-eagle-import:RESISTOR0805_NOOUTLINE
- added R152, R153: 100K, Resistor_SMD:R_0402_1005Metric, symbol Device:R
- added R49: 10K, Resistor_SMD:R_0805_2012Metric, symbol Adafruit TFP401 to 40pin TFT-eagle-import:RESISTOR_0805MP
- added SJ2, SJ3: SOLDERJUMPER, Library-display-driver:SOLDERJUMPER_ARROW_NOPASTE, symbol Adafruit TFP401 to 40pin TFT-eagle-import:SOLDERJUMPER
- added SJ4: +50mA, Library-display-driver:SOLDERJUMPER_ARROW_NOPASTE, symbol Adafruit TFP401 to 40pin TFT-eagle-import:SOLDERJUMPER
- added SJ5: +25mA, Library-display-driver:SOLDERJUMPER_ARROW_NOPASTE, symbol Adafruit TFP401 to 40pin TFT-eagle-import:SOLDERJUMPER
- added U10: 24LC02BT-I/OT, Package_TO_SOT_SMD:SOT-23-5, symbol Adafruit TFP401 to 40pin TFT-eagle-import:EEPROM_I2C_MCP24AA32
- added U11: LT1117(3V3), Package_TO_SOT_SMD:SOT-223-3_TabPin2, symbol Adafruit TFP401 to 40pin TFT-eagle-import:VREG_SOT223
- added U39: TFP401, LibraryGlobalFootprints:TFP401 - S-PQFP-G100, symbol Adafruit TFP401 to 40pin TFT-eagle-import:TFP401
- added U45: FAN5333ASX, Package_TO_SOT_SMD:SOT-23-5, symbol Adafruit TFP401 to 40pin TFT-eagle-import:VREG_FAN5331
- added X6: AFC07-S20FCC-00, Connector_FFC-FPC:TE_2-1734839-0_1x20-1MP_P0.5mm_Horizontal, symbol LibraryGlobalSymbols:HDMI_20-pin-header-MOLEX_47151DIM
- added X7: AFC07-S40ECA-00, LibraryGlobalFootprints:FFC_Receptable_1x40_P0.5mm_AFC07-S40ECA-00, symbol Adafruit TFP401 to 40pin TFT-eagle-import:XF2-40?-RARBT
- J9: value RJ45_LED_Shielded -> RJ45_Shielded; footprint LibraryGlobalFootprints:RC01812 -> CONN-SMD_RJ-064; symbol Connector:RJ45_LED_Shielded -> LibraryGlobalSymbols:RJ-064-1; LCSC Part (none) -> C7205199
- renumbered BT1 to BATT1, BT2 to BATT2
Connections:
- net 5V_IN is gone; now on net VBATT: U43.4
- net CAM_GPIO0: now also J11.6 (Pin_6); no longer J20.6 (Pin_6)
- net CAM_GPIO1: now also J11.5 (Pin_5); no longer J20.5 (Pin_5)
- net CHA_GND: now also J9.10 (EH), J9.11 (EH), J9.12 (EH), J9.9 (EH); no longer J9.SH
- net CM5_3V3: now also D42.2 (A), D43.2 (A); no longer J9.10, J9.12
- net GND: now also C179.2, C180.2, C181.2, C182.2, C183.1, C184.2, C185.2, C186.2, C55.2, C56.2, C57.2, C58.2, C59.-, C60.2, C61.2, C62.2, C63.2, C64.2, C65.2, H5.1, JP3.1, JP7.2, Q4.2 (S), R148.2, R152.1, R153.1, R49.1, R50.2, SJ3.1, SJ4.1, SJ5.2, U10.2 (GND), U10.5 (WP), U11.1 (GND), U39.1 (DFO), U39.19 (OGND@1), U39.28 (OGND@2), U39.39 (GND@2), U39.4 (PIXS), U39.45 (OGND@3), U39.5 (GND@1), U39.58 (OGND@4), U39.68 (GND@3), U39.76 (OGND@5), U39.79 (AGND@1), U39.83 (AGND@2), U39.87 (AGND@3), U39.89 (AGND@4), U39.92 (AGND@5), U39.98 (PGND), U39.P$1 (TP), U39.P$10 (TP), U39.P$11 (TP), U39.P$12 (TP), U39.P$13 (TP), U39.P$14 (TP), U39.P$15 (TP), U39.P$16 (TP), U39.P$2 (TP), U39.P$3 (TP), U39.P$4 (TP), U39.P$5 (TP), U39.P$6 (TP), U39.P$7 (TP), U39.P$8 (TP), U39.P$9 (TP), U39.THERMAL (TP), U45.2 (GND), X6.12 (TX0_SHIELD), X6.15 (TX1_SHIELD), X6.18 (TX2_SHIELD), X6.8 (GND), X6.9 (TXC_SHIELD), X7.29 (MS), X7.3 (MS), X7.36 (MS)
- net MIPI0_CLK_N: now also J11.15 (Pin_15); no longer J20.15 (Pin_15)
- net MIPI0_CLK_P: now also J11.14 (Pin_14); no longer J20.14 (Pin_14)
- net MIPI0_D0_N: now also J11.21 (Pin_21); no longer J20.21 (Pin_21)
- net MIPI0_D0_P: now also J11.20 (Pin_20); no longer J20.20 (Pin_20)
- net MIPI0_D1_N: now also J11.18 (Pin_18); no longer J20.18 (Pin_18)
- net MIPI0_D1_P: now also J11.17 (Pin_17); no longer J20.17 (Pin_17)
- net MIPI0_D2_N: now also J11.12 (Pin_12); no longer J20.12 (Pin_12)
- net MIPI0_D2_P: now also J11.11 (Pin_11); no longer J20.11 (Pin_11)
- net MIPI0_D3_N: now also J11.9 (Pin_9); no longer J20.9 (Pin_9)
- net MIPI0_D3_P: now also J11.8 (Pin_8); no longer J20.8 (Pin_8)
- net MIPI0_SCL: now also J11.3 (Pin_3), R55.2; no longer J20.3 (Pin_3), R83.2
- net MIPI0_SDA: now also J11.2 (Pin_2), R54.2; no longer J20.2 (Pin_2), R84.2
- net MIPI1_CLK_N: now also J20.15 (Pin_15); no longer J11.15 (Pin_15)
- net MIPI1_CLK_P: now also J20.14 (Pin_14); no longer J11.14 (Pin_14)
- net MIPI1_D0_N: now also J20.21 (Pin_21); no longer J11.21 (Pin_21)
- net MIPI1_D0_P: now also J20.20 (Pin_20); no longer J11.20 (Pin_20)
- net MIPI1_D1_N: now also J20.18 (Pin_18); no longer J11.18 (Pin_18)
- net MIPI1_D1_P: now also J20.17 (Pin_17); no longer J11.17 (Pin_17)
- net MIPI1_D2_N: now also J20.12 (Pin_12); no longer J11.12 (Pin_12)
- net MIPI1_D2_P: now also J20.11 (Pin_11); no longer J11.11 (Pin_11)
- net MIPI1_D3_N: now also J20.9 (Pin_9); no longer J11.9 (Pin_9)
- net MIPI1_D3_P: now also J20.8 (Pin_8); no longer J11.8 (Pin_8)
- net MIPI1_SCL: now also J20.3 (Pin_3), R83.2; no longer J11.3 (Pin_3), R55.2
- net MIPI1_SDA: now also J20.2 (Pin_2), R84.2; no longer J11.2 (Pin_2), R54.2
- net PWR_TRIGGER_3V3: now also R153.2
- net PWR_TRIGGER_5V: now also R152.2
- net VIN: now also C179.1, C183.2, C59.+, C65.1, L1.P$1 (1), R146.1, U11.3 (IN), U45.5 (VIN)
- net at R110.1: now also D43.1 (K); no longer J9.9
- net at R82.1: now also D42.1 (K); no longer J9.11
- net 3V3_IN renamed VBATT
- new net: R53.6 (2), X7.10 (MS)
- new net: R52.5 (2), X7.5 (MS)
- new net: C57.1, C58.1, C60.1, C61.1, FB2.2 (P$2), U39.18 (OVDD@1), U39.29 (OVDD@2), U39.43 (OVDD@3), U39.57 (OVDD@4), U39.78 (OVDD@5)
- new net: R147.2, SJ4.2
- new net: R149.2, SJ5.1
- new net: R22.1, X6.4 (HOTPLUG)
- new net: R51.2 (1), U39.47 (VSYNC)
- new net: C180.1, FB4.2 (P$2), U39.97 (PVDD)
- new net: Q4.1 (G), R150.2
- new net: R144.5 (2), X7.21 (MS)
- new net: R129.7 (2), X7.19 (MS)
- new net: R129.8 (2), X7.20 (MS)
- new net: R128.6 (2), X7.14 (MS)
- new net: R144.7 (2), X7.23 (MS)
- new net: R129.6 (2), X7.18 (MS)
- new net: LED3.1 (K), R151.1
- new net: Q4.3 (D), R151.2
- new net: R52.7 (2), X7.7 (MS)
- new net: R145.5 (2), X7.25 (MS)
- new net: D3.2 (A), JP3.2, R146.2, U45.4 (SHDN)
- new net: R52.8 (2), X7.8 (MS)
- new net: R51.1, U39.48 (HSYNC)
- new net: R49.2, SJ2.1, U39.100 (OCK_INV)
- new net: R144.6 (2), X7.22 (MS)
- new net: R48.2, SJ3.2, U39.3 (ST)
- new net: R145.7 (2), X7.27 (MS)
- new net: LED2.1 (K), R50.1
- new net: R145.8 (2), X7.28 (MS)
- new net: R52.6 (2), X7.6 (MS)
- new net: R128.8 (2), X7.16 (MS)
- new net: R53.7 (2), X7.11 (MS)
- new net: R51.3 (1), U39.46 (DE)
- new net: D1.2 (A), L1.P$2 (2), U45.1 (SW)
- new net: R145.6 (2), X7.26 (MS)
- new net: R129.5 (2), X7.17 (MS)
- new net: R51.4 (1), U39.44 (ODCK)
- new net: R128.5 (2), X7.13 (MS)
- new net: R53.5 (2), X7.9 (MS)
- new net: R144.8 (2), X7.24 (MS)
- new net: R53.8 (2), X7.12 (MS)
- new net: R128.7 (2), X7.15 (MS)
- new net 24V: C184.1, C185.1, D1.1 (K), D2.1 (K), X7.2 (MS)
- new net 5.0V: C62.1, JP7.1, R20.2, R21.2, R22.2, U10.4 (VCC), X6.1 (+5V), X6.2 (+5V), X6.3 (+5V)
- new net ACTIVE: D3.1 (K), R150.1, U39.8 (SCDT), X7.31 (MS)
- new net AVDD: C63.1, C64.1, FB3.2 (P$2), U39.82 (AVDD@1), U39.84 (AVDD@2), U39.88 (AVDD@3), U39.95 (AVDD@4)
- new net B0: R144.4 (1), U39.10 (QE0)
- new net B1: R144.3 (1), U39.11 (QE1)
- new net B2: R144.2 (1), U39.12 (QE2)
- new net B3: R144.1, U39.13 (QE3)
- new net B4: R145.4 (1), U39.14 (QE4)
- new net B5: R145.3 (1), U39.15 (QE5)
- new net B6: R145.2 (1), U39.16 (QE6)
- new net B7: R145.1, U39.17 (QE7)
- new net CTL1: U39.40 (CTL1)
- new net CTL2: U39.41 (CTL2)
- new net CTL3: U39.42 (CTL3)
- new net CT_INT: J26.1 (Pin_1), X7.37 (MS)
- new net CT_RESET: J26.2 (Pin_2), X7.38 (MS)
- new net CT_SCL: J26.3 (Pin_3), X7.39 (MS)
- new net CT_SDA: J26.4 (Pin_4), X7.40 (MS)
- new net DISPEN: R51.6 (2), X7.34 (MS)
- new net G0: R128.4 (1), U39.20 (QE8)
- new net G1: R128.3 (1), U39.21 (QE9)
- new net G2: R128.2 (1), U39.22 (QE10)
- new net G3: R128.1, U39.23 (QE11)
- new net G4: R129.4 (1), U39.24 (QE12)
- new net G5: R129.3 (1), U39.25 (QE13)
- new net G6: R129.2 (1), U39.26 (QE14)
- new net G7: R129.1, U39.27 (QE15)
- new net HSYNC: R51.8 (2), X7.32 (MS)
- new net LEDK: C186.1, D2.2 (A), R147.1, R148.1, R149.1, U45.3 (FB), X7.1 (MSV)
- new net PIXCLK: R51.5 (2), X7.30 (MS)
- new net PWRDN: U39.2 (#PD)
- new net PWRDN_O: U39.9 (#PDO)
- new net R0: R52.4 (1), U39.30 (QE16)
- new net R1: R52.3 (1), U39.31 (QE17)
- new net R2: R52.2 (1), U39.32 (QE18)
- new net R3: R52.1, U39.33 (QE19)
- new net R4: R53.4 (1), U39.34 (QE20)
- new net R5: R53.3 (1), U39.35 (QE21)
- new net R6: R53.2 (1), U39.36 (QE22)
- new net R7: R53.1, U39.37 (QE23)
- new net SCL: JP7.3, R21.1, U10.1 (SCL), X6.6 (DCLK)
- new net SDA: JP7.4, R20.1, U10.3 (SDA), X6.5 (DDAT)
- new net TX0+: U39.90 (RX0+), X6.14 (TX0+)
- new net TX0-: U39.91 (RX0-), X6.13 (TX0-)
- new net TX1+: U39.85 (RX1+), X6.17 (TX1+)
- new net TX1-: U39.86 (RX1-), X6.16 (TX1-)
- new net TX2+: U39.80 (RX2+), X6.20 (TX2+)
- new net TX2-: U39.81 (RX2-), X6.19 (TX2-)
- new net TXC+: U39.93 (RXC+), X6.11 (TXC+)
- new net TXC-: U39.94 (RXC-), X6.10 (TXC-)
- new net VDD: C181.1, C182.1, FB1.1 (P$1), FB2.1 (P$1), FB3.1 (P$1), FB4.1 (P$1), LED2.2 (A), LED3.2 (A), U11.2 (OUT), U11.4 (OUT), X7.4 (MS)
- new net VDDIO: C55.1, C56.1, FB1.2 (P$2), R48.1, SJ2.2, U39.38 (DVDD@2), U39.6 (DVDD@1), U39.67 (DVDD@3), U39.7 (#STAG), U39.99 (RSVD)
- new net VSYNC: R51.7 (2), X7.33 (MS)
- no-connect marks 127 -> 152
Other:
- moved on the sheet: C133, C134, C135, C136, R110, R112, R113, R114, R115, R82, U31, U37
