File: PCB/test-power-module-3/test-pwr-3.kicad_sch (KiCad schematic)
At the start: 625 parts, among them J1 CPU_FAN, J10 DM3AT-SF-PEJM5, J11 Conn_01x22, J12 HDMI_C_1.3, J13 USB_C_Receptacle_USB2.0_16P, J14 USB_C_Receptacle_USB2.0_16P, J15 PZ254-2-20-W-8.5, J16 1-2199119-5, J17 2199230-3, J18 SIM_Card, J19 TSOP77438TR, J2 GP_LB, J20 Conn_01x22, J21 DX07S024JJ2R1300, J22 USB3_A, J23 Conn_01x06_Pin, J24 Conn_01x06_Pin, J25 USB_C_Receptacle_USB2.0_16P, J3 GP_RB, J4 JOYSTICK, J5 Conn_01x06_Pin, J6 USB_C_Receptacle_USB2.0_16P, J7 Conn_01x05, J8 PJ-342B, J9 RJ45_LED_Shielded, Q1 IRLML6244, Q2 CJ2101, Q3 SI4174DY-T1-GE3_N-Channel_FET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, Q5 IRLML6244, Q6 SI4174DY-T1-GE3_N-Channel_FET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, Q7 SI4174DY-T1-GE3_N-Channel_FET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, Q8 SI4174DY-T1-GE3_N-Channel_FET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, U1 W25Q128JVS, U12 SY6280_OCP, U13 USBLC6-2SC6, U14 USBLC6-2SC6, U15 SY6280_OCP, U16 BQ76905RGRR, U17 ATtiny404-SS, U18 TPS25751SRSMR, U19 HD3SS3220IRNHT, U2 STM32F072CBT6, U20 TPD4EUSB30DQAR, U21 TPD4EUSB30DQAR, U22 AT24CS01-SSHM, U23 CH334R, U24 AT3H7B-CuH-S, U25 SY6280_OCP, U26 SY6280_OCP, U27 USBLC6-2SC6, U28 SY6280_OCP, U29 SY6280_OCP, U3 XC6206, U30 SY6280_OCP, U32 AT3H7B-CuH-S, U33 SY6280_OCP, U34 SY6280_OCP, U35 TLV70012_SOT23-5, U36 TUSB8041, U37 RAK4630, U38 TPS70933DBVR, U39 USBLC6-2SC6, U4 BQ25792RQMR, U40 MLX90632, U41 TPS566231RQFR, U42 TPS566231RQFR, U5 RP2040, U6 USBLC6-2SC6, U7 CH334R, U8 PAM8406AB, U9 PCM2706CPJT, X1 X322512MSB4SI, X2 X322512MSB4SI, X3 X322512MSB4SI, X4 X322512MSB4SI, X5 X322512MSB4SI

Commit message: test usb 3 hub, test pwr regs v3
Parts:
- removed J4: JOYSTICK, LibraryGlobalFootprints:1x04_P2.54 SMD pads only, symbol Connector:Conn_01x04_Pin
- added R140, R141: 430R, Resistor_SMD:R_0402_1005Metric, symbol Device:R
- added TP27, TP28, TP29, TP30, TP31: TestPoint_Small, TestPoint:TestPoint_Pad_D1.0mm, symbol Connector:TestPoint_Small
- added U43, U44: AT3H7B-CuH-S, LibraryGlobalFootprints:SSOP-4_AT3H7B-CuH-S, symbol Isolator:PC817
Connections:
- net +3.3V_MAIN: now also J7.5 (Pin_5), TP27.1; no longer J7.1 (Pin_1)
- net BQ_3V3: now also U43.1, U44.1
- net GND: now also J7.2 (Pin_2), TP31.1; no longer J7.4 (Pin_4)
- net JOYSTICK_BTN: now also TP29.1
- net JOYSTICK_X: now also J7.4 (Pin_4), TP28.1; no longer J7.2 (Pin_2)
- net JOYSTICK_Y: now also J7.1 (Pin_1), TP30.1; no longer J7.5 (Pin_5)
- net PWR_TRIGGER: now also R140.2, R141.2
- net PWR_TRIGGER_3V3: now reaches TP25.1, U42.3 (EN)
- net PWR_TRIGGER_3V3: now also U44.3
- net PWR_TRIGGER_5V: now reaches TP24.1, U41.3 (EN)
- net PWR_TRIGGER_5V: now also U43.3
- new net: R140.1, U43.2
- new net: R141.1, U44.2
- new net 3V3_IN: U44.4
- new net 5V_IN: U43.4
Other:
- moved on the sheet: TP16, TP18
