File: PCB/cyberdeck-r1b/cyberdeck-r1b.kicad_sch (KiCad schematic)
At the start: 531 parts, among them J1 CPU_FAN, J10 DM3AT-SF-PEJM5, J11 Conn_01x22, J12 HDMI_C_1.3, J13 USB_C_Receptacle_USB2.0_16P, J15 Conn_02x20_Odd_Even, J16 1-2199119-5, J17 2199119-3, J18 SIM_Card, J19 TSOP77438TR, J2 GP_LB, J20 Conn_01x22, J21 DX07S024JJ2R1300, J22 USB_C_Receptacle_USB2.0_16P, J3 GP_RB, J5 Conn_01x06_Pin, J6 USB_C_Receptacle_USB2.0_16P, J7 Conn_01x05, J8 PJ-342B, J9 SPK, Q1 IRLML6244, Q2 CJ2101, Q3 SI4174DY-T1-GE3_N-Channel_FET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, Q4 BSS138, Q5 IRLML6244, Q6 SI4174DY-T1-GE3_N-Channel_FET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, Q7 SI4174DY-T1-GE3_N-Channel_FET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, Q8 SI4174DY-T1-GE3_N-Channel_FET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, U1 W25Q128JVS, U10 TPS62180YZFR, U11 TPS62180YZFR, U12 SY6280_OCP, U14 USBLC6-2SC6, U15 SY6280_OCP, U16 BQ76905RGRR, U17 ATtiny404-SS, U18 TPS25751SRSMR, U19 HD3SS3220IRNHT, U2 STM32F072CBT6, U20 TPD4EUSB30DQAR, U21 TPD4EUSB30DQAR, U22 AT24CS01-SSHM, U24 AT3H7B-CuH-S, U25 USBLC6-2SC6, U28 SY6280_OCP, U3 XC6206, U32 AT3H7B-CuH-S, U33 AT3H7B-CuH-S, U34 AT3H7B-CuH-S, U4 BQ25792RQMR, U5 RP2040, U6 USBLC6-2SC6, U7 CH334R, U8 PAM8406AB, U9 PCM2706CPJT, X1 X322512MSB4SI, X2 X322512MSB4SI, X3 X322512MSB4SI

Commit message: stuff and things
Parts:
- U17: LCSC (none) -> C1339119
Other:
- note added: "Lithium Batt Protect/Balance Circuit"
- note removed: "Lithium Batt Protection Circuit"
