File: PCB/usb-3-hub/usb-3-hub.kicad_pcb (KiCad board)
At the start: 2 copper layers, 78.7 x 51.6 mm, 96 parts, among them J17 2199230-3, J18 SIM_Card, J21 DX07S024JJ2R1300, J22 USB3_A, J23 DX07S024JJ2R1300, J24 USB3_A, U13 USBLC6-2SC6, U14 USBLC6-2SC6, U19 HD3SS3220IRNHT, U20 TPD4EUSB30DQAR, U21 TPD4EUSB30DQAR, U22 TPD4EUSB30DQAR, U23 HD3SS3220IRNHT, U24 TPD4EUSB30DQAR, U29 SY6280_OCP, U33 SY6280_OCP, U35 TLV70012_SOT23-5, U36 TUSB8041, U42 TPS566231RQFR, X5 X322512MSB4SI

Commit message: stuff and things
Parts:
- removed U35: TLV70012_SOT23-5, Package_TO_SOT_SMD:SOT-23-5
- added C177: 1uF, Capacitor_SMD:C_0402_1005Metric, F.Cu at (195.2, 39.4)
- added C178: 100nF, Capacitor_SMD:C_0402_1005Metric, F.Cu at (190.3, 40.5)
- added C179: 100nF, Capacitor_SMD:C_0402_1005Metric, F.Cu at (190.4, 38.5)
- added C180: 22uF, Capacitor_SMD:C_0805_2012Metric, F.Cu at (188.8, 39.4)
- added C181: 22uF, Capacitor_SMD:C_0805_2012Metric, F.Cu at (189.0, 36.2)
- added C182: 22uF, Capacitor_SMD:C_0805_2012Metric, F.Cu at (201.3, 45.9)
- added C183: 22uF, Capacitor_SMD:C_0805_2012Metric, F.Cu at (203.2, 42.4)
- added C184: 47uF, Capacitor_SMD:C_1206_3216Metric, F.Cu at (200.7, 41.8)
- added L8: 2.2uH, Inductor_SMD:L_Sunlord_MWSA0603S, F.Cu at (194.7, 43.7)
- added R137: 12K, Resistor_SMD:R_0402_1005Metric, F.Cu at (195.2, 38.3)
- added R138: 10K, Resistor_SMD:R_0402_1005Metric, F.Cu at (198.3, 39.5)
- added R79: 10K, Resistor_SMD:R_0402_1005Metric, F.Cu at (211.5, 45.9)
- added R80: 10K, Resistor_SMD:R_0402_1005Metric, F.Cu at (217.8, 48.7)
- added R82: 10K, Resistor_SMD:R_0402_1005Metric, F.Cu at (211.6, 44.8)
- added U43: TPS566231RQFR, LibraryGlobalFootprints:TPS566231, F.Cu at (192.5, 38.7)
- X5: value X322512MSB4SI -> X322524MOB4SI
- moved G*** 34.0 mm to (183.8, 44.6)
- moved R98 22.6 mm to (207.2, 34.9), turned to 0 degrees
- moved D36 2.44 mm to (207.2, 33.7)
Routing:
- net Net-(D36-A): track 25.4 -> 1.18 mm, vias 2 -> 0
- net +3.3V_M2B: track 37.8 -> 52.3 mm, vias 2 -> 3
- net +5V_MAIN: track 81.9 -> 95.8 mm, vias 7 -> 9
- net +1.1V_HUB: track 46.8 -> 60.0 mm, vias 2 -> 0
- net Net-(U43-FB): track 0.00 -> 6.77 mm
- net /GNSSEnable: track 0.00 -> 6.33 mm
- net /FlightModeDisable: track 0.00 -> 5.39 mm
- net /M2B_POWER_OFF: track 0.00 -> 4.39 mm
- net /M2B_LED: track 10.4 -> 14.5 mm
- net Net-(U43-SW): track 0.00 -> 3.11 mm
- net +3.3V_MAIN: track 143.6 -> 140.5 mm, vias 14 -> 13
- net Net-(U43-VCC): track 0.00 -> 1.39 mm
- net GND: vias 111 -> 150
Other:
- board text added: "1.1V VREG"
- board text added: "micro SIM"
- board text added: "power"
- board text added: "wwan activity"
- board text removed: "bzzzzzzzzzzz"
- board text removed: "data go brrr"
- board text removed: "emotional support component"
- board text removed: "insert coin(s)"
- board text removed: "internet doing things"
- board text removed: "test point (decoy)"
