File: PCB/usb-3-hub/usb-3-hub.kicad_sch (KiCad schematic)
At the start: 96 parts, among them J17 2199230-3, J18 SIM_Card, J21 DX07S024JJ2R1300, J22 USB3_A, J23 DX07S024JJ2R1300, J24 USB3_A, U13 USBLC6-2SC6, U14 USBLC6-2SC6, U19 HD3SS3220IRNHT, U20 TPD4EUSB30DQAR, U21 TPD4EUSB30DQAR, U22 TPD4EUSB30DQAR, U23 HD3SS3220IRNHT, U24 TPD4EUSB30DQAR, U29 SY6280_OCP, U33 SY6280_OCP, U35 TLV70012_SOT23-5, U36 TUSB8041, U42 TPS566231RQFR, X5 X322512MSB4SI

Commit message: stuff and things
Parts:
- removed U35: TLV70012_SOT23-5, Package_TO_SOT_SMD:SOT-23-5, symbol Regulator_Linear:TLV70012_SOT23-5
- added C177: 1uF, Capacitor_SMD:C_0402_1005Metric, symbol Device:C_Small
- added C178, C179: 100nF, Capacitor_SMD:C_0402_1005Metric, symbol Device:C_Small
- added C180, C181, C182, C183: 22uF, Capacitor_SMD:C_0805_2012Metric, symbol Device:C_Small
- added C184: 47uF, Capacitor_SMD:C_1206_3216Metric, symbol Device:C_Small
- added L8: 2.2uH, Inductor_SMD:L_Sunlord_MWSA0603S, symbol Device:L
- added R137: 12K, Resistor_SMD:R_0402_1005Metric, symbol Device:R
- added R138, R82: 10K, Resistor_SMD:R_0402_1005Metric, symbol Device:R
- added U43: TPS566231RQFR, LibraryGlobalFootprints:TPS566231, symbol LibraryGlobalSymbols:TPS566231RQFR
- R79, R80: now fitted; now in the parts list
- X5: value X322512MSB4SI -> X322524MOB4SI; LCSC C9002 -> C70590
Connections:
- net +1.1V_HUB: now also C182.2, C183.2, C184.2, L8.2, R138.2
- net +3.3V_M2B: now also R82.1
- net +5V_MAIN: now also C179.2, C180.1, C181.1, U43.5 (VIN), U43.6 (VIN)
- net GND: now also C177.1, C179.1, C180.2, C181.2, C182.1, C183.1, C184.1, R137.1, U43.4 (PGND)
- net M2B_POWER_OFF: now also R82.2
- new net: R137.2, R138.1, U43.2 (FB)
- new net: C177.2, U43.1 (VCC)
- new net: C178.1, U43.7 (BST)
- new net: C178.2, L8.1, U43.8 (SW)
- no-connect marks 69 -> 71
Other:
- moved on the sheet: C168, C169, C170, C171, C172, C173, C174, C175, C176, C18, C54, C76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
